File: extruderController/extruderControllerv1.brd (EAGLE design)
At the start: 117.8 x 68.6 mm, 49 parts, among them IC1 LM1117MPX-5.0, IC2 MAX3467CPA, IC4 ULN2003AD, Q2 PH7030L, Q3 PH7030L, Q4 PH7030L, Q5 PH7030L, Q6 PH7030L, U1 ATMEGA2560AU, X1 22-23-2081, X2 22-23-2081, X3 0446200002, X4 22-23-2021, X5 22-23-2051, X6 22-23-2041, X7 22-23-2041

Commit message: k
Parts:
- added C12: 0.1uF, rcl:C0603
- added R12, R13: (no value), rcl:R1210
- moved X4 109.6 mm to (15.2, 64.8), turned to 0 degrees
- moved D1 77.0 mm to (20.3, 58.4)
- moved C5 71.6 mm to (30.5, 64.8)
- moved C1 70.3 mm to (25.4, 63.5)
- moved C6 54.6 mm to (40.6, 58.4)
- moved IC1 49.9 mm to (35.6, 61.0), turned to 180 degrees
- moved R1 47.8 mm to (40.6, 48.3)
- moved C7 33.7 mm to (43.2, 49.5)
- moved C2 33.6 mm to (44.5, 63.5), turned to 270 degrees
- moved X3 31.2 mm to (109.2, 33.0), turned to 270 degrees
- moved SV1 11.7 mm to (61.0, 55.9)
- moved C4 10.5 mm to (33.0, 54.6)
- moved Q1 10.2 mm to (30.5, 50.8)
- moved C3 9.25 mm to (27.9, 54.6)
- moved IC2 8.98 mm to (94.0, 33.0)
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Connections:
- removed net VCC: IC2.1
- new net N$27: IC2.7, R13.1, X3.5
- new net N$33: IC2.6, R12.1, X3.3
- new net N$35: IC2.5, R12.2, X3.1
- new net N$36: IC2.8, R13.2, X3.7
- net +5V: now also C12.1, IC2.1
- net GND: now also C12.2, X3.2, X3.4, X3.6, X3.8

Commit message: s
Parts:
- removed X3: 0446200002, con-molex:0446200002
- removed X4: 22-23-2021, con-molex:22-23-2021
- removed X7: 22-23-2041, con-molex:22-23-2041
- added C13, C14, C15, C16, C17, C18: 0.1uF, rcl:C0603
- added D2, D3, D4, D5, D6: 250mA/100V, SparkFun-DiscreteSemi:SOD-323
- added J1: RJ45, SparkFun-Connectors:RJ45-8
- added J2: (no value), SparkFun-Connectors:SCREWTERMINAL-3.5MM-2
- added J3, J4, J5: (no value), SparkFun-Connectors:2X8
- added LED1: (no value), led:SML1206
- added R14, R15, R16, R17, R18: (no value), rcl:R0805
- added X8, X9: 22-23-2031, con-molex:22-23-2031
- moved C12 41.8 mm to (55.9, 52.1)
- moved R13 41.5 mm to (63.5, 52.1), turned to 180 degrees
- moved IC2 41.0 mm to (55.9, 48.3)
- moved R12 39.8 mm to (66.0, 47.0), turned to 0 degrees
- moved H3 24.1 mm to (88.9, 5.08)
- moved H4 24.1 mm to (88.9, 63.5)
- moved SV1 17.9 mm to (43.2, 53.8)
- moved R1 12.9 mm to (28.2, 44.7), turned to 0 degrees
- moved U1 10.2 mm to (39.4, 38.1)
- moved IC4 9.92 mm to (66.0, 24.1)
- moved C4 7.64 mm to (25.4, 54.1), turned to 0 degrees
- moved X6 7.62 mm to (77.5, 3.81)
- moved C6 6.48 mm to (41.9, 64.8)
- moved R3 5.45 mm to (18.8, 50.8)
- moved R5 5.45 mm to (18.8, 41.9)
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Connections:
- new net N$30: IC4.13, R14.1
- new net N$38: IC4.12, R15.1
- new net N$39: IC4.11, R16.1
- new net N$40: IC4.10, R17.1
- new net N$41: LED1.A, R18.2
- new net PD0: U1.43, X9.2
- new net PD1: U1.44, X8.2
- net +12V: now also D2.C, D3.C, D4.C, D5.C, D6.C, J2.1; no longer X4.1
- net +5V: now also C13.1, C14.1, C15.1, C16.1, C17.1, C18.1, IC4.9, LED1.C, X8.1, X9.1
- net GND: now also C13.2, C14.2, C15.2, C16.2, C17.2, C18.2, J1.1, J1.3, J1.5, J1.7, J2.2, R18.1, X8.3, X9.3; no longer X3.2, X3.4, X3.6, X3.8, X4.2
- net N$12: now also R15.2, X1.3; no longer IC4.11, X1.5
- net N$13: now also R16.2, X1.5; no longer IC4.12, X1.3
- net N$14: now also R17.2, X1.7; no longer IC4.13, X1.1
- net N$22: now also D2.A
- net N$25: now also D3.A
- net N$27: now also J1.6; no longer X3.5
- net N$28: now also D4.A
- net N$3: now also R14.2, X1.1; no longer IC4.10, X1.7
- net N$31: now also D5.A
- net N$33: now also J1.4; no longer X3.3
- net N$34: now also D6.A
- net N$35: now also J1.2; no longer X3.1
- net N$36: now also J1.8; no longer X3.7
Routing:
- net PJ7: track 0.00 -> 23.6 mm
- net PA0: track 0.00 -> 22.3 mm
- net PA1: track 0.00 -> 20.8 mm
- net PA2: track 0.00 -> 19.3 mm
- net PA3: track 0.00 -> 19.2 mm
- net PL0: track 0.00 -> 18.6 mm
- net N$19: track 0.00 -> 18.3 mm
- net N$20: track 0.00 -> 15.6 mm
- net GND: track 0.00 -> 14.7 mm
- net PB2(MOSI): track 0.00 -> 14.3 mm
- net PL1: track 0.00 -> 13.8 mm
- net +5V: track 0.00 -> 13.7 mm
- net PL2: track 0.00 -> 12.9 mm
- net PB1(SCK): track 0.00 -> 11.6 mm
- net PB3(MISO): track 0.00 -> 10.2 mm
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Other:
- board size 117.8 x 68.6 mm -> 93.7 x 68.6 mm
- board text added: "Controller"
- board text added: "Extruder"
- board text added: "Hopper level"
- board text added: "v1"
