File: extruderController/extruderControllerv1.sch (EAGLE design)
At the start: 49 parts, among them IC1 LM1117MPX-5.0, IC2 MAX3467CPA, IC4 ULN2003AD, Q2 PH7030L, Q3 PH7030L, Q4 PH7030L, Q5 PH7030L, Q6 PH7030L, U1 ATMEGA2560AU, X1 22-23-2081, X2 22-23-2081, X3 0446200002, X4 22-23-2021, X5 22-23-2051, X6 22-23-2041, X7 22-23-2041

Commit message: k
Parts:
- added C12: 0.1uF, rcl:C-EUC0603
- added R12, R13: (no value), rcl:R-EU_R1210
Connections:
- new net N$27: IC2.B, R13.1, X3.5
- new net N$33: IC2.Z, R12.1, X3.3
- new net N$35: IC2.Y, R12.2, X3.1
- new net N$36: IC2.A, R13.2, X3.7
- net +5V: now also C12.1, IC2.VCC
- net GND: now also C12.2, IC2.GND, X3.2, X3.4, X3.6, X3.8
Other:
- moved on the sheet: X3
Changed lines of the file:
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@@
 <part name="GND20" library="supply1" library_urn="urn:adsk.eagle:library:371" deviceset="GND" device=""/>
 <part name="GND21" library="supply1" library_urn="urn:adsk.eagle:library:371" deviceset="GND" device=""/>
+<part name="C12" library="rcl" library_urn="urn:adsk.eagle:library:334" deviceset="C-EU" device="C0603" package3d_urn="urn:adsk.eagle:package:23616/2" value="0.1uF"/>
+<part name="R12" library="rcl" library_urn="urn:adsk.eagle:library:334" deviceset="R-EU_" device="R1210" package3d_urn="urn:adsk.eagle:package:23554/2"/>
+<part name="R13" library="rcl" library_urn="urn:adsk.eagle:library:334" deviceset="R-EU_" device="R1210" package3d_urn="urn:adsk.eagle:package:23554/2"/>
+<part name="P+14" library="supply1" library_urn="urn:adsk.eagle:library:371" deviceset="+5V" device=""/>
+<part name="P+15" library="supply1" library_urn="urn:adsk.eagle:library:371" deviceset="+5V" device=""/>
+<part name="GND22" library="supply1" library_urn="urn:adsk.eagle:library:371" deviceset="GND" device=""/>
+<part name="GND23" library="supply1" library_urn="urn:adsk.eagle:library:371" deviceset="GND" device=""/>
+<part name="GND24" library="supply1" library_urn="urn:adsk.eagle:library:371" deviceset="GND" device=""/>
 </parts>
 <sheets>
@@
 <attribute name="NAME" x="-259.08" y="132.842" size="1.524" layer="95" rot="R180"/>
 </instance>
-<instance part="X3" gate="P" x="190.5" y="127" smashed="yes">
-<attribute name="NAME" x="194.31" y="137.668" size="1.778" layer="95"/>
-<attribute name="VALUE" x="194.31" y="116.078" size="1.778" layer="96"/>
+<instance part="X3" gate="P" x="180.34" y="124.46" smashed="yes">
+<attribute name="NAME" x="184.15" y="135.128" size="1.778" layer="95"/>
+<attribute name="VALUE" x="184.15" y="113.538" size="1.778" layer="96"/>
 </instance>
 <instance part="SV1" gate="1" x="-22.86" y="149.86" smashed="yes">
@@
 <instance part="GND21" gate="1" x="-254" y="-40.64" smashed="yes">
 <attribute name="VALUE" x="-256.54" y="-43.18" size="1.778" layer="96"/>
+</instance>
+<instance part="C12" gate="G$1" x="162.56" y="106.68" smashed="yes">
+<attribute name="NAME" x="164.084" y="107.061" size="1.778" layer="95"/>
+<attribute name="VALUE" x="164.084" y="101.981" size="1.778" layer="96"/>
+</instance>
+<instance part="R12" gate="G$1" x="157.48" y="132.08" smashed="yes">
+<attribute name="NAME" x="153.67" y="133.5786" size="1.778" layer="95"/>
+<attribute name="VALUE" x="153.67" y="128.778" size="1.778" layer="96"/>
+</instance>
+<instance part="R13" gate="G$1" x="157.48" y="121.92" smashed="yes">
+<attribute name="NAME" x="153.67" y="123.4186" size="1.778" layer="95"/>
+<attribute name="VALUE" x="153.67" y="118.618" size="1.778" layer="96"/>
+</instance>
+<instance part="P+14" gate="1" x="149.86" y="139.7" smashed="yes" rot="R270">
+<attribute name="VALUE" x="144.78" y="142.24" size="1.778" layer="96"/>
+</instance>
+<instance part="P+15" gate="1" x="162.56" y="111.76" smashed="yes">
+<attribute name="VALUE" x="160.02" y="106.68" size="1.778" layer="96" rot="R90"/>
+</instance>
+<instance part="GND22" gate="1" x="147.32" y="104.14" smashed="yes">
+<attribute name="VALUE" x="144.78" y="101.6" size="1.778" layer="96"/>
+</instance>
+<instance part="GND23" gate="1" x="162.56" y="99.06" smashed="yes">
+<attribute name="VALUE" x="160.02" y="96.52" size="1.778" layer="96"/>
+</instance>
+<instance part="GND24" gate="1" x="175.26" y="111.76" smashed="yes">
+<attribute name="VALUE" x="172.72" y="109.22" size="1.778" layer="96"/>
 </instance>
 </instances>
@@
 <pinref part="GND21" gate="1" pin="GND"/>
 <wire x1="-254" y1="-38.1" x2="-254" y2="-35.56" width="0.1524" layer="91"/>
+</segment>
+<segment>
+<pinref part="IC2" gate="G$1" pin="GND"/>
+<pinref part="GND22" gate="1" pin="GND"/>
+<wire x1="147.32" y1="106.68" x2="147.32" y2="114.3" width="0.1524" layer="91"/>
+</segment>
+<segment>
+<pinref part="C12" gate="G$1" pin="2"/>
+<pinref part="GND23" gate="1" pin="GND"/>
+</segment>
+<segment>
+<pinref part="X3" gate="P" pin="2"/>
+<wire x1="177.8" y1="132.08" x2="175.26" y2="132.08" width="0.1524" layer="91"/>
+<wire x1="175.26" y1="132.08" x2="175.26" y2="127" width="0.1524" layer="91"/>
+<pinref part="X3" gate="P" pin="4"/>
+<wire x1="175.26" y1="127" x2="177.8" y2="127" width="0.1524" layer="91"/>
+<pinref part="X3" gate="P" pin="6"/>
+<wire x1="175.26" y1="127" x2="175.26" y2="121.92" width="0.1524" layer="91"/>
+<wire x1="175.26" y1="121.92" x2="177.8" y2="121.92" width="0.1524" layer="91"/>
+<junction x="175.26" y="127"/>
+<pinref part="X3" gate="P" pin="8"/>
+<wire x1="175.26" y1="121.92" x2="175.26" y2="116.84" width="0.1524" layer="91"/>
+<wire x1="175.26" y1="116.84" x2="177.8" y2="116.84" width="0.1524" layer="91"/>
+<junction x="175.26" y="121.92"/>
+<pinref part="GND24" gate="1" pin="GND"/>
+<wire x1="175.26" y1="116.84" x2="175.26" y2="114.3" width="0.1524" layer="91"/>
+<junction x="175.26" y="116.84"/>
 </segment>
 </net>
@@
 <wire x1="-185.42" y1="-40.64" x2="-187.96" y2="-40.64" width="0.1524" layer="91"/>
 </segment>
+<segment>
+<pinref part="IC2" gate="G$1" pin="VCC"/>
+<pinref part="P+14" gate="1" pin="+5V"/>
+</segment>
+<segment>
+<pinref part="C12" gate="G$1" pin="1"/>
+<pinref part="P+15" gate="1" pin="+5V"/>
+</segment>
 </net>
 <net name="N$1" class="0">
@@
 </segment>
 </net>
+<net name="N$27" class="0">
+<segment>
+<pinref part="IC2" gate="G$1" pin="B"/>
+<pinref part="R13" gate="G$1" pin="1"/>
+<wire x1="152.4" y1="119.38" x2="147.32" y2="119.38" width="0.1524" layer="91"/>
+<wire x1="152.4" y1="121.92" x2="152.4" y2="119.38" width="0.1524" layer="91"/>
+<wire x1="152.4" y1="119.38" x2="152.4" y2="116.84" width="0.1524" layer="91"/>
+<junction x="152.4" y="119.38"/>
+<pinref part="X3" gate="P" pin="5"/>
+<wire x1="177.8" y1="124.46" x2="170.18" y2="124.46" width="0.1524" layer="91"/>
+<wire x1="152.4" y1="116.84" x2="170.18" y2="116.84" width="0.1524" layer="91"/>
+<wire x1="170.18" y1="116.84" x2="170.18" y2="124.46" width="0.1524" layer="91"/>
+</segment>
+</net>
+<net name="N$33" class="0">
+<segment>
+<pinref part="IC2" gate="G$1" pin="Z"/>
+<wire x1="147.32" y1="129.54" x2="152.4" y2="129.54" width="0.1524" layer="91"/>
+<pinref part="R12" gate="G$1" pin="1"/>
+<wire x1="152.4" y1="132.08" x2="152.4" y2="129.54" width="0.1524" layer="91"/>
+<junction x="152.4" y="129.54"/>
+<pinref part="X3" gate="P" pin="3"/>
+<wire x1="177.8" y1="129.54" x2="152.4" y2="129.54" width="0.1524" layer="91"/>
+</segment>
+</net>
+<net name="N$35" class="0">
+<segment>
+<pinref part="IC2" gate="G$1" pin="Y"/>
+<wire x1="147.32" y1="134.62" x2="162.56" y2="134.62" width="0.1524" layer="91"/>
+<wire x1="162.56" y1="134.62" x2="177.8" y2="134.62" width="0.1524" layer="91"/>
+<pinref part="R12" gate="G$1" pin="2"/>
+<wire x1="162.56" y1="132.08" x2="162.56" y2="134.62" width="0.1524" layer="91"/>
+<junction x="162.56" y="134.62"/>
+<pinref part="X3" gate="P" pin="1"/>
+</segment>
+</net>
+<net name="N$36" class="0">
+<segment>
+<pinref part="X3" gate="P" pin="7"/>
+<pinref part="IC2" gate="G$1" pin="A"/>
+<wire x1="147.32" y1="124.46" x2="162.56" y2="124.46" width="0.1524" layer="91"/>
+<pinref part="R13" gate="G$1" pin="2"/>
+<wire x1="162.56" y1="121.92" x2="162.56" y2="124.46" width="0.1524" layer="91"/>
+<junction x="162.56" y="124.46"/>
+<wire x1="162.56" y1="124.46" x2="167.64" y2="124.46" width="0.1524" layer="91"/>
+<wire x1="177.8" y1="119.38" x2="167.64" y2="119.38" width="0.1524" layer="91"/>
+<wire x1="167.64" y1="119.38" x2="167.64" y2="124.46" width="0.1524" layer="91"/>
+</segment>
+</net>

Commit message: s
Parts:
- removed X3: 0446200002, con-molex:0446200002
- removed X4: 22-23-2021, con-molex:22-23-2021
- removed X7: 22-23-2041, con-molex:22-23-2041
- added C13, C14, C15, C16, C17, C18: 0.1uF, rcl:C-EUC0603
- added D2, D3, D4, D5, D6: 250mA/100V, SparkFun-DiscreteSemi:DIODE-BAS16J
- added J1: RJ45, SparkFun-Connectors:RJ45-8
- added J2: (no value), SparkFun-Connectors:CONN_023.5MM
- added J3, J4, J5: (no value), SparkFun-Connectors:CONN_08X2
- added LED1: (no value), led:LEDSML1206
- added R14, R15, R16, R17, R18: (no value), rcl:R-EU_R0805
- added X8, X9: 22-23-2031, con-molex:22-23-2031
Connections:
- new net N$30: IC4.O4, R14.1
- new net N$38: IC4.O5, R15.1
- new net N$39: IC4.O6, R16.1
- new net N$40: IC4.O7, R17.1
- new net N$41: LED1.A, R18.2
- new net PD0: U1.(SCL/INT0)PD0, X9-2.S
- new net PD1: U1.(SDA/INT1)PD1, X8-2.S
- net +12V: now also D2.C, D3.C, D4.C, D5.C, D6.C, J2.1; no longer X4-1.S
- net +5V: now also C13.1, C14.1, C15.1, C16.1, C17.1, C18.1, IC4.CD+, LED1.C, X8-1.S, X9-1.S
- net GND: now also C13.2, C14.2, C15.2, C16.2, C17.2, C18.2, J1.1, J1.3, J1.5, J1.7, J2.2, R18.1, X8-3.S, X9-3.S; no longer X3.2, X3.4, X3.6, X3.8, X4-2.S
- net N$12: now also R15.2, X1-3.S; no longer IC4.O6, X1-5.S
- net N$13: now also R16.2, X1-5.S; no longer IC4.O5, X1-3.S
- net N$14: now also R17.2, X1-7.S; no longer IC4.O4, X1-1.S
- net N$22: now also D2.A
- net N$25: now also D3.A
- net N$27: now also J1.6; no longer X3.5
- net N$28: now also D4.A
- net N$3: now also R14.2, X1-1.S; no longer IC4.O7, X1-7.S
- net N$31: now also D5.A
- net N$33: now also J1.4; no longer X3.3
- net N$34: now also D6.A
- net N$35: now also J1.2; no longer X3.1
- net N$36: now also J1.8; no longer X3.7
Other:
- moved on the sheet: X1-1, X1-3, X1-5, X1-7
