File: extruderController/extruderControllerv01.sch (EAGLE design)
At the start: 73 parts, among them IC1 LM1117MPX-5.0, IC2 MAX3467CPA, IC4 ULN2003AD, J1 RJ45, Q2 PH7030L, Q3 PH7030L, Q4 PH7030L, Q5 PH7030L, Q6 PH7030L, U1 ATMEGA2560AU, X1 22-23-2081, X2 22-23-2081, X5 22-23-2051, X6 22-23-2041, X8 22-23-2031, X9 22-23-2031

Commit message: g
Parts:
- removed J3, J4, J5: (no value), SparkFun-Connectors:CONN_08X2
- added IC3: ATMEGA2561-16AU, atmel-2005:ATMEGA2561-16AU
Connections:
- removed net N$15: Q3.S, Q4.S, Q5.S, Q6.S, R11.2, R5.2, R7.2, R9.2
- net GND: now also Q3.S, Q4.S, Q5.S, Q6.S, R11.2, R3.2, R5.2, R7.2, R9.2
Changed lines of the file:
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@@
 <part name="P+21" library="supply1" library_urn="urn:adsk.eagle:library:371" deviceset="+5V" device=""/>
 <part name="GND30" library="supply1" library_urn="urn:adsk.eagle:library:371" deviceset="GND" device=""/>
-<part name="J3" library="SparkFun-Connectors" library_urn="urn:adsk.eagle:library:513" deviceset="CONN_08X2" device="" package3d_urn="urn:adsk.eagle:package:38152/1"/>
-<part name="J4" library="SparkFun-Connectors" library_urn="urn:adsk.eagle:library:513" deviceset="CONN_08X2" device="" package3d_urn="urn:adsk.eagle:package:38152/1"/>
-<part name="J5" library="SparkFun-Connectors" library_urn="urn:adsk.eagle:library:513" deviceset="CONN_08X2" device="" package3d_urn="urn:adsk.eagle:package:38152/1"/>
 <part name="D2" library="SparkFun-DiscreteSemi" library_urn="urn:adsk.eagle:library:514" deviceset="DIODE" device="-BAS16J" package3d_urn="urn:adsk.eagle:package:38441/1" value="250mA/100V"/>
 <part name="P+22" library="supply1" library_urn="urn:adsk.eagle:library:371" deviceset="+12V" device=""/>
@@
 <part name="P+26" library="supply1" library_urn="urn:adsk.eagle:library:371" deviceset="+12V" device=""/>
 <part name="P+27" library="supply1" library_urn="urn:adsk.eagle:library:371" deviceset="+5V" device=""/>
+<part name="IC3" library="atmel-2005" deviceset="ATMEGA2561*" device="AU" technology="-16"/>
 </parts>
 <sheets>
@@
 <attribute name="VALUE" x="-189.23" y="-104.902" size="1.778" layer="96"/>
 </instance>
-<instance part="GND15" gate="1" x="-170.18" y="-111.76" smashed="yes">
-<attribute name="VALUE" x="-172.72" y="-114.3" size="1.778" layer="96"/>
+<instance part="GND15" gate="1" x="-170.18" y="-104.14" smashed="yes">
+<attribute name="VALUE" x="-172.72" y="-106.68" size="1.778" layer="96"/>
 </instance>
 <instance part="Q3" gate="G$1" x="-172.72" y="-119.38" smashed="yes">
@@
 <attribute name="VALUE" x="-213.36" y="-55.88" size="1.778" layer="96"/>
 </instance>
-<instance part="J3" gate="G$1" x="86.36" y="60.96" smashed="yes">
-<attribute name="VALUE" x="82.55" y="48.514" size="1.778" layer="96" font="vector"/>
-<attribute name="NAME" x="82.55" y="74.168" size="1.778" layer="95" font="vector"/>
-</instance>
-<instance part="J4" gate="G$1" x="86.36" y="30.48" smashed="yes">
-<attribute name="VALUE" x="82.55" y="18.034" size="1.778" layer="96" font="vector"/>
-<attribute name="NAME" x="82.55" y="43.688" size="1.778" layer="95" font="vector"/>
-</instance>
-<instance part="J5" gate="G$1" x="86.36" y="0" smashed="yes">
-<attribute name="VALUE" x="82.55" y="-12.446" size="1.778" layer="96" font="vector"/>
-<attribute name="NAME" x="82.55" y="13.208" size="1.778" layer="95" font="vector"/>
-</instance>
 <instance part="D2" gate="G$1" x="-175.26" y="-86.36" smashed="yes" rot="R180">
 <attribute name="NAME" x="-172.72" y="-88.392" size="1.778" layer="95" font="vector" rot="R180"/>
@@
 <instance part="P+27" gate="1" x="-226.06" y="-35.56" smashed="yes" rot="R270">
 <attribute name="VALUE" x="-231.14" y="-33.02" size="1.778" layer="96"/>
+</instance>
+<instance part="IC3" gate="G$1" x="119.38" y="-7.62" smashed="yes">
+<attribute name="VALUE" x="88.9" y="-86.36" size="1.778" layer="96"/>
+<attribute name="NAME" x="88.9" y="72.39" size="1.778" layer="95"/>
 </instance>
 </instances>
@@
 <pinref part="Q2" gate="G$1" pin="S"/>
 <pinref part="GND15" gate="1" pin="GND"/>
-<wire x1="-170.18" y1="-109.22" x2="-170.18" y2="-101.6" width="0.1524" layer="91"/>
+<pinref part="R3" gate="G$1" pin="2"/>
+<wire x1="-180.34" y1="-101.6" x2="-170.18" y2="-101.6" width="0.1524" layer="91"/>
+<junction x="-170.18" y="-101.6"/>
+</segment>
+<segment>
+<pinref part="Q3" gate="G$1" pin="S"/>
+<pinref part="R5" gate="G$1" pin="2"/>
+<wire x1="-170.18" y1="-127" x2="-180.34" y2="-127" width="0.1524" layer="91"/>
+<pinref part="GND16" gate="1" pin="GND"/>
+<junction x="-170.18" y="-127"/>
+</segment>
+<segment>
+<pinref part="Q4" gate="G$1" pin="S"/>
+<pinref part="R7" gate="G$1" pin="2"/>
+<wire x1="-170.18" y1="-152.4" x2="-180.34" y2="-152.4" width="0.1524" layer="91"/>
+<pinref part="GND17" gate="1" pin="GND"/>
+<junction x="-170.18" y="-152.4"/>
+</segment>
+<segment>
+<pinref part="Q5" gate="G$1" pin="S"/>
+<pinref part="R9" gate="G$1" pin="2"/>
+<wire x1="-170.18" y1="-177.8" x2="-180.34" y2="-177.8" width="0.1524" layer="91"/>
+<pinref part="GND18" gate="1" pin="GND"/>
+<junction x="-170.18" y="-177.8"/>
+</segment>
+<segment>
+<pinref part="Q6" gate="G$1" pin="S"/>
+<pinref part="R11" gate="G$1" pin="2"/>
+<wire x1="-170.18" y1="-203.2" x2="-180.34" y2="-203.2" width="0.1524" layer="91"/>
+<pinref part="GND19" gate="1" pin="GND"/>
+<junction x="-170.18" y="-203.2"/>
 </segment>
 </net>
@@
 </segment>
 </net>
-<net name="N$15" class="0">
-<segment>
-<pinref part="Q3" gate="G$1" pin="S"/>
-<pinref part="R5" gate="G$1" pin="2"/>
-<wire x1="-170.18" y1="-127" x2="-180.34" y2="-127" width="0.1524" layer="91"/>
-<pinref part="GND16" gate="1" pin="GND"/>
-<junction x="-170.18" y="-127"/>
-</segment>
-<segment>
-<pinref part="Q4" gate="G$1" pin="S"/>
-<pinref part="R7" gate="G$1" pin="2"/>
-<wire x1="-170.18" y1="-152.4" x2="-180.34" y2="-152.4" width="0.1524" layer="91"/>
-<pinref part="GND17" gate="1" pin="GND"/>
-<junction x="-170.18" y="-152.4"/>
-</segment>
-<segment>
-<pinref part="Q5" gate="G$1" pin="S"/>
-<pinref part="R9" gate="G$1" pin="2"/>
-<wire x1="-170.18" y1="-177.8" x2="-180.34" y2="-177.8" width="0.1524" layer="91"/>
-<pinref part="GND18" gate="1" pin="GND"/>
-<junction x="-170.18" y="-177.8"/>
-</segment>
-<segment>
-<pinref part="Q6" gate="G$1" pin="S"/>
-<pinref part="R11" gate="G$1" pin="2"/>
-<wire x1="-170.18" y1="-203.2" x2="-180.34" y2="-203.2" width="0.1524" layer="91"/>
-<pinref part="GND19" gate="1" pin="GND"/>
-<junction x="-170.18" y="-203.2"/>
-</segment>
-</net>
