File: extruderController/extruderControllerv02.brd (EAGLE design)
At the start: 93.7 x 68.6 mm, 73 parts, among them IC1 LM1117MPX-5.0, IC2 MAX3467CPA, IC4 ULN2003AD, J1 RJ45, Q2 PH7030L, Q3 PH7030L, Q4 PH7030L, Q5 PH7030L, Q6 PH7030L, U1 ATMEGA2560AU, X1 22-23-2081, X2 22-23-2081, X5 22-23-2051, X6 22-23-2041, X8 22-23-2031, X9 22-23-2031

Commit message: g
Parts:
- removed C15: 0.1uF, rcl:C0603
- removed J4: (no value), SparkFun-Connectors:2X8
- removed U1: ATMEGA2560AU, SparkFun-IC-Microcontroller:TQFP100
- added IC3: ATMEGA2561-16AU, atmel-2005:TQFP64
- added J6: (no value), SparkFun-Connectors:1X11
- J3, J5: device SparkFun-Connectors:2X8 -> SparkFun-Connectors:1X11
- moved C14 19.1 mm to (47.5, 41.7), turned to 270 degrees
- moved C7 15.5 mm to (26.4, 43.4), turned to 270 degrees
- moved C13 11.6 mm to (48.8, 34.8)
- moved J5 9.56 mm to (84.3, 32.5)
- moved J3 3.53 mm to (87.1, 32.5)
- moved R1 1.70 mm to (27.4, 46.2)
- moved C17 1.27 mm to (84.6, 19.3)
- moved H1 1.02 mm to (5.08, 64.5)
- moved C16 0.92 mm to (84.6, 28.7)
- moved H4 0.80 mm to (88.6, 64.3)
Connections:
- removed net N$37: IC4.2
- removed net PH0: IC2.2, U1.12
- removed net PH1: IC2.3, U1.13
- removed net PJ7: IC4.3, U1.79
- removed net PL0: R2.1, R3.1, U1.35
- removed net PL1: R4.1, R5.1, U1.36
- removed net PL2: R6.1, R7.1, U1.37
- removed net PL6: R8.1, R9.1, U1.41
- removed net PL7: R10.1, R11.1, U1.42
- new net N$46: J6.9
- new net N$47: J6.10
- new net N$48: J6.11
- new net PA4: IC3.47, J5.5
- new net PA5: IC3.46, J5.4
- new net PA6: IC3.45, J5.3
- new net PA7: IC3.44, J5.2
- new net PB0: IC3.10, J5.10
- new net PB4: IC3.14, J5.9
- new net PB5: IC3.15, J5.8
- new net PB6: IC3.16, J5.7
- new net PB7: IC3.17, J5.6
- new net PC4: IC3.39, J6.5
- new net PC5: IC3.40, J6.6
- new net PC6: IC3.41, J6.3
- new net PC7: IC3.42, J6.4
- new net PD2: IC3.27, U$1.7, U$2.7, U$3.7, U$4.7
- new net PD3: IC3.28, J5.11
- new net PD4: IC3.29, R2.1, R3.1
- new net PD5: IC3.30, U$1.5, U$2.5, U$3.5, U$4.5
- new net PD6: IC3.31, R4.1, R5.1
- new net PD7: IC3.32, R6.1, R7.1
- new net PE0: IC3.2, J5.1
- new net PE1: IC2.3, IC3.3
- new net PE2: IC2.2, IC3.4
- new net PE3: IC3.5, J3.2
- new net PE4: IC3.6, J3.1
- new net PE5: IC3.7, J6.2
- new net PE6: IC3.8, X9.2
- new net PE7: IC3.9, X8.2
- new net PF0: IC3.61, J3.9
- new net PF1: IC3.60, J3.8
- new net PF2: IC3.59, J3.7
- new net PF3: IC3.58, J3.6
- new net PF4: IC3.57, J3.5
- new net PF5: IC3.56, J3.4
- new net PF6: IC3.55, J3.3
- new net PF7: IC3.54, IC4.3
- new net PG0: IC3.33, R8.1, R9.1
- new net PG1: IC3.34, R10.1, R11.1
- new net PG2: IC3.43, J6.1
- new net PG3: IC3.18, J3.11
- new net PG4: IC3.19, J3.10
- new net PG5: IC3.1, IC4.2
- net +5V: now also IC3.21, IC3.52, IC3.62, IC3.63, IC3.64; no longer C15.1, U1.10, U1.100, U1.31, U1.61, U1.80, U1.98, U1.99
- net GND: now also IC3.22, IC3.53; no longer C15.2, U1.11, U1.32, U1.62, U1.81
- net N$19: now also IC3.23; no longer U1.33
- net N$20: now also IC3.24; no longer U1.34
- net PA0: now also IC3.51; no longer U1.78
- net PA1: now also IC3.50; no longer U1.77
- net PA2: now also IC3.49; no longer U1.76
- net PA3: now also IC3.48; no longer U1.75
- net PB1(SCK): now also IC3.11; no longer U$1.5, U$2.5, U$3.5, U$4.5, U1.20
- net PB2(MOSI): now also IC3.12; no longer U1.21
- net PB3(MISO): now also IC3.13; no longer U$1.7, U$2.7, U$3.7, U$4.7, U1.22
- net PC0: now also IC3.35; no longer U1.53
- net PC1: now also IC3.36; no longer U1.54
- net PC2: now also IC3.37; no longer U1.55
- net PC3: now also IC3.38; no longer U1.56
- net PD0: now also IC3.25, J6.7; no longer U1.43, X9.2
- net PD1: now also IC3.26, J6.8; no longer U1.44, X8.2
- net RESET: now also IC3.20; no longer U1.30
Routing:
- net +5V: track 164.7 -> 292.6 mm, vias 0 -> 7
- net PE6: track 0.00 -> 74.8 mm, vias 0 -> 2
- net PE7: track 0.00 -> 70.8 mm, vias 0 -> 2
- net PD0: track 73.5 -> 3.97 mm, vias 2 -> 1
- net PD1: track 67.7 -> 2.99 mm, vias 2 -> 1
- net PG2: track 0.00 -> 56.8 mm, vias 0 -> 1
- net PD2: track 0.00 -> 56.0 mm, vias 0 -> 2
- net PD5: track 0.00 -> 51.2 mm, vias 0 -> 8
- net PC4: track 0.00 -> 40.7 mm, vias 0 -> 1
- net PC5: track 0.00 -> 39.3 mm, vias 0 -> 1
- net PG5: track 0.00 -> 38.4 mm
- net PC6: track 0.00 -> 38.0 mm, vias 0 -> 1
- net PC7: track 0.00 -> 36.9 mm, vias 0 -> 1
- net PB3(MISO): track 46.1 -> 10.6 mm
- net PB1(SCK): track 45.9 -> 11.7 mm, vias 6 -> 0
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Other:
- board size 93.7 x 68.6 mm -> 93.7 x 69.3 mm
