File: extruderController/extruderControllerv02.brd (EAGLE design)
At the start: 93.7 x 69.3 mm, 72 parts, among them IC1 LM1117MPX-5.0, IC2 MAX3467CPA, IC3 ATMEGA2561-16AU, IC4 ULN2003AD, J1 RJ45, Q2 PH7030L, Q3 PH7030L, Q4 PH7030L, Q5 PH7030L, Q6 PH7030L, X1 22-23-2081, X2 22-23-2081, X3 22-23-2101, X6 22-23-2041, X8 22-23-2031, X9 22-23-2031

Commit message: k
Parts:
- R1: value (none) -> 10k
- R12, R13: value (none) -> 120
- R18: value (none) -> 330
- moved X3 9.14 mm to (4.06, 33.3)
- moved D5 8.57 mm to (11.7, 30.0)
- moved D2 7.64 mm to (11.4, 55.4)
- moved D3 7.64 mm to (11.4, 46.7)
- moved D4 7.64 mm to (11.4, 38.1)
- moved C3 7.33 mm to (30.7, 57.7), turned to 90 degrees
- moved D6 7.27 mm to (11.9, 20.1)
- moved C4 6.75 mm to (28.4, 57.7), turned to 90 degrees
- moved C7 5.24 mm to (29.7, 47.5), turned to 180 degrees
- moved R1 5.24 mm to (31.5, 49.5)
- moved R11 4.06 mm to (26.7, 17.0)
- moved R10 3.82 mm to (25.4, 20.1)
- moved R2 3.09 mm to (24.6, 55.1)
- moved R4 2.90 mm to (24.4, 46.2)
- moved R8 2.81 mm to (24.4, 29.2)
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Connections:
- net GND: now also Q2.2, Q2.3, Q3.2, Q3.3, Q4.2, Q4.3, Q5.2, Q5.3, Q6.2, Q6.3
Routing:
- net N$22: track 28.5 -> 0.00 mm, vias 0 -> 42
- net N$25: track 26.2 -> 0.00 mm, vias 0 -> 42
- net N$28: track 22.2 -> 0.27 mm, vias 0 -> 42
- net N$31: track 19.2 -> 0.00 mm, vias 0 -> 1
- net N$34: track 18.8 -> 0.24 mm, vias 0 -> 1
- net GND: track 60.8 -> 71.8 mm, vias 35 -> 71
- net +12V: track 12.5 -> 22.4 mm, vias 5 -> 3
- net N$19: track 21.8 -> 28.6 mm
- net N$20: track 26.3 -> 22.7 mm
- net PG0: track 12.7 -> 9.45 mm
- net N$32: track 2.10 -> 4.96 mm
- net +5V: track 368.6 -> 365.8 mm
- net PD7: track 11.7 -> 8.94 mm
- net N$2: track 2.35 -> 4.20 mm
- net N$29: track 2.35 -> 4.05 mm
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- added copper zone on layer 1, net N$22
- added copper zone on layer 16, net N$22
- added copper zone on layer 1, net N$25
- added copper zone on layer 16, net N$25
- added copper zone on layer 1, net N$28
- added copper zone on layer 16, net N$28
- added copper zone on layer 1, net N$31
- added copper zone on layer 16, net N$31
- added copper zone on layer 1, net N$34
- added copper zone on layer 16, net N$34
Other:
- board text added: "+12V"
- board text added: "+5V"
- board text added: "I/O"
- board text added: "ISP"
- board text added: "MISO"
- board text added: "MOSI"
- board text added: "RESET"
- board text added: "RS485"
- board text added: "SCK"
- board text added: "Screw rotation"
- board text added: "v1"
- board text removed: "Screw RPM"
- board text removed: "v1p2"

Commit message: c
Parts:
- added J4: (no value), SparkFun-Connectors:SCREWTERMINAL-3.5MM-2
- R10, R2, R4, R6, R8: value (none) -> 10
- R11, R3, R5, R7, R9: value (none) -> 100k
- moved C3 1.70 mm to (32.3, 58.4)
- moved C4 1.48 mm to (29.7, 58.4)
- moved IC1 1.48 mm to (36.3, 62.2)
- moved R11 0.76 mm to (25.9, 17.0)
- moved C16 0.51 mm to (84.6, 29.5)
- moved C13 0.25 mm to (48.8, 34.8)
Connections:
- net +12V: now also J4.1
- net GND: now also J4.2
Routing:
- net +12V: track 22.4 -> 35.1 mm, vias 3 -> 5
- net PG1: track 16.3 -> 18.1 mm
- net N$19: track 28.6 -> 26.9 mm
- net N$18: track 16.3 -> 17.6 mm
- net PC0: track 11.9 -> 10.6 mm
- net GND: track 71.8 -> 72.8 mm, vias 71 -> 104
- net +5V: track 365.8 -> 364.8 mm
- net PD4: track 24.4 -> 23.7 mm
- net N$34: vias 1 -> 42

Commit message: c
Parts:
- removed R12: 120, rcl:R1210
- moved R13 0.25 mm to (63.8, 52.1)
Connections:
- removed net N$35: IC2.5, J1.2, R12.2
- new net N$45: IC2.6, J1.4
- net GND: now also J1.2, J1.6; no longer J1.5, J1.7
- net N$27: now also J1.8; no longer J1.6
- net N$33: now also IC2.5, J1.5; no longer IC2.6, J1.4, R12.1
- net N$36: now also J1.7; no longer J1.8
Routing:
- net N$35: track 19.5 -> 0.00 mm
- net N$45: track 0.00 -> 15.1 mm
- net N$33: track 16.1 -> 29.5 mm
- net N$36: track 8.96 -> 14.5 mm
- net N$27: track 12.4 -> 15.1 mm
- net N$14: track 26.7 -> 24.6 mm
- net N$7: track 28.9 -> 27.3 mm
- net N$5: track 25.5 -> 23.9 mm
- net N$13: track 23.2 -> 21.5 mm
- net N$6: track 30.0 -> 28.5 mm
- net N$4: track 26.5 -> 25.2 mm
- net N$8: track 32.9 -> 31.7 mm
- net N$12: track 19.8 -> 18.6 mm
- net N$9: track 31.5 -> 30.5 mm
- net PE6: track 73.0 -> 72.1 mm
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
Commit message: f
Parts:
- added J8: 615016137621, SamacSys_Parts:WR-MJ
Changed lines of the file:
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@@
 <?xml version="1.0" encoding="utf-8"?>
 <!DOCTYPE eagle SYSTEM "eagle.dtd">
-<eagle version="9.3.1">
+<eagle version="9.2.2">
 <drawing>
 <settings>
@@
 <attribute name="VALUE" x="3.048" y="51.562" size="0.6096" layer="27" font="vector" ratio="20" rot="R90"/>
 </element>
+<element name="J8" library="SamacSys_Parts" package="WR-MJ" value="615016137621" x="64.262" y="66.802" smashed="yes" rot="R180">
+<attribute name="DESCRIPTION" value="Wurth Elektronik Female Cat5e RJ45 Connector, Shielded, Right Angle, PCB Mount Mount," x="64.262" y="66.802" size="1.778" layer="27" rot="R180" display="off"/>
+<attribute name="HEIGHT" value="mm" x="64.262" y="66.802" size="1.778" layer="27" rot="R180" display="off"/>
+<attribute name="MANUFACTURER_NAME" value="Wurth Elektronik" x="64.262" y="66.802" size="1.778" layer="27" rot="R180" display="off"/>
+<attribute name="MANUFACTURER_PART_NUMBER" value="615016137621" x="64.262" y="66.802" size="1.778" layer="27" rot="R180" display="off"/>
+<attribute name="MOUSER_PART_NUMBER" value="710-615016137621" x="64.262" y="66.802" size="1.778" layer="27" rot="R180" display="off"/>
+<attribute name="MOUSER_PRICE-STOCK" value="https://www.mouser.com/Search/Refine.aspx?Keyword=710-615016137621" x="64.262" y="66.802" size="1.778" layer="27" rot="R180" display="off"/>
+<attribute name="NAME" x="64.606" y="62.194" size="1.27" layer="25" rot="R180" align="center"/>
+<attribute name="VALUE" x="64.606" y="62.194" size="1.27" layer="27" rot="R180" align="center"/>
+</element>
 </elements>
