File: extruderController/extruderControllerv02.sch (EAGLE design)
At the start: 73 parts, among them IC1 LM1117MPX-5.0, IC2 MAX3467CPA, IC4 ULN2003AD, J1 RJ45, Q2 PH7030L, Q3 PH7030L, Q4 PH7030L, Q5 PH7030L, Q6 PH7030L, U1 ATMEGA2560AU, X1 22-23-2081, X2 22-23-2081, X5 22-23-2051, X6 22-23-2041, X8 22-23-2031, X9 22-23-2031

Commit message: g
Parts:
- removed C15: 0.1uF, rcl:C-EUC0603
- removed J4: (no value), SparkFun-Connectors:CONN_08X2
- removed U1: ATMEGA2560AU, SparkFun-IC-Microcontroller:ATMEGA2560AU
- added IC3: ATMEGA2561-16AU, atmel-2005:ATMEGA2561-16AU
- added J6: (no value), SparkFun-Connectors:CONN_11
- J3, J5: device SparkFun-Connectors:CONN_08X2 -> SparkFun-Connectors:CONN_11
Connections:
- removed net N$15: Q3.S, Q4.S, Q5.S, Q6.S, R11.2, R5.2, R7.2, R9.2
- removed net N$37: IC4.I2
- removed net PH0: IC2.RO, U1.PH0(RXD2)
- removed net PH1: IC2.DI, U1.PH1(TXD2)
- removed net PJ7: IC4.I3, U1.PJ7
- removed net PL0: R2.1, R3.1, U1.PL0(ICP4)
- removed net PL1: R4.1, R5.1, U1.PL1(ICP5)
- removed net PL2: R6.1, R7.1, U1.PL2(T5)
- removed net PL6: R8.1, R9.1, U1.PL6
- removed net PL7: R10.1, R11.1, U1.PL7
- new net N$46: J6.9
- new net N$47: J6.10
- new net N$48: J6.11
- new net PA4: IC3.(AD4)PA4, J5.5
- new net PA5: IC3.(AD5)PA5, J5.4
- new net PA6: IC3.(AD6)PA6, J5.3
- new net PA7: IC3.(AD7)PA7, J5.2
- new net PB0: IC3.(SS/PCINT0)PB0, J5.10
- new net PB4: IC3.(OC2A/PCINT4)PB4, J5.9
- new net PB5: IC3.(OC1A/PCINT5)PB5, J5.8
- new net PB6: IC3.(OC1B/PCINT6)PB6, J5.7
- new net PB7: IC3.(OC0A/OC1C/PCINT7)PB7, J5.6
- new net PC4: IC3.(A12)PC4, J6.5
- new net PC5: IC3.(A13)PC5, J6.6
- new net PC6: IC3.(A14)PC6, J6.3
- new net PC7: IC3.(A15)PC7, J6.4
- new net PD2: IC3.(RXD1/INT2)PD2, U$1.MISO, U$2.MISO, U$3.MISO, U$4.MISO
- new net PD3: IC3.(TXD1/INT3)PD3, J5.11
- new net PD4: IC3.(ICP1)PD4, R2.1, R3.1
- new net PD5: IC3.(XCK1)PD5, U$1.SCK, U$2.SCK, U$3.SCK, U$4.SCK
- new net PD6: IC3.(T1)PD6, R4.1, R5.1
- new net PD7: IC3.(T0)PD7, R6.1, R7.1
- new net PE0: IC3.(RXD0/PCIN8/PDI)PE0, J5.1
- new net PE1: IC2.DI, IC3.(TXD0/PDO)PE1
- new net PE2: IC2.RO, IC3.(XCK0/AIN0)PE2
- new net PE3: IC3.(OC3A/AIN1)PE3, J3.2
- new net PE4: IC3.(OC3B/INT4)PE4, J3.1
- new net PE5: IC3.(OC3C/INT5)PE5, J6.2
- new net PE6: IC3.(T3/INT6)PE6, X9-2.S
- new net PE7: IC3.(CLKO/ICP3/INT7)PE7, X8-2.S
- new net PF0: IC3.(ADC0)PF0, J3.9
- new net PF1: IC3.(ADC1)PF1, J3.8
- new net PF2: IC3.(ADC2)PF2, J3.7
- new net PF3: IC3.(ADC3)PF3, J3.6
- new net PF4: IC3.(ADC4/TCK)PF4, J3.5
- new net PF5: IC3.(ADC5/TMS)PF5, J3.4
- new net PF6: IC3.(ADC6/TDO)PF6, J3.3
- new net PF7: IC3.(ADC7/TDI)PF7, IC4.I3
- new net PG0: IC3.(WR)PG0, R8.1, R9.1
- new net PG1: IC3.(RD)PG1, R10.1, R11.1
- new net PG2: IC3.(ALE)PG2, J6.1
- new net PG3: IC3.(TOSC2)PG3, J3.11
- new net PG4: IC3.(TOSC1)PG4, J3.10
- new net PG5: IC3.(OC0B)PG5, IC4.I2
- net +5V: now also IC3.AGND, IC3.AREF, IC3.AVCC, IC3.VCC, IC3.VCC1; no longer C15.1, U1.AGND, U1.AREF, U1.AVCC, U1.VCC, U1.VCC1, U1.VCC2, U1.VCC3
- net GND: now also IC3.GND, IC3.GND1, Q3.S, Q4.S, Q5.S, Q6.S, R11.2, R3.2, R5.2, R7.2, R9.2; no longer C15.2, U1.GND, U1.GND1, U1.GND2, U1.GND3
- net N$19: now also IC3.XTAL2; no longer U1.XTAL2
- net N$20: now also IC3.XTAL1; no longer U1.XTAL1
- net PA0: now also IC3.(AD0)PA0; no longer U1.(AD0)PA0
- net PA1: now also IC3.(AD1)PA1; no longer U1.(AD1)PA1
- net PA2: now also IC3.(AD2)PA2; no longer U1.(AD2)PA2
- net PA3: now also IC3.(AD3)PA3; no longer U1.(AD3)PA3
- net PB1(SCK): now also IC3.(SCK/PCINT1)PB1; no longer U$1.SCK, U$2.SCK, U$3.SCK, U$4.SCK, U1.(SCK/PCINT1)PB1
- net PB2(MOSI): now also IC3.(MOSI/PCINT2)PB2; no longer U1.(MOSI/PCINT2)PB2
- net PB3(MISO): now also IC3.(MISO/PCINT3)PB3; no longer U$1.MISO, U$2.MISO, U$3.MISO, U$4.MISO, U1.(MISO/PCINT3)PB3
- net PC0: now also IC3.(A8)PC0; no longer U1.(A8)PC0
- net PC1: now also IC3.(A9)PC1; no longer U1.(A9)PC1
- net PC2: now also IC3.(A10)PC2; no longer U1.(A10)PC2
- net PC3: now also IC3.(A11)PC3; no longer U1.(A11)PC3
- net PD0: now also IC3.(SCL/INT0)PD0, J6.7; no longer U1.(SCL/INT0)PD0, X9-2.S
- net PD1: now also IC3.(SDA/INT1)PD1, J6.8; no longer U1.(SDA/INT1)PD1, X8-2.S
- net RESET: now also IC3.RESET; no longer U1.RESET
Other:
- moved on the sheet: C12, C13, C14, C3, C4, C7, IC2, J1, Q1, R1, R12, R13
