File: extruderController/extruderControllerv02.sch (EAGLE design)
At the start: 72 parts, among them IC1 LM1117MPX-5.0, IC2 MAX3467CPA, IC3 ATMEGA2561-16AU, IC4 ULN2003AD, J1 RJ45, Q2 PH7030L, Q3 PH7030L, Q4 PH7030L, Q5 PH7030L, Q6 PH7030L, X1 22-23-2081, X2 22-23-2081, X3 22-23-2101, X6 22-23-2041, X8 22-23-2031, X9 22-23-2031

Commit message: k
Parts:
- R1: value (none) -> 10k
- R12, R13: value (none) -> 120
- R18: value (none) -> 330
Connections:
- net GND: now also Q2.S@1, Q2.S@2, Q3.S@1, Q3.S@2, Q4.S@1, Q4.S@2, Q5.S@1, Q5.S@2, Q6.S@1, Q6.S@2
Changed lines of the file:
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@@
 <?xml version="1.0" encoding="utf-8"?>
 <!DOCTYPE eagle SYSTEM "eagle.dtd">
-<eagle version="9.2.2">
+<eagle version="9.3.1">
 <drawing>
 <settings>
@@
 <part name="C4" library="rcl" library_urn="urn:adsk.eagle:library:334" deviceset="C-EU" device="C0603" package3d_urn="urn:adsk.eagle:package:23616/2"/>
 <part name="GND13" library="supply1" library_urn="urn:adsk.eagle:library:371" deviceset="GND" device=""/>
-<part name="R1" library="rcl" library_urn="urn:adsk.eagle:library:334" deviceset="R-EU_" device="R0805" package3d_urn="urn:adsk.eagle:package:23553/2"/>
+<part name="R1" library="rcl" library_urn="urn:adsk.eagle:library:334" deviceset="R-EU_" device="R0805" package3d_urn="urn:adsk.eagle:package:23553/2" value="10k"/>
 <part name="P+11" library="supply1" library_urn="urn:adsk.eagle:library:371" deviceset="+5V" device=""/>
 <part name="C7" library="rcl" library_urn="urn:adsk.eagle:library:334" deviceset="C-EU" device="C0603" package3d_urn="urn:adsk.eagle:package:23616/2" value="0.1uF"/>
@@
 <part name="GND21" library="supply1" library_urn="urn:adsk.eagle:library:371" deviceset="GND" device=""/>
 <part name="C12" library="rcl" library_urn="urn:adsk.eagle:library:334" deviceset="C-EU" device="C0603" package3d_urn="urn:adsk.eagle:package:23616/2" value="0.1uF"/>
-<part name="R12" library="rcl" library_urn="urn:adsk.eagle:library:334" deviceset="R-EU_" device="R1210" package3d_urn="urn:adsk.eagle:package:23554/2"/>
-<part name="R13" library="rcl" library_urn="urn:adsk.eagle:library:334" deviceset="R-EU_" device="R1210" package3d_urn="urn:adsk.eagle:package:23554/2"/>
+<part name="R12" library="rcl" library_urn="urn:adsk.eagle:library:334" deviceset="R-EU_" device="R1210" package3d_urn="urn:adsk.eagle:package:23554/2" value="120"/>
+<part name="R13" library="rcl" library_urn="urn:adsk.eagle:library:334" deviceset="R-EU_" device="R1210" package3d_urn="urn:adsk.eagle:package:23554/2" value="120"/>
 <part name="P+14" library="supply1" library_urn="urn:adsk.eagle:library:371" deviceset="+5V" device=""/>
 <part name="P+15" library="supply1" library_urn="urn:adsk.eagle:library:371" deviceset="+5V" device=""/>
@@
 <part name="GND8" library="supply1" library_urn="urn:adsk.eagle:library:371" deviceset="GND" device=""/>
 <part name="LED1" library="led" library_urn="urn:adsk.eagle:library:259" deviceset="LED" device="SML1206" package3d_urn="urn:adsk.eagle:package:15829/1"/>
-<part name="R18" library="rcl" library_urn="urn:adsk.eagle:library:334" deviceset="R-EU_" device="R0805" package3d_urn="urn:adsk.eagle:package:23553/2"/>
+<part name="R18" library="rcl" library_urn="urn:adsk.eagle:library:334" deviceset="R-EU_" device="R0805" package3d_urn="urn:adsk.eagle:package:23553/2" value="330"/>
 <part name="GND25" library="supply1" library_urn="urn:adsk.eagle:library:371" deviceset="GND" device=""/>
 <part name="P+16" library="supply1" library_urn="urn:adsk.eagle:library:371" deviceset="+5V" device=""/>
@@
 <part name="IC3" library="atmel-2005" deviceset="ATMEGA2561*" device="AU" technology="-16"/>
 <part name="C14" library="rcl" library_urn="urn:adsk.eagle:library:334" deviceset="C-EU" device="C0603" package3d_urn="urn:adsk.eagle:package:23616/2" value="0.1uF"/>
-<part name="P+28" library="supply1" library_urn="urn:adsk.eagle:library:371" deviceset="+5V" device=""/>
-<part name="GND31" library="supply1" library_urn="urn:adsk.eagle:library:371" deviceset="GND" device=""/>
 <part name="J3" library="SparkFun-Connectors" deviceset="CONN_11" device=""/>
 <part name="J5" library="SparkFun-Connectors" deviceset="CONN_11" device=""/>
@@
 <instance part="D2" gate="G$1" x="-175.26" y="-86.36" smashed="yes" rot="R180">
 <attribute name="NAME" x="-172.72" y="-88.392" size="1.778" layer="95" font="vector" rot="R180"/>
-<attribute name="VALUE" x="-172.72" y="-81.788" size="1.778" layer="96" font="vector" rot="R180" align="top-left"/>
+<attribute name="VALUE" x="-172.72" y="-84.328" size="1.778" layer="96" font="vector" rot="R180" align="top-left"/>
 </instance>
 <instance part="P+22" gate="1" x="-182.88" y="-86.36" smashed="yes" rot="R90">
@@
 <instance part="D3" gate="G$1" x="-175.26" y="-111.76" smashed="yes" rot="R180">
 <attribute name="NAME" x="-172.72" y="-113.792" size="1.778" layer="95" font="vector" rot="R180"/>
-<attribute name="VALUE" x="-172.72" y="-107.188" size="1.778" layer="96" font="vector" rot="R180" align="top-left"/>
+<attribute name="VALUE" x="-172.72" y="-109.728" size="1.778" layer="96" font="vector" rot="R180" align="top-left"/>
 </instance>
 <instance part="D4" gate="G$1" x="-175.26" y="-137.16" smashed="yes" rot="R180">
 <attribute name="NAME" x="-172.72" y="-139.192" size="1.778" layer="95" font="vector" rot="R180"/>
-<attribute name="VALUE" x="-172.72" y="-132.588" size="1.778" layer="96" font="vector" rot="R180" align="top-left"/>
+<attribute name="VALUE" x="-172.72" y="-135.128" size="1.778" layer="96" font="vector" rot="R180" align="top-left"/>
 </instance>
 <instance part="D5" gate="G$1" x="-175.26" y="-162.56" smashed="yes" rot="R180">
@@
 <attribute name="NAME" x="-69.596" y="94.361" size="1.778" layer="95"/>
 <attribute name="VALUE" x="-69.596" y="89.281" size="1.778" layer="96"/>
-</instance>
-<instance part="P+28" gate="1" x="96.52" y="12.7" smashed="yes" rot="R90">
-<attribute name="VALUE" x="101.6" y="10.16" size="1.778" layer="96" rot="R180"/>
-</instance>
-<instance part="GND31" gate="1" x="114.3" y="10.16" smashed="yes">
-<attribute name="VALUE" x="111.76" y="7.62" size="1.778" layer="96"/>
 </instance>
 <instance part="J3" gate="G$1" x="121.92" y="63.5" smashed="yes">
@@
 <wire x1="-180.34" y1="-101.6" x2="-170.18" y2="-101.6" width="0.1524" layer="91"/>
 <junction x="-170.18" y="-101.6"/>
+<pinref part="Q2" gate="G$1" pin="S@2"/>
+<pinref part="Q2" gate="G$1" pin="S@1"/>
+<wire x1="-170.18" y1="-99.06" x2="-170.18" y2="-96.52" width="0.1524" layer="91"/>
+<wire x1="-170.18" y1="-101.6" x2="-170.18" y2="-99.06" width="0.1524" layer="91"/>
+<junction x="-170.18" y="-99.06"/>
 </segment>
 <segment>
@@
 <pinref part="GND16" gate="1" pin="GND"/>
 <junction x="-170.18" y="-127"/>
+<pinref part="Q3" gate="G$1" pin="S@1"/>
+<wire x1="-170.18" y1="-127" x2="-170.18" y2="-124.46" width="0.1524" layer="91"/>
+<pinref part="Q3" gate="G$1" pin="S@2"/>
+<wire x1="-170.18" y1="-124.46" x2="-170.18" y2="-121.92" width="0.1524" layer="91"/>
+<junction x="-170.18" y="-124.46"/>
 </segment>
 <segment>
@@
 <pinref part="GND17" gate="1" pin="GND"/>
 <junction x="-170.18" y="-152.4"/>
+<pinref part="Q4" gate="G$1" pin="S@1"/>
+<wire x1="-170.18" y1="-152.4" x2="-170.18" y2="-149.86" width="0.1524" layer="91"/>
+<pinref part="Q4" gate="G$1" pin="S@2"/>
+<wire x1="-170.18" y1="-149.86" x2="-170.18" y2="-147.32" width="0.1524" layer="91"/>
+<junction x="-170.18" y="-149.86"/>
 </segment>
 <segment>
@@
 <pinref part="GND18" gate="1" pin="GND"/>
 <junction x="-170.18" y="-177.8"/>
+<pinref part="Q5" gate="G$1" pin="S@1"/>
+<wire x1="-170.18" y1="-177.8" x2="-170.18" y2="-175.26" width="0.1524" layer="91"/>
+<pinref part="Q5" gate="G$1" pin="S@2"/>
+<wire x1="-170.18" y1="-175.26" x2="-170.18" y2="-172.72" width="0.1524" layer="91"/>
+<junction x="-170.18" y="-175.26"/>
 </segment>
 <segment>
@@
 <pinref part="GND19" gate="1" pin="GND"/>
 <junction x="-170.18" y="-203.2"/>
-</segment>
-<segment>
+<pinref part="Q6" gate="G$1" pin="S@1"/>
+<wire x1="-170.18" y1="-203.2" x2="-170.18" y2="-200.66" width="0.1524" layer="91"/>
+<pinref part="Q6" gate="G$1" pin="S@2"/>
+<wire x1="-170.18" y1="-200.66" x2="-170.18" y2="-198.12" width="0.1524" layer="91"/>
+<junction x="-170.18" y="-200.66"/>
+</segment>
+<segment>

Commit message: c
Parts:
- added J4: (no value), SparkFun-Connectors:CONN_023.5MM
- Q1: SPICEPREFIX (none) -> B
- R10, R2, R4, R6, R8: value (none) -> 10
- R11, R3, R5, R7, R9: value (none) -> 100k
Connections:
- net +12V: now also J4.1
- net GND: now also J4.2
Other:
- note added: "I/O"
- moved on the sheet: C1, C10, C11, C12, C16, C17, C18, C2, C5, C6, C8, C9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

Commit message: c
Parts:
- removed R12: 120, rcl:R-EU_R1210
Connections:
- removed net N$35: IC2.Y, J1.2, R12.2
- new net N$45: IC2.Z, J1.4
- net GND: now also J1.2, J1.6; no longer J1.5, J1.7
- net N$27: now also J1.8; no longer J1.6
- net N$33: now also IC2.Y, J1.5; no longer IC2.Z, J1.4, R12.1
- net N$36: now also J1.7; no longer J1.8
Changed lines of the file:
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@@
 <?xml version="1.0" encoding="utf-8"?>
 <!DOCTYPE eagle SYSTEM "eagle.dtd">
-<eagle version="9.2.2">
+<eagle version="9.3.1">
 <drawing>
 <settings>
@@
 <part name="GND21" library="supply1" library_urn="urn:adsk.eagle:library:371" deviceset="GND" device=""/>
 <part name="C12" library="rcl" library_urn="urn:adsk.eagle:library:334" deviceset="C-EU" device="C0603" package3d_urn="urn:adsk.eagle:package:23616/2" value="0.1uF"/>
-<part name="R12" library="rcl" library_urn="urn:adsk.eagle:library:334" deviceset="R-EU_" device="R1210" package3d_urn="urn:adsk.eagle:package:23554/2" value="120"/>
 <part name="R13" library="rcl" library_urn="urn:adsk.eagle:library:334" deviceset="R-EU_" device="R1210" package3d_urn="urn:adsk.eagle:package:23554/2" value="120"/>
 <part name="P+14" library="supply1" library_urn="urn:adsk.eagle:library:371" deviceset="+5V" device=""/>
@@
 <attribute name="VALUE" x="118.364" y="165.481" size="1.778" layer="96"/>
 </instance>
-<instance part="R12" gate="G$1" x="111.76" y="195.58" smashed="yes">
-<attribute name="NAME" x="107.95" y="197.0786" size="1.778" layer="95"/>
-<attribute name="VALUE" x="107.95" y="192.278" size="1.778" layer="96"/>
-</instance>
 <instance part="R13" gate="G$1" x="111.76" y="185.42" smashed="yes">
 <attribute name="NAME" x="107.95" y="186.9186" size="1.778" layer="95"/>
@@
 <attribute name="VALUE" x="114.3" y="160.02" size="1.778" layer="96"/>
 </instance>
-<instance part="GND24" gate="1" x="134.62" y="175.26" smashed="yes">
-<attribute name="VALUE" x="132.08" y="172.72" size="1.778" layer="96"/>
+<instance part="GND24" gate="1" x="127" y="175.26" smashed="yes">
+<attribute name="VALUE" x="124.46" y="172.72" size="1.778" layer="96"/>
 </instance>
 <instance part="X8" gate="-1" x="109.22" y="12.7" smashed="yes" rot="R180">
@@
 <pinref part="R18" gate="G$1" pin="1"/>
 <pinref part="GND25" gate="1" pin="GND"/>
-</segment>
-<segment>
-<pinref part="J1" gate="JP1" pin="1"/>
-<wire x1="137.16" y1="198.12" x2="134.62" y2="198.12" width="0.1524" layer="91"/>
-<wire x1="134.62" y1="198.12" x2="134.62" y2="193.04" width="0.1524" layer="91"/>
-<pinref part="J1" gate="JP1" pin="3"/>
-<wire x1="134.62" y1="193.04" x2="137.16" y2="193.04" width="0.1524" layer="91"/>
-<wire x1="134.62" y1="193.04" x2="134.62" y2="187.96" width="0.1524" layer="91"/>
-<junction x="134.62" y="193.04"/>
-<pinref part="J1" gate="JP1" pin="5"/>
-<wire x1="134.62" y1="187.96" x2="137.16" y2="187.96" width="0.1524" layer="91"/>
-<wire x1="134.62" y1="187.96" x2="134.62" y2="182.88" width="0.1524" layer="91"/>
-<junction x="134.62" y="187.96"/>
-<pinref part="J1" gate="JP1" pin="7"/>
-<wire x1="134.62" y1="182.88" x2="137.16" y2="182.88" width="0.1524" layer="91"/>
-<pinref part="GND24" gate="1" pin="GND"/>
-<wire x1="134.62" y1="182.88" x2="134.62" y2="177.8" width="0.1524" layer="91"/>
-<junction x="134.62" y="182.88"/>
 </segment>
 <segment>
@@
 <pinref part="GND31" gate="1" pin="GND"/>
 <wire x1="-93.98" y1="203.2" x2="-93.98" y2="205.74" width="0.1524" layer="91"/>
+</segment>
+<segment>
+<pinref part="J1" gate="JP1" pin="1"/>
+<pinref part="J1" gate="JP1" pin="2"/>
+<wire x1="137.16" y1="198.12" x2="137.16" y2="195.58" width="0.1524" layer="91"/>
+<pinref part="J1" gate="JP1" pin="3"/>
+<wire x1="137.16" y1="193.04" x2="137.16" y2="195.58" width="0.1524" layer="91"/>
+<junction x="137.16" y="195.58"/>
+<wire x1="137.16" y1="195.58" x2="127" y2="195.58" width="0.1524" layer="91"/>
+<wire x1="127" y1="195.58" x2="127" y2="185.42" width="0.1524" layer="91"/>
+<pinref part="J1" gate="JP1" pin="6"/>
+<wire x1="127" y1="185.42" x2="137.16" y2="185.42" width="0.1524" layer="91"/>
+<wire x1="127" y1="185.42" x2="127" y2="177.8" width="0.1524" layer="91"/>
+<junction x="127" y="185.42"/>
+<pinref part="GND24" gate="1" pin="GND"/>
 </segment>
 </net>
@@
 <wire x1="106.68" y1="182.88" x2="101.6" y2="182.88" width="0.1524" layer="91"/>
 <wire x1="106.68" y1="185.42" x2="106.68" y2="182.88" width="0.1524" layer="91"/>
-<pinref part="J1" gate="JP1" pin="6"/>
-<wire x1="137.16" y1="185.42" x2="119.38" y2="185.42" width="0.1524" layer="91"/>
-<wire x1="119.38" y1="185.42" x2="119.38" y2="182.88" width="0.1524" layer="91"/>
-<wire x1="119.38" y1="182.88" x2="106.68" y2="182.88" width="0.1524" layer="91"/>
+<pinref part="J1" gate="JP1" pin="8"/>
+<wire x1="137.16" y1="180.34" x2="106.68" y2="180.34" width="0.1524" layer="91"/>
+<wire x1="106.68" y1="180.34" x2="106.68" y2="182.88" width="0.1524" layer="91"/>
 <junction x="106.68" y="182.88"/>
-</segment>
-</net>
-<net name="N$33" class="0">
-<segment>
-<pinref part="IC2" gate="G$1" pin="Z"/>
-<wire x1="101.6" y1="193.04" x2="106.68" y2="193.04" width="0.1524" layer="91"/>
-<pinref part="R12" gate="G$1" pin="1"/>
-<wire x1="106.68" y1="195.58" x2="106.68" y2="193.04" width="0.1524" layer="91"/>
-<wire x1="106.68" y1="193.04" x2="132.08" y2="193.04" width="0.1524" layer="91"/>
-<junction x="106.68" y="193.04"/>
-<wire x1="132.08" y1="193.04" x2="132.08" y2="190.5" width="0.1524" layer="91"/>
-<pinref part="J1" gate="JP1" pin="4"/>
-<wire x1="132.08" y1="190.5" x2="137.16" y2="190.5" width="0.1524" layer="91"/>
-</segment>
-</net>
-<net name="N$35" class="0">
-<segment>
-<pinref part="IC2" gate="G$1" pin="Y"/>
-<wire x1="101.6" y1="198.12" x2="116.84" y2="198.12" width="0.1524" layer="91"/>
-<pinref part="R12" gate="G$1" pin="2"/>
-<wire x1="116.84" y1="195.58" x2="116.84" y2="198.12" width="0.1524" layer="91"/>
-<wire x1="116.84" y1="198.12" x2="132.08" y2="198.12" width="0.1524" layer="91"/>
-<wire x1="132.08" y1="198.12" x2="132.08" y2="195.58" width="0.1524" layer="91"/>
-<junction x="116.84" y="198.12"/>
-<pinref part="J1" gate="JP1" pin="2"/>
-<wire x1="132.08" y1="195.58" x2="137.16" y2="195.58" width="0.1524" layer="91"/>
 </segment>
 </net>
@@
 <pinref part="R13" gate="G$1" pin="2"/>
 <wire x1="116.84" y1="185.42" x2="116.84" y2="187.96" width="0.1524" layer="91"/>
-<wire x1="116.84" y1="187.96" x2="132.08" y2="187.96" width="0.1524" layer="91"/>
+<wire x1="116.84" y1="187.96" x2="129.54" y2="187.96" width="0.1524" layer="91"/>
 <junction x="116.84" y="187.96"/>
-<wire x1="132.08" y1="187.96" x2="132.08" y2="180.34" width="0.1524" layer="91"/>
-<pinref part="J1" gate="JP1" pin="8"/>
-<wire x1="132.08" y1="180.34" x2="137.16" y2="180.34" width="0.1524" layer="91"/>
+<wire x1="129.54" y1="187.96" x2="129.54" y2="182.88" width="0.1524" layer="91"/>
+<pinref part="J1" gate="JP1" pin="7"/>
+<wire x1="129.54" y1="182.88" x2="137.16" y2="182.88" width="0.1524" layer="91"/>
 </segment>
 </net>
@@
 </segment>
 </net>
+<net name="N$45" class="0">
+<segment>
+<pinref part="IC2" gate="G$1" pin="Z"/>
+<wire x1="101.6" y1="193.04" x2="134.62" y2="193.04" width="0.1524" layer="91"/>
+<pinref part="J1" gate="JP1" pin="4"/>
+<wire x1="137.16" y1="190.5" x2="134.62" y2="190.5" width="0.1524" layer="91"/>
+<wire x1="134.62" y1="190.5" x2="134.62" y2="193.04" width="0.1524" layer="91"/>
+</segment>
+</net>
+<net name="N$33" class="0">
+<segment>
+<pinref part="J1" gate="JP1" pin="5"/>
+<wire x1="137.16" y1="187.96" x2="132.08" y2="187.96" width="0.1524" layer="91"/>
+<pinref part="IC2" gate="G$1" pin="Y"/>
+<wire x1="101.6" y1="198.12" x2="132.08" y2="198.12" width="0.1524" layer="91"/>
+<wire x1="132.08" y1="187.96" x2="132.08" y2="198.12" width="0.1524" layer="91"/>
+</segment>
+</net>

Commit message: f
Parts:
- added J8: 615016137621, SamacSys_Parts:615016137621
Changed lines of the file:
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@@
 <?xml version="1.0" encoding="utf-8"?>
 <!DOCTYPE eagle SYSTEM "eagle.dtd">
-<eagle version="9.3.1">
+<eagle version="9.2.2">
 <drawing>
 <settings>
@@
 <part name="P+28" library="supply1" library_urn="urn:adsk.eagle:library:371" deviceset="+12V" device=""/>
 <part name="GND31" library="supply1" library_urn="urn:adsk.eagle:library:371" deviceset="GND" device=""/>
+<part name="J8" library="SamacSys_Parts" deviceset="615016137621" device=""/>
 </parts>
 <sheets>
@@
 <text x="-243.84" y="210.82" size="5.08" layer="91">Main stepper control output</text>
 <text x="66.04" y="76.2" size="5.08" layer="91">Hall effect sensor (rpm) input</text>
-<text x="66.04" y="218.44" size="5.08" layer="91">RS485 communication</text>
+<text x="66.04" y="256.54" size="5.08" layer="91">RS485 communication</text>
 <text x="66.04" y="27.94" size="5.08" layer="91">Hopper level sensor input</text>
 <wire x1="-109.22" y1="167.64" x2="55.88" y2="167.64" width="0.254" layer="95" style="longdash"/>
@@
 <instance part="GND31" gate="1" x="-93.98" y="200.66" smashed="yes">
 <attribute name="VALUE" x="-96.52" y="198.12" size="1.778" layer="96"/>
+</instance>
+<instance part="J8" gate="G$1" x="119.38" y="233.68" smashed="yes">
+<attribute name="NAME" x="138.43" y="241.3" size="1.778" layer="95" align="center-left"/>
+<attribute name="VALUE" x="138.43" y="238.76" size="1.778" layer="96" align="center-left"/>
 </instance>
 </instances>
@@
 <net name="N$42" class="0">
 <segment>
-<wire x1="63.5" y1="226.06" x2="63.5" y2="154.94" width="0.1524" layer="91" style="longdash"/>
+<wire x1="63.5" y1="264.16" x2="63.5" y2="154.94" width="0.1524" layer="91" style="longdash"/>
 <wire x1="63.5" y1="154.94" x2="170.18" y2="154.94" width="0.1524" layer="91" style="longdash"/>
-<wire x1="170.18" y1="154.94" x2="170.18" y2="226.06" width="0.1524" layer="91" style="longdash"/>
-<wire x1="170.18" y1="226.06" x2="63.5" y2="226.06" width="0.1524" layer="91" style="longdash"/>
-</segment>
-</net>
+<wire x1="170.18" y1="154.94" x2="170.18" y2="264.16" width="0.1524" layer="91" style="longdash"/>
+<wire x1="170.18" y1="264.16" x2="63.5" y2="264.16" width="0.1524" layer="91" style="longdash"/>
+</segment>
+</net>
