File: extruderController/interfaceModule.sch (EAGLE design)
At the start: 4 parts, among them IC2 MAX3467CPA, J1 RJ45, J2 USB_B_PTH

Commit message: f
Connections:
- new net DA: IC2.A, J1.1
- new net DB: IC2.B, J1.2
- new net DY: IC2.Y, J1.7
- new net DZ: IC2.Z, J1.8
Changed lines of the file:
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@@
 <?xml version="1.0" encoding="utf-8"?>
 <!DOCTYPE eagle SYSTEM "eagle.dtd">
-<eagle version="9.3.1">
+<eagle version="9.2.2">
 <drawing>
 <settings>
@@
 </segment>
 </net>
+<net name="DB" class="0">
+<segment>
+<pinref part="IC2" gate="G$1" pin="B"/>
+<wire x1="-106.68" y1="101.6" x2="-114.3" y2="101.6" width="0.1524" layer="91"/>
+<label x="-114.3" y="101.6" size="1.778" layer="95"/>
+</segment>
+<segment>
+<pinref part="J1" gate="JP1" pin="2"/>
+<wire x1="-139.7" y1="88.9" x2="-132.08" y2="88.9" width="0.1524" layer="91"/>
+<label x="-137.16" y="88.9" size="1.778" layer="95"/>
+</segment>
+</net>
+<net name="DA" class="0">
+<segment>
+<pinref part="IC2" gate="G$1" pin="A"/>
+<wire x1="-106.68" y1="96.52" x2="-114.3" y2="96.52" width="0.1524" layer="91"/>
+<label x="-114.3" y="96.52" size="1.778" layer="95"/>
+</segment>
+<segment>
+<pinref part="J1" gate="JP1" pin="1"/>
+<wire x1="-139.7" y1="86.36" x2="-132.08" y2="86.36" width="0.1524" layer="91"/>
+<label x="-137.16" y="86.36" size="1.778" layer="95"/>
+</segment>
+</net>
+<net name="DZ" class="0">
+<segment>
+<pinref part="IC2" gate="G$1" pin="Z"/>
+<wire x1="-106.68" y1="91.44" x2="-114.3" y2="91.44" width="0.1524" layer="91"/>
+<label x="-114.3" y="91.44" size="1.778" layer="95"/>
+</segment>
+<segment>
+<pinref part="J1" gate="JP1" pin="8"/>
+<wire x1="-139.7" y1="104.14" x2="-132.08" y2="104.14" width="0.1524" layer="91"/>
+<label x="-137.16" y="104.14" size="1.778" layer="95"/>
+</segment>
+</net>
+<net name="DY" class="0">
+<segment>
+<pinref part="IC2" gate="G$1" pin="Y"/>
+<wire x1="-106.68" y1="86.36" x2="-114.3" y2="86.36" width="0.1524" layer="91"/>
+<label x="-114.3" y="86.36" size="1.778" layer="95"/>
+</segment>
+<segment>
+<pinref part="J1" gate="JP1" pin="7"/>
+<wire x1="-139.7" y1="101.6" x2="-132.08" y2="101.6" width="0.1524" layer="91"/>
+<label x="-137.16" y="101.6" size="1.778" layer="95"/>
+</segment>
+</net>

Commit message: d
Parts:
- removed IC2: MAX3467CPA, maxim:MAX3467CPA
- added C1, C2, C4: 0.1uF, rcl:C-EUC0603
- added C3: 33nF, rcl:C-EUC0603
- added IC3: ISO3086DW, SamacSys_Parts:ISO3086DW
- added LED1, LED2: (no value), led:LEDSML1206
- added LSP1, LSP2: SE14, solpad:SE14
- added PS1: IRM-03-5, SamacSys_Parts:IRM-03-5
- added R1, R2: 120, rcl:R-EU_R1210
- added R5: 470, rcl:R-EU_R0805
- added R6, R7: 27, rcl:R-EU_R0805
- added R8, R9: 220, rcl:R-EU_R0805
Connections:
- new net AGND: C1.2, IC3.GND_2, IC3.GND_2_2, IC3.GND_2_3, J1.3, J1.4, J1.5, J1.6, PS1.-V
- new net N$1: LSP1.MP, PS1.AC/L
- new net N$10: LED1.C, R8.2
- new net N$2: LSP2.MP, PS1.AC/N
- new net N$3: IC1.USBDM, R6.2
- new net N$4: IC1.AVCC, R5.1
- new net N$5: IC1.USBDP, R7.2
- new net N$6: C3.2, IC1.3V3OUT
- new net N$7: IC1.TXLED, R8.1
- new net N$8: IC1.RXLED, R9.1
- new net N$9: LED2.C, R9.2
- new net VCC/2: C1.1, IC3.VCC2, PS1.+V
- net +5V: now also C2.1, C4.1, IC1.RESET, IC1.VCC1, IC1.VCC2, IC1.VCIO, IC3.VCC1, LED1.A, LED2.A, R5.2
- net DA: now also IC3.A, R1.2; no longer IC2.A
- net DB: now also IC3.B, R1.1; no longer IC2.B
- net DY: now also IC3.Y, R2.1; no longer IC2.Y
- net DZ: now also IC3.Z, R2.2; no longer IC2.Z
- net GND: now also C2.2, C3.1, C4.2, IC1.GND1, IC1.GND2, IC1.PWRCTL, IC3.GND_1, IC3.GND_1_2, IC3.GND_1_3
- net RXD: now also IC3.R; no longer IC2.RO
- net TXD: now also IC3.D; no longer IC2.DI
- net USBD+: now also R7.1
- net USBD-: now also R6.1
Other:
- moved on the sheet: IC1

Commit message: v
Parts:
- added D1, D2: CDSOT23-SM712, SamacSys_Parts:CDSOT23-SM712
- added LED3: (no value), led:LEDSML1206
- added R3: 220, rcl:R-EU_R0805
Connections:
- new net N$11: LED3.C, R3.2
- net AGND: now also D1.3, D2.3, R3.1
- net DA: now also D2.2, J1.7; no longer J1.1
- net DB: now also D2.1, J1.8; no longer J1.2
- net DY: now also D1.2, J1.1; no longer J1.7
- net DZ: now also D1.1, J1.2; no longer J1.8
- net VCC/2: now also LED3.A
Other:
- moved on the sheet: C3, C4, IC1, J2, R1, R2, R5, R6, R7, R8, R9
