File: extruderController/extruderControllerv03.brd (EAGLE design)
At the start: 93.7 x 69.3 mm, 73 parts, among them IC1 LM1117MPX-5.0, IC2 MAX3467CPA, IC3 ATMEGA2561-16AU, IC4 ULN2003AD, J1 RJ45, Q2 PH7030L, Q3 PH7030L, Q4 PH7030L, Q5 PH7030L, Q6 PH7030L, X1 22-23-2081, X2 22-23-2081, X3 22-23-2101, X6 22-23-2041, X8 22-23-2031, X9 22-23-2031

Commit message: f
Parts:
- removed J1: RJ45, SparkFun-Connectors:RJ45-8
- added J8: 615016137621, SamacSys_Parts:WR-MJ
- moved R18 31.4 mm to (63.5, 35.1), turned to 180 degrees
- moved LED1 23.9 mm to (58.4, 35.1), turned to 0 degrees
- moved R13 12.1 mm to (65.3, 40.1), turned to 270 degrees
- moved C2 6.61 mm to (40.4, 63.8)
- moved C12 5.00 mm to (53.8, 47.5)
- moved IC2 4.89 mm to (56.6, 43.4)
- moved C3 4.44 mm to (36.6, 57.4), turned to 180 degrees
- moved IC1 4.07 mm to (32.3, 62.0)
- moved C6 3.89 mm to (45.7, 65.5)
- moved C1 3.25 mm to (22.9, 61.5)
- moved C5 3.09 mm to (27.4, 65.3)
- moved D1 2.81 mm to (14.5, 58.2)
- moved J2 2.29 mm to (12.4, 64.8)
- moved C4 2.05 mm to (27.9, 57.4), turned to 0 degrees
- moved R12 1.08 mm to (65.3, 46.2), turned to 90 degrees
Connections:
- removed net N$27: IC2.7, J1.7, R13.1
- removed net N$35: IC2.5, J1.4
- removed net N$36: IC2.8, J1.8, R13.2
- removed net N$45: IC2.6, J1.5
- new net DA: IC2.8, J8.1, J8.9, R12.2
- new net DB: IC2.7, J8.10, J8.2, R12.1
- new net DY: IC2.5, J8.15, J8.7, R13.2
- new net DZ: IC2.6, J8.16, J8.8, R13.1
- net GND: now also J8.11, J8.12, J8.13, J8.14, J8.3, J8.4, J8.5, J8.6; no longer J1.1, J1.2, J1.3, J1.6
Routing:
- net DY: track 0.00 -> 43.4 mm, vias 0 -> 1
- net DZ: track 0.00 -> 34.4 mm
- net DA: track 0.00 -> 33.3 mm, vias 0 -> 1
- net DB: track 0.00 -> 32.7 mm, vias 0 -> 1
- net +5V: track 364.8 -> 387.8 mm, vias 8 -> 9
- net N$27: track 11.5 -> 0.00 mm
- net N$35: track 9.54 -> 0.00 mm
- net N$36: track 8.96 -> 0.00 mm
- net GND: track 72.8 -> 70.3 mm, vias 104 -> 103
- net PE1: track 12.2 -> 14.4 mm
- net PE2: track 12.9 -> 15.1 mm
- net N$41: track 3.65 -> 2.38 mm
- net N$20: track 22.7 -> 23.6 mm
- net N$19: track 26.9 -> 26.4 mm

Commit message: e
Connections:
- net PE0: now also IC2.2; no longer J3.7
- net PE2: now also J3.7; no longer IC2.2
Routing:
- net PE0: track 70.8 -> 15.0 mm
- net PE2: track 15.1 -> 70.2 mm, vias 0 -> 2
Changed lines of the file:
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@@
 <?xml version="1.0" encoding="utf-8"?>
 <!DOCTYPE eagle SYSTEM "eagle.dtd">
-<eagle version="9.2.2">
+<eagle version="9.3.1">
 <drawing>
 <settings>
@@
 <layers>
 <layer number="1" name="Top" color="4" fill="1" visible="yes" active="yes"/>
-<layer number="16" name="Bottom" color="1" fill="1" visible="no" active="yes"/>
+<layer number="16" name="Bottom" color="1" fill="1" visible="yes" active="yes"/>
 <layer number="17" name="Pads" color="2" fill="1" visible="yes" active="yes"/>
 <layer number="18" name="Vias" color="2" fill="1" visible="yes" active="yes"/>
@@
 <signal name="PE2">
 <contactref element="IC3" pad="4"/>
-<contactref element="IC2" pad="2"/>
-<wire x1="41.6433" y1="45.8597" x2="41.6433" y2="46.7233" width="0.3048" layer="1"/>
-<wire x1="43.0502" y1="48.1302" x2="47.3738" y2="48.1302" width="0.3048" layer="1"/>
-<wire x1="41.6433" y1="46.7233" x2="43.0502" y2="48.1302" width="0.3048" layer="1"/>
-<wire x1="51.435" y1="44.069" x2="53.5686" y2="44.069" width="0.3048" layer="1"/>
-<wire x1="47.3738" y1="48.1302" x2="51.435" y2="44.069" width="0.3048" layer="1"/>
+<contactref element="J3" pad="7"/>
+<via x="39.12361875" y="40.64761875" extent="1-16" drill="0.35"/>
+<wire x1="51.87166875" y1="30.5816" x2="42.551" y2="30.5816" width="0.3048" layer="16"/>
+<wire x1="39.12361875" y1="40.64761875" x2="39.12361875" y2="40.59753125" width="0.3048" layer="16"/>
+<wire x1="39.12361875" y1="40.59753125" x2="38.941" y2="40.4149125" width="0.3048" layer="16"/>
+<wire x1="38.941" y1="40.4149125" x2="38.941" y2="34.1916" width="0.3048" layer="16"/>
+<wire x1="38.941" y1="34.1916" x2="42.551" y2="30.5816" width="0.3048" layer="16"/>
+<via x="73.66" y="40.053" extent="1-16" drill="0.35"/>
+<wire x1="78.42486875" y1="40.053" x2="73.66" y2="40.053" width="0.3048" layer="1"/>
+<wire x1="73.66" y1="40.053" x2="61.34306875" y2="40.053" width="0.3048" layer="16"/>
+<wire x1="61.34306875" y1="40.053" x2="51.87166875" y2="30.5816" width="0.3048" layer="16"/>
+<wire x1="83.81246875" y1="46.4566" x2="83.0834" y2="45.72753125" width="0.3048" layer="1"/>
+<wire x1="87.122" y1="47.752" x2="85.8266" y2="46.4566" width="0.3048" layer="1"/>
+<wire x1="85.8266" y1="46.4566" x2="83.81246875" y2="46.4566" width="0.3048" layer="1"/>
+<wire x1="83.0834" y1="45.72753125" x2="83.0834" y2="44.71153125" width="0.3048" layer="1"/>
+<wire x1="83.0834" y1="44.71153125" x2="78.42486875" y2="40.053" width="0.3048" layer="1"/>
+<wire x1="41.6433" y1="45.8597" x2="41.6433" y2="43.1673" width="0.3048" layer="1"/>
+<wire x1="41.6433" y1="43.1673" x2="39.12361875" y2="40.64761875" width="0.3048" layer="1"/>
 </signal>
 <signal name="PE1">
@@
 <signal name="PE0">
 <contactref element="IC3" pad="2"/>
-<wire x1="43.2181" y1="45.8597" x2="43.2181" y2="44.7421" width="0.3048" layer="1"/>
-<wire x1="43.2181" y1="44.7421" x2="39.12361875" y2="40.64761875" width="0.3048" layer="1"/>
-<via x="39.12361875" y="40.64761875" extent="1-16" drill="0.35"/>
-<wire x1="51.87166875" y1="30.5816" x2="42.551" y2="30.5816" width="0.3048" layer="16"/>
-<wire x1="39.12361875" y1="40.64761875" x2="39.12361875" y2="40.59753125" width="0.3048" layer="16"/>
-<wire x1="39.12361875" y1="40.59753125" x2="38.941" y2="40.4149125" width="0.3048" layer="16"/>
-<wire x1="38.941" y1="40.4149125" x2="38.941" y2="34.1916" width="0.3048" layer="16"/>
-<wire x1="38.941" y1="34.1916" x2="42.551" y2="30.5816" width="0.3048" layer="16"/>
-<contactref element="J3" pad="7"/>
-<via x="73.66" y="40.053" extent="1-16" drill="0.35"/>
-<wire x1="78.42486875" y1="40.053" x2="73.66" y2="40.053" width="0.3048" layer="1"/>
-<wire x1="73.66" y1="40.053" x2="61.34306875" y2="40.053" width="0.3048" layer="16"/>
-<wire x1="61.34306875" y1="40.053" x2="51.87166875" y2="30.5816" width="0.3048" layer="16"/>
-<wire x1="83.81246875" y1="46.4566" x2="83.0834" y2="45.72753125" width="0.3048" layer="1"/>
-<wire x1="87.122" y1="47.752" x2="85.8266" y2="46.4566" width="0.3048" layer="1"/>
-<wire x1="85.8266" y1="46.4566" x2="83.81246875" y2="46.4566" width="0.3048" layer="1"/>
-<wire x1="83.0834" y1="45.72753125" x2="83.0834" y2="44.71153125" width="0.3048" layer="1"/>
-<wire x1="83.0834" y1="44.71153125" x2="78.42486875" y2="40.053" width="0.3048" layer="1"/>
+<contactref element="IC2" pad="2"/>
+<wire x1="53.5686" y1="44.069" x2="51.6389125" y2="44.069" width="0.3048" layer="1"/>
+<wire x1="51.6389125" y1="44.069" x2="48.23495625" y2="47.47295625" width="0.3048" layer="1"/>
+<via x="48.23495625" y="47.47295625" extent="1-16" drill="0.35"/>
+<wire x1="48.23495625" y1="47.47295625" x2="48.23495625" y2="46.71095625" width="0.3048" layer="16"/>
+<wire x1="48.23495625" y1="46.71095625" x2="46.736" y2="45.212" width="0.3048" layer="16"/>
+<wire x1="46.736" y1="45.212" x2="45.72" y2="45.212" width="0.3048" layer="16"/>
+<wire x1="45.72" y1="45.212" x2="45.212" y2="45.72" width="0.3048" layer="16"/>
+<wire x1="45.212" y1="45.72" x2="45.212" y2="46.228" width="0.3048" layer="16"/>
+<wire x1="45.212" y1="46.228" x2="44.45" y2="46.99" width="0.3048" layer="16"/>
+<via x="44.45" y="46.99" extent="1-16" drill="0.35"/>
+<wire x1="44.45" y1="46.99" x2="43.688" y2="46.99" width="0.3048" layer="1"/>
+<wire x1="43.688" y1="46.99" x2="43.2181" y2="46.5201" width="0.3048" layer="1"/>
+<wire x1="43.2181" y1="46.5201" x2="43.2181" y2="45.8597" width="0.3048" layer="1"/>
 </signal>
 <signal name="PF5">

Commit message: o
Parts:
- added J1: (no value), SparkFun-Connectors:1X04
Connections:
- net +5V: now also J1.4
- net GND: now also J1.1
- net PE0: now also J1.2
- net PE1: now also J1.3
Routing:
- net PE1: track 14.4 -> 44.9 mm, vias 0 -> 1
- net PE0: track 15.0 -> 38.7 mm, vias 2 -> 3
- net +5V: track 387.8 -> 398.9 mm
- net DY: track 43.4 -> 40.3 mm
- net DZ: track 34.4 -> 35.7 mm
- net GND: vias 103 -> 106
Other:
- board text added: "EXTURBATOR"
- board text added: "RX"
- board text added: "TX"
- board text added: "UART0"
- board text removed: "Controller"
