File: extruderController/extruderControllerv03.brd (EAGLE design)
At the start: 93.7 x 69.3 mm, 74 parts, among them IC1 LM1117MPX-5.0, IC2 MAX3467CPA, IC3 ATMEGA2561-16AU, IC4 ULN2003AD, J8 615016137621, Q2 PH7030L, Q3 PH7030L, Q4 PH7030L, Q5 PH7030L, Q6 PH7030L, X1 22-23-2081, X2 22-23-2081, X3 22-23-2101, X6 22-23-2041, X8 22-23-2031, X9 22-23-2031

Commit message: d
Parts:
- moved R18 7.62 mm to (55.9, 34.8), turned to 0 degrees
- moved LED1 3.06 mm to (61.5, 34.8), turned to 180 degrees
Connections:
- net GND: no longer R18.1
- net PF6: now also R18.1
Routing:
- net PA4: track 72.4 -> 67.0 mm
- net PA5: track 71.4 -> 66.2 mm
- net PA6: track 70.4 -> 65.5 mm
- net PA7: track 69.4 -> 64.7 mm
- net PG2: track 68.4 -> 64.0 mm
- net PC7: track 67.5 -> 63.4 mm
- net PC5: track 65.8 -> 61.7 mm
- net PC4: track 65.3 -> 61.2 mm
- net PC6: track 66.7 -> 62.7 mm
- net PF6: track 57.8 -> 61.3 mm, vias 2 -> 3
- net +5V: track 398.9 -> 401.3 mm
- net PD5: track 47.9 -> 49.8 mm, vias 8 -> 5
- net N$10: track 34.8 -> 36.6 mm
- net N$11: track 33.9 -> 35.7 mm
- net GND: track 70.3 -> 69.1 mm, vias 106 -> 113
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
Commit message: g
Routing:
- net PB3(MISO): track 10.7 -> 11.6 mm
- net PE7: track 68.4 -> 67.6 mm
- net PE6: track 72.2 -> 72.8 mm
- net GND: vias 113 -> 114

Commit message: v
Routing:
- net DA: track 32.9 -> 33.6 mm
Changed lines of the file:
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@@
 <layers>
 <layer number="1" name="Top" color="4" fill="1" visible="yes" active="yes"/>
-<layer number="16" name="Bottom" color="1" fill="1" visible="no" active="yes"/>
+<layer number="16" name="Bottom" color="1" fill="1" visible="yes" active="yes"/>
 <layer number="17" name="Pads" color="2" fill="1" visible="yes" active="yes"/>
 <layer number="18" name="Vias" color="2" fill="1" visible="yes" active="yes"/>
@@
 <wire x1="44.2849" y1="36.9189" x2="42.672" y2="35.306" width="0.3048" layer="1"/>
 <via x="42.672" y="35.306" extent="1-16" drill="0.35"/>
-<wire x1="42.672" y1="35.306" x2="44.196" y2="33.782" width="0.3048" layer="16"/>
-<wire x1="50.546" y1="33.782" x2="44.196" y2="33.782" width="0.3048" layer="16"/>
+<wire x1="43.942" y1="33.782" x2="42.672" y2="35.052" width="0.3048" layer="16"/>
+<wire x1="42.672" y1="35.306" x2="42.672" y2="35.052" width="0.3048" layer="16"/>
+<wire x1="50.546" y1="33.782" x2="43.942" y2="33.782" width="0.3048" layer="16"/>
 <contactref element="J5" pad="10"/>
 <wire x1="84.328" y1="55.372" x2="83.5152" y2="54.5592" width="0.3048" layer="1"/>
@@
 <contactref element="R12" pad="2"/>
 <contactref element="IC2" pad="8"/>
-<wire x1="59.7154" y1="45.339" x2="59.7154" y2="48.2854" width="0.6096" layer="1"/>
+<wire x1="59.2074" y1="47.7774" x2="59.2074" y2="45.339" width="0.6096" layer="1"/>
+<wire x1="59.7154" y1="45.339" x2="59.2074" y2="45.339" width="0.6096" layer="1"/>
 <wire x1="61.468" y1="50.038" x2="61.468" y2="51.054" width="0.6096" layer="1"/>
-<wire x1="61.468" y1="50.038" x2="59.7154" y2="48.2854" width="0.6096" layer="1"/>
+<wire x1="61.468" y1="50.038" x2="59.2074" y2="47.7774" width="0.6096" layer="1"/>
 <via x="61.468" y="51.054" extent="1-16" drill="0.35"/>
 <wire x1="61.468" y1="51.054" x2="61.722" y2="51.308" width="0.6096" layer="16"/>

Commit message: j
Parts:
- added R19: 1M, rcl:R0805
- added R20: 27, rcl:R0805
- moved C4 2.27 mm to (29.0, 55.4)
- moved C3 2.03 mm to (36.6, 55.4)
- moved Q1 2.03 mm to (32.8, 51.6)
- moved C7 1.55 mm to (29.5, 46.0), turned to 0 degrees
- moved R1 1.52 mm to (31.5, 48.0)
Connections:
- new net N$35: IC3.24, R20.1
- net N$19: now also R19.2
- net N$20: now also R19.1, R20.2; no longer IC3.24
Routing:
- net GND: track 69.1 -> 52.4 mm, vias 114 -> 116
- net N$35: track 0.00 -> 3.61 mm
- net N$19: track 26.4 -> 28.4 mm
- net PD4: track 23.2 -> 24.4 mm
- net N$14: track 24.6 -> 25.5 mm
- net RESET: track 25.2 -> 24.6 mm
- net N$13: track 21.5 -> 22.1 mm

Commit message: f
Parts:
- removed X6: 22-23-2041, con-molex:22-23-2041
- added X4: 22-23-2051, con-molex:22-23-2051
- moved C18 4.17 mm to (70.9, 10.9)
- moved LED1 3.59 mm to (65.0, 35.3)
- moved R18 2.84 mm to (58.7, 35.3)
- moved R12 0.25 mm to (65.3, 46.0)
Connections:
- new net N$27: IC4.16, X4.1
- net +5V: now also X4.4; no longer X6.3
- net GND: now also X4.5; no longer X6.4
- net N$15: now also X4.2; no longer X6.1
- net N$21: now also X4.3; no longer X6.2
- net PF5: now also IC4.2; no longer J3.10
- net PF6: no longer J5.10
- net PG5: now also IC4.1; no longer IC4.2
Routing:
- net PF6: track 61.5 -> 25.2 mm, vias 3 -> 2
- net PF5: track 63.2 -> 32.4 mm, vias 2 -> 0
- net N$27: track 0.00 -> 19.4 mm
- net +5V: track 401.1 -> 406.0 mm, vias 9 -> 11
- net GND: track 52.4 -> 54.3 mm
- net PE6: track 72.8 -> 71.2 mm
- net PE7: track 67.6 -> 66.0 mm
- net PF7: track 31.7 -> 30.7 mm
- net N$41: track 2.89 -> 3.65 mm
- net PA0: track 28.0 -> 28.7 mm
- net N$15: track 19.4 -> 18.9 mm
- net N$21: track 18.9 -> 18.4 mm
Other:
- board text added: "ENA"
- board text added: "HOPPER LEVEL"
- board text added: "SCREW ROTATION"
- board text removed: "Hopper level"
- board text removed: "Screw rotation"

Commit message: f
Parts:
- removed J1: (no value), SparkFun-Connectors:1X04
- added X5: TSW-102-07-G-D, con-samtec:TSW-102-XX-G-D
- moved R12 0.51 mm to (64.8, 46.0)
- moved R13 0.51 mm to (64.8, 40.1)
Connections:
- net +5V: now also X5.3; no longer J1.4
- net GND: now also X5.4; no longer J1.1
- net PE0: now also X5.2; no longer J1.2
- net PE1: now also X5.1; no longer J1.3
Routing:
- net +5V: track 406.0 -> 410.2 mm
- net PE1: track 44.5 -> 43.8 mm
- net DY: track 39.8 -> 39.3 mm
- net DA: track 33.5 -> 33.0 mm

Commit message: e
Connections:
- net PE3: now also IC4.1
- net PG5: no longer IC4.1
Routing:
- net PE3: track 0.00 -> 46.7 mm
- net PG5: track 41.3 -> 0.00 mm
Changed lines of the file:
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@@
 <layers>
 <layer number="1" name="Top" color="4" fill="1" visible="yes" active="yes"/>
-<layer number="16" name="Bottom" color="1" fill="1" visible="no" active="yes"/>
+<layer number="16" name="Bottom" color="1" fill="1" visible="yes" active="yes"/>
 <layer number="17" name="Pads" color="2" fill="1" visible="yes" active="yes"/>
 <layer number="18" name="Vias" color="2" fill="1" visible="yes" active="yes"/>
@@
 <via x="37.592" y="44.45" extent="1-16" drill="0.35"/>
 <via x="31.75" y="38.608" extent="1-16" drill="0.35"/>
-<via x="42.672" y="43.18" extent="1-16" drill="0.35"/>
+<via x="42.672" y="42.672" extent="1-16" drill="0.35"/>
 <via x="28.448" y="26.416" extent="1-16" drill="0.35"/>
 <via x="35.306" y="25.654" extent="1-16" drill="0.35"/>
@@
 <contactref element="IC3" pad="4"/>
 <contactref element="J3" pad="7"/>
-<via x="40.64761875" y="42.93361875" extent="1-16" drill="0.35"/>
+<via x="41.66361875" y="44.45761875" extent="1-16" drill="0.35"/>
 <wire x1="51.87166875" y1="30.5816" x2="42.551" y2="30.5816" width="0.3048" layer="16"/>
-<wire x1="40.64761875" y1="42.93361875" x2="40.44370625" y2="42.93361875" width="0.3048" layer="16"/>
-<wire x1="40.44370625" y1="42.93361875" x2="38.941" y2="41.4309125" width="0.3048" layer="16"/>
+<wire x1="41.66361875" y1="44.45761875" x2="41.66361875" y2="44.15353125" width="0.3048" layer="16"/>
+<wire x1="41.66361875" y1="44.15353125" x2="38.941" y2="41.4309125" width="0.3048" layer="16"/>
 <wire x1="38.941" y1="41.4309125" x2="38.941" y2="34.1916" width="0.3048" layer="16"/>
 <wire x1="38.941" y1="34.1916" x2="42.551" y2="30.5816" width="0.3048" layer="16"/>
@@
 <wire x1="83.0834" y1="45.72753125" x2="83.0834" y2="44.96553125" width="0.3048" layer="1"/>
 <wire x1="83.0834" y1="44.96553125" x2="78.17086875" y2="40.053" width="0.3048" layer="1"/>
-<wire x1="41.6433" y1="45.8597" x2="41.6433" y2="44.9453" width="0.3048" layer="1"/>
-<wire x1="41.6433" y1="44.9453" x2="40.64761875" y2="43.94961875" width="0.3048" layer="1"/>
-<wire x1="40.64761875" y1="43.94961875" x2="40.64761875" y2="42.93361875" width="0.3048" layer="1"/>
+<wire x1="41.6433" y1="45.8597" x2="41.6433" y2="44.4779375" width="0.3048" layer="1"/>
+<wire x1="41.6433" y1="44.4779375" x2="41.66361875" y2="44.45761875" width="0.3048" layer="1"/>
 </signal>
 <signal name="PE1">
@@
 <signal name="PG5">
 <contactref element="IC3" pad="1"/>
-<wire x1="48.514" y1="39.116" x2="55.9816" y2="31.6484" width="0.3048" layer="1"/>
-<wire x1="48.514" y1="39.116" x2="48.514" y2="43.18" width="0.3048" layer="1"/>
-<wire x1="48.514" y1="43.18" x2="46.482" y2="45.212" width="0.3048" layer="1"/>
-<wire x1="44.6532" y1="45.212" x2="44.0055" y2="45.8597" width="0.3048" layer="1"/>
-<wire x1="46.482" y1="45.212" x2="44.6532" y2="45.212" width="0.3048" layer="1"/>
-<contactref element="IC4" pad="1"/>
-<wire x1="72.35003125" y1="29.5402" x2="73.0758" y2="29.5402" width="0.3048" layer="1"/>
-<wire x1="73.0758" y1="29.5402" x2="74.676" y2="27.94" width="0.3048" layer="1"/>
-<wire x1="70.24183125" y1="31.6484" x2="72.35003125" y2="29.5402" width="0.3048" layer="1"/>
-<wire x1="74.676" y1="27.94" x2="74.676" y2="27.3304" width="0.3048" layer="1"/>
-<wire x1="74.676" y1="27.3304" x2="74.549" y2="27.2034" width="0.3048" layer="1"/>
-<wire x1="55.9816" y1="31.6484" x2="70.24183125" y2="31.6484" width="0.3048" layer="1"/>
 </signal>
 <signal name="PA4">
@@
 <signal name="PE3">
 <contactref element="IC3" pad="5"/>
+<contactref element="IC4" pad="1"/>
+<wire x1="40.8559" y1="45.8597" x2="40.8559" y2="44.2341" width="0.3048" layer="1"/>
+<wire x1="40.8559" y1="44.2341" x2="41.402" y2="43.688" width="0.3048" layer="1"/>
+<wire x1="41.402" y1="43.688" x2="43.688" y2="43.688" width="0.3048" layer="1"/>
+<wire x1="43.688" y1="43.688" x2="44.958" y2="44.958" width="0.3048" layer="1"/>
+<wire x1="44.958" y1="44.958" x2="46.85141875" y2="44.958" width="0.3048" layer="1"/>
+<wire x1="48.514" y1="39.116" x2="55.9816" y2="31.6484" width="0.3048" layer="1"/>
+<wire x1="70.24183125" y1="31.6484" x2="72.35003125" y2="29.5402" width="0.3048" layer="1"/>
+<wire x1="72.35003125" y1="29.5402" x2="73.5838" y2="29.5402" width="0.3048" layer="1"/>
+<wire x1="55.9816" y1="31.6484" x2="70.24183125" y2="31.6484" width="0.3048" layer="1"/>
+<wire x1="74.549" y1="28.575" x2="74.549" y2="27.2034" width="0.3048" layer="1"/>
+<wire x1="46.85141875" y1="44.958" x2="48.514" y2="43.29541875" width="0.3048" layer="1"/>
+<wire x1="48.514" y1="43.29541875" x2="48.514" y2="39.116" width="0.3048" layer="1"/>
+<wire x1="73.5838" y1="29.5402" x2="74.549" y2="28.575" width="0.3048" layer="1"/>
 </signal>
 <signal name="PE0">

Commit message: V
Routing:
- net +5V: track 410.2 -> 410.7 mm
Other:
- board text added: "HOPPER"
- board text added: "SCREW"
- board text removed: "HOPPER LEVEL"
- board text removed: "SCREW ROTATION"
Changed lines of the file:
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@@
 <grid distance="10" unitdist="mil" unit="mil" style="lines" multiple="1" display="yes" altdistance="5" altunitdist="mil" altunit="mil"/>
 <layers>
-<layer number="1" name="Top" color="4" fill="1" visible="yes" active="yes"/>
+<layer number="1" name="Top" color="4" fill="1" visible="no" active="yes"/>
 <layer number="16" name="Bottom" color="1" fill="1" visible="yes" active="yes"/>
 <layer number="17" name="Pads" color="2" fill="1" visible="yes" active="yes"/>
@@
 <text x="69.85" y="7.62" size="1.016" layer="25" font="vector" ratio="20" rot="R90">GND</text>
 <text x="72.644" y="7.62" size="1.016" layer="25" font="vector" ratio="20" rot="R90">5V</text>
-<text x="85.852" y="15.494" size="1.016" layer="25" font="vector" ratio="20" rot="SR180">SCREW ROTATION</text>
+<text x="85.852" y="15.494" size="1.016" layer="25" font="vector" ratio="20" rot="SR180">HOPPER</text>
 <text x="42.672" y="7.62" size="1.016" layer="25" font="vector" ratio="20" rot="R90">5V</text>
 <text x="47.752" y="7.62" size="1.016" layer="25" font="vector" ratio="20" rot="R90">5V</text>
@@
 <text x="85.852" y="18.288" size="1.016" layer="25" font="vector" ratio="20" rot="SR180">5V</text>
 <text x="86.106" y="12.954" size="1.016" layer="25" font="vector" ratio="20" rot="SR180">GND</text>
-<text x="86.106" y="26.162" size="1.016" layer="25" font="vector" ratio="20" rot="SR180">HOPPER LEVEL</text>
+<text x="86.106" y="26.162" size="1.016" layer="25" font="vector" ratio="20" rot="SR180">SCREW</text>
 <text x="10.16" y="22.352" size="1.016" layer="25" font="vector" ratio="20" rot="SR180">12V</text>
 <text x="10.16" y="27.432" size="1.016" layer="25" font="vector" ratio="20" rot="SR180">12V</text>
@@
 <wire x1="45.8597" y1="43.2181" x2="45.8597" y2="44.0055" width="0.3048" layer="1"/>
 <wire x1="30.3403" y1="40.8559" x2="29.5021" y2="40.8559" width="0.508" layer="1"/>
-<wire x1="28.6258" y1="41.7322" x2="29.5021" y2="40.8559" width="0.508" layer="1"/>
+<wire x1="28.3718" y1="41.9862" x2="29.5021" y2="40.8559" width="0.508" layer="1"/>
 <wire x1="30.546" y1="48.006" x2="30.314" y2="47.774" width="0.508" layer="1"/>
 <wire x1="31.496" y1="49.276" x2="30.546" y2="48.326" width="0.508" layer="1"/>
@@
 <wire x1="47.244" y1="59.182" x2="46.736" y2="59.69" width="0.6096" layer="1"/>
 <wire x1="46.482" y1="59.944" x2="46.736" y2="59.69" width="0.6096" layer="1"/>
-<wire x1="78.31896875" y1="58.956" x2="78.31896875" y2="55.71296875" width="0.8128" layer="16"/>
-<wire x1="76.2" y1="53.594" x2="78.31896875" y2="55.71296875" width="0.8128" layer="16"/>
+<wire x1="78.31896875" y1="58.956" x2="78.31896875" y2="50.37896875" width="0.8128" layer="16"/>
+<wire x1="73.914" y1="45.974" x2="78.31896875" y2="50.37896875" width="0.8128" layer="16"/>
 <wire x1="41.402" y1="47.244" x2="44.958" y2="50.8" width="1.27" layer="1"/>
 <wire x1="48.514" y1="50.8" x2="44.958" y2="50.8" width="1.27" layer="1"/>
-<wire x1="30.546" y1="48.006" x2="29.718" y2="48.006" width="0.508" layer="1"/>
-<wire x1="28.614" y1="46.902" x2="28.614" y2="45.974" width="0.508" layer="1"/>
-<wire x1="29.718" y1="48.006" x2="28.614" y2="46.902" width="0.508" layer="1"/>
-<wire x1="28.614" y1="45.974" x2="28.6258" y2="45.9622" width="0.508" layer="1"/>
-<wire x1="28.6258" y1="45.9622" x2="28.6258" y2="41.7322" width="0.508" layer="1"/>
+<wire x1="30.546" y1="48.006" x2="29.464" y2="48.006" width="0.508" layer="1"/>
+<wire x1="28.36" y1="46.902" x2="28.36" y2="46.228" width="0.508" layer="1"/>
+<wire x1="28.36" y1="46.228" x2="28.614" y2="45.974" width="0.508" layer="1"/>
+<wire x1="29.464" y1="48.006" x2="28.36" y2="46.902" width="0.508" layer="1"/>
+<wire x1="28.614" y1="45.974" x2="28.3718" y2="45.7318" width="0.508" layer="1"/>
+<wire x1="28.3718" y1="45.7318" x2="28.3718" y2="41.9862" width="0.508" layer="1"/>
 <wire x1="53.5686" y1="45.339" x2="54.483" y2="45.339" width="0.508" layer="1"/>
 <wire x1="54.483" y1="45.339" x2="55.118" y2="44.704" width="0.508" layer="1"/>
@@
 <wire x1="87.122" y1="13.97" x2="86.614" y2="13.97" width="0.8128" layer="1"/>
 <contactref element="X5" pad="3"/>
-<wire x1="73.914" y1="45.974" x2="76.2" y2="48.26" width="0.8128" layer="16"/>
-<wire x1="76.2" y1="48.26" x2="76.2" y2="53.594" width="0.8128" layer="16"/>
 <wire x1="55.118" y1="43.688" x2="58.166" y2="40.64" width="0.508" layer="1"/>
 <wire x1="58.166" y1="40.64" x2="60.452" y2="40.64" width="0.508" layer="1"/>
@@
 <contactref element="R1" pad="2"/>
 <wire x1="30.3403" y1="41.6433" x2="29.7307" y2="41.6433" width="0.3048" layer="1"/>
-<wire x1="29.7307" y1="41.6433" x2="29.4386" y2="41.9354" width="0.3048" layer="1"/>
+<wire x1="29.7307" y1="41.6433" x2="29.1846" y2="42.1894" width="0.3048" layer="1"/>
 <wire x1="33.528" y1="47.498" x2="32.954" y2="47.498" width="0.3048" layer="1"/>
 <wire x1="32.954" y1="47.498" x2="32.606" y2="47.846" width="0.3048" layer="1"/>
 <wire x1="32.606" y1="47.846" x2="32.446" y2="48.006" width="0.3048" layer="1"/>
-<wire x1="29.4386" y1="44.41115" x2="29.98545" y2="44.958" width="0.3048" layer="1"/>
-<wire x1="29.98545" y1="44.958" x2="30.988" y2="44.958" width="0.3048" layer="1"/>
+<wire x1="29.1846" y1="44.41115" x2="29.73145" y2="44.958" width="0.3048" layer="1"/>
+<wire x1="29.73145" y1="44.958" x2="30.988" y2="44.958" width="0.3048" layer="1"/>
 <wire x1="30.988" y1="44.958" x2="31.496" y2="45.466" width="0.3048" layer="1"/>
 <wire x1="31.496" y1="46.736" x2="32.606" y2="47.846" width="0.3048" layer="1"/>
-<wire x1="29.4386" y1="41.9354" x2="29.4386" y2="44.41115" width="0.3048" layer="1"/>
+<wire x1="29.1846" y1="42.1894" x2="29.1846" y2="44.41115" width="0.3048" layer="1"/>
 <wire x1="31.496" y1="45.466" x2="31.496" y2="46.736" width="0.3048" layer="1"/>
 </signal>
