File: extruderController/extruderControllerv03.brd (EAGLE design)
At the start: 93.7 x 69.3 mm, 76 parts, among them IC1 LM1117MPX-5.0, IC2 MAX3467CPA, IC3 ATMEGA2561-16AU, IC4 ULN2003AD, J8 615016137621, Q2 PH7030L, Q3 PH7030L, Q4 PH7030L, Q5 PH7030L, Q6 PH7030L, X1 22-23-2081, X2 22-23-2081, X3 22-23-2101, X4 22-23-2051, X5 TSW-102-07-G-D, X8 22-23-2031, X9 22-23-2031

Commit message: c
Parts:
- turned C3 to 0 degrees
- turned C4 to 180 degrees
Routing:
- net N$19: track 28.4 -> 25.0 mm
- net N$20: track 23.7 -> 20.4 mm
- net GND: vias 116 -> 118
Changed lines of the file:
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@@
 <grid distance="10" unitdist="mil" unit="mil" style="lines" multiple="1" display="yes" altdistance="5" altunitdist="mil" altunit="mil"/>
 <layers>
-<layer number="1" name="Top" color="4" fill="1" visible="no" active="yes"/>
+<layer number="1" name="Top" color="4" fill="1" visible="yes" active="yes"/>
 <layer number="16" name="Bottom" color="1" fill="1" visible="yes" active="yes"/>
 <layer number="17" name="Pads" color="2" fill="1" visible="yes" active="yes"/>
@@
 <element name="H3" library="holes" library_urn="urn:adsk.eagle:library:237" package="3,3-PAD" package3d_urn="urn:adsk.eagle:package:14283/1" value="MOUNT-PAD-ROUND3.3" x="88.9" y="5.08" smashed="yes"/>
 <element name="H4" library="holes" library_urn="urn:adsk.eagle:library:237" package="3,3-PAD" package3d_urn="urn:adsk.eagle:package:14283/1" value="MOUNT-PAD-ROUND3.3" x="88.646" y="64.262" smashed="yes"/>
-<element name="C3" library="rcl" library_urn="urn:adsk.eagle:library:334" package="C0603" package3d_urn="urn:adsk.eagle:package:23616/2" value="" x="36.576" y="55.372" smashed="yes" rot="R180">
-<attribute name="SPICEPREFIX" value="C" x="36.576" y="55.372" size="1.778" layer="27" rot="R180" display="off"/>
-<attribute name="VALUE" x="37.211" y="57.277" size="1.27" layer="27" rot="R180"/>
-</element>
-<element name="C4" library="rcl" library_urn="urn:adsk.eagle:library:334" package="C0603" package3d_urn="urn:adsk.eagle:package:23616/2" value="" x="28.956" y="55.372" smashed="yes">
-<attribute name="SPICEPREFIX" value="C" x="28.956" y="55.372" size="1.778" layer="27" display="off"/>
-<attribute name="VALUE" x="28.321" y="53.467" size="1.27" layer="27"/>
+<element name="C3" library="rcl" library_urn="urn:adsk.eagle:library:334" package="C0603" package3d_urn="urn:adsk.eagle:package:23616/2" value="" x="36.576" y="55.372" smashed="yes">
+<attribute name="SPICEPREFIX" value="C" x="36.576" y="55.372" size="1.778" layer="27" display="off"/>
+<attribute name="VALUE" x="35.941" y="53.467" size="1.27" layer="27"/>
+</element>
+<element name="C4" library="rcl" library_urn="urn:adsk.eagle:library:334" package="C0603" package3d_urn="urn:adsk.eagle:package:23616/2" value="" x="28.956" y="55.372" smashed="yes" rot="R180">
+<attribute name="SPICEPREFIX" value="C" x="28.956" y="55.372" size="1.778" layer="27" rot="R180" display="off"/>
+<attribute name="VALUE" x="29.591" y="57.277" size="1.27" layer="27" rot="R180"/>
 </element>
 <element name="R1" library="rcl" library_urn="urn:adsk.eagle:library:334" package="R0805" package3d_urn="urn:adsk.eagle:package:23553/2" value="10k" x="31.496" y="48.006" smashed="yes">
@@
 </element>
 <element name="R19" library="rcl" library_urn="urn:adsk.eagle:library:334" package="R0805" package3d_urn="urn:adsk.eagle:package:23553/2" value="1M" x="32.766" y="55.372" smashed="yes">
-<attribute name="NAME" x="32.131" y="56.642" size="1.27" layer="25"/>
 <attribute name="SPICEPREFIX" value="R" x="32.766" y="55.372" size="1.778" layer="27" display="off"/>
 <attribute name="VALUE" x="32.131" y="52.832" size="1.27" layer="27"/>
 </element>
 <element name="R20" library="rcl" library_urn="urn:adsk.eagle:library:334" package="R0805" package3d_urn="urn:adsk.eagle:package:23553/2" value="27" x="27.94" y="37.592" smashed="yes" rot="R90">
-<attribute name="NAME" x="26.67" y="36.957" size="1.27" layer="25" rot="R90"/>
 <attribute name="SPICEPREFIX" value="R" x="27.94" y="37.592" size="1.778" layer="27" rot="R90" display="off"/>
 <attribute name="VALUE" x="30.48" y="36.957" size="1.27" layer="27" rot="R90"/>
@@
 <wire x1="51.943" y1="41.529" x2="51.816" y2="41.402" width="0.6096" layer="1"/>
 <via x="51.816" y="41.402" extent="1-16" drill="0.35"/>
-<via x="35.306" y="56.896" extent="1-16" drill="0.35"/>
+<via x="37.338" y="56.896" extent="1-16" drill="0.35"/>
 <via x="32.766" y="52.07" extent="1-16" drill="0.35"/>
-<via x="30.226" y="56.896" extent="1-16" drill="0.35"/>
+<via x="28.194" y="56.896" extent="1-16" drill="0.35"/>
 <contactref element="J8" pad="3"/>
 <contactref element="J8" pad="5"/>
@@
 <contactref element="X4" pad="5"/>
 <contactref element="X5" pad="4"/>
+<via x="35.56" y="56.896" extent="1-16" drill="0.35"/>
+<via x="29.718" y="56.896" extent="1-16" drill="0.35"/>
 </signal>
 <signal name="+12V">
@@
 <wire x1="35.306" y1="51.562" x2="33.782" y2="50.038" width="0.3048" layer="1"/>
 <wire x1="33.782" y1="50.038" x2="30.48" y2="50.038" width="0.3048" layer="1"/>
-<wire x1="35.306" y1="51.562" x2="37.426" y2="53.682" width="0.6096" layer="1"/>
-<wire x1="37.426" y1="53.682" x2="37.426" y2="55.372" width="0.6096" layer="1"/>
 <contactref element="R19" pad="2"/>
-<wire x1="33.716" y1="55.372" x2="35.306" y2="53.782" width="0.3048" layer="1"/>
-<wire x1="35.306" y1="53.782" x2="35.306" y2="51.562" width="0.3048" layer="1"/>
+<wire x1="33.716" y1="55.372" x2="35.306" y2="55.372" width="0.508" layer="1"/>
+<wire x1="35.306" y1="55.372" x2="35.726" y2="55.372" width="0.508" layer="1"/>
+<wire x1="35.306" y1="51.562" x2="35.306" y2="55.372" width="0.508" layer="1"/>
 </signal>
 <signal name="N$20">
@@
 <wire x1="30.226" y1="51.562" x2="30.226" y2="50.546" width="0.3048" layer="1"/>
 <wire x1="30.226" y1="50.546" x2="27.2288" y2="47.5488" width="0.3048" layer="1"/>
-<wire x1="28.106" y1="55.372" x2="28.106" y2="53.682" width="0.6096" layer="1"/>
-<wire x1="28.106" y1="53.682" x2="30.226" y2="51.562" width="0.6096" layer="1"/>
 <contactref element="R20" pad="2"/>
 <contactref element="R19" pad="1"/>
-<wire x1="31.816" y1="55.372" x2="30.226" y2="53.782" width="0.3048" layer="1"/>
-<wire x1="30.226" y1="53.782" x2="30.226" y2="51.562" width="0.3048" layer="1"/>
 <wire x1="27.2288" y1="39.2532" x2="27.94" y2="38.542" width="0.3048" layer="1"/>
 <wire x1="27.2288" y1="47.5488" x2="27.2288" y2="39.2532" width="0.3048" layer="1"/>
+<wire x1="29.806" y1="55.372" x2="30.226" y2="55.372" width="0.508" layer="1"/>
+<wire x1="30.226" y1="55.372" x2="31.816" y2="55.372" width="0.508" layer="1"/>
+<wire x1="30.226" y1="51.562" x2="30.226" y2="55.372" width="0.508" layer="1"/>
 </signal>
 <signal name="PD2">

Commit message: e
Parts:
- C3, C4: value (none) -> 22pF
- R14, R15, R16, R17: value (none) -> 120
Changed lines of the file:
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@@
 <?xml version="1.0" encoding="utf-8"?>
 <!DOCTYPE eagle SYSTEM "eagle.dtd">
-<eagle version="9.2.2">
+<eagle version="9.3.1">
 <drawing>
 <settings>
@@
 <element name="H3" library="holes" library_urn="urn:adsk.eagle:library:237" package="3,3-PAD" package3d_urn="urn:adsk.eagle:package:14283/1" value="MOUNT-PAD-ROUND3.3" x="88.9" y="5.08" smashed="yes"/>
 <element name="H4" library="holes" library_urn="urn:adsk.eagle:library:237" package="3,3-PAD" package3d_urn="urn:adsk.eagle:package:14283/1" value="MOUNT-PAD-ROUND3.3" x="88.646" y="64.262" smashed="yes"/>
-<element name="C3" library="rcl" library_urn="urn:adsk.eagle:library:334" package="C0603" package3d_urn="urn:adsk.eagle:package:23616/2" value="" x="36.576" y="55.372" smashed="yes">
+<element name="C3" library="rcl" library_urn="urn:adsk.eagle:library:334" package="C0603" package3d_urn="urn:adsk.eagle:package:23616/2" value="22pF" x="36.576" y="55.372" smashed="yes">
 <attribute name="SPICEPREFIX" value="C" x="36.576" y="55.372" size="1.778" layer="27" display="off"/>
 <attribute name="VALUE" x="35.941" y="53.467" size="1.27" layer="27"/>
 </element>
-<element name="C4" library="rcl" library_urn="urn:adsk.eagle:library:334" package="C0603" package3d_urn="urn:adsk.eagle:package:23616/2" value="" x="28.956" y="55.372" smashed="yes" rot="R180">
+<element name="C4" library="rcl" library_urn="urn:adsk.eagle:library:334" package="C0603" package3d_urn="urn:adsk.eagle:package:23616/2" value="22pF" x="28.956" y="55.372" smashed="yes" rot="R180">
 <attribute name="SPICEPREFIX" value="C" x="28.956" y="55.372" size="1.778" layer="27" rot="R180" display="off"/>
 <attribute name="VALUE" x="29.591" y="57.277" size="1.27" layer="27" rot="R180"/>
@@
 <attribute name="OC_NEWARK" value="30C0862" x="89.916" y="14.986" size="1.778" layer="27" rot="R270" display="off"/>
 </element>
-<element name="R14" library="rcl" library_urn="urn:adsk.eagle:library:334" package="R0805" package3d_urn="urn:adsk.eagle:package:23553/2" value="" x="70.612" y="15.24" smashed="yes" rot="R270">
+<element name="R14" library="rcl" library_urn="urn:adsk.eagle:library:334" package="R0805" package3d_urn="urn:adsk.eagle:package:23553/2" value="120" x="70.612" y="15.24" smashed="yes" rot="R270">
 <attribute name="SPICEPREFIX" value="R" x="70.612" y="15.24" size="1.778" layer="27" rot="R270" display="off"/>
 <attribute name="VALUE" x="68.072" y="15.875" size="1.27" layer="27" rot="R270"/>
 </element>
-<element name="R15" library="rcl" library_urn="urn:adsk.eagle:library:334" package="R0805" package3d_urn="urn:adsk.eagle:package:23553/2" value="" x="68.326" y="15.24" smashed="yes" rot="R270">
+<element name="R15" library="rcl" library_urn="urn:adsk.eagle:library:334" package="R0805" package3d_urn="urn:adsk.eagle:package:23553/2" value="120" x="68.326" y="15.24" smashed="yes" rot="R270">
 <attribute name="SPICEPREFIX" value="R" x="68.326" y="15.24" size="1.778" layer="27" rot="R270" display="off"/>
 <attribute name="VALUE" x="65.786" y="15.875" size="1.27" layer="27" rot="R270"/>
 </element>
-<element name="R16" library="rcl" library_urn="urn:adsk.eagle:library:334" package="R0805" package3d_urn="urn:adsk.eagle:package:23553/2" value="" x="66.04" y="15.24" smashed="yes" rot="R270">
+<element name="R16" library="rcl" library_urn="urn:adsk.eagle:library:334" package="R0805" package3d_urn="urn:adsk.eagle:package:23553/2" value="120" x="66.04" y="15.24" smashed="yes" rot="R270">
 <attribute name="SPICEPREFIX" value="R" x="66.04" y="15.24" size="1.778" layer="27" rot="R270" display="off"/>
 <attribute name="VALUE" x="63.5" y="15.875" size="1.27" layer="27" rot="R270"/>
 </element>
-<element name="R17" library="rcl" library_urn="urn:adsk.eagle:library:334" package="R0805" package3d_urn="urn:adsk.eagle:package:23553/2" value="" x="63.754" y="15.24" smashed="yes" rot="R270">
+<element name="R17" library="rcl" library_urn="urn:adsk.eagle:library:334" package="R0805" package3d_urn="urn:adsk.eagle:package:23553/2" value="120" x="63.754" y="15.24" smashed="yes" rot="R270">
 <attribute name="SPICEPREFIX" value="R" x="63.754" y="15.24" size="1.778" layer="27" rot="R270" display="off"/>
 <attribute name="VALUE" x="61.214" y="15.875" size="1.27" layer="27" rot="R270"/>

Commit message: g
Parts:
- removed R14, R15, R16, R17: 120, rcl:R0805
- moved IC4 6.35 mm to (70.1, 17.8)
Connections:
- removed net N$3: R14.2, X1.1
- removed net N$38: IC4.12, R15.1
- removed net N$39: IC4.11, R16.1
- removed net N$40: IC4.10, R17.1
- net N$12: now also IC4.12; no longer R15.2
- net N$13: now also IC4.11; no longer R16.2
- net N$14: now also IC4.10; no longer R17.2
- net N$30: now also X1.1; no longer R14.1
Routing:
- net N$3: track 15.2 -> 0.00 mm
- net N$30: track 5.02 -> 17.1 mm
- net N$15: track 18.9 -> 12.5 mm
- net N$27: track 19.4 -> 13.1 mm
- net N$21: track 18.4 -> 12.0 mm
- net N$40: track 6.18 -> 0.00 mm
- net N$39: track 5.76 -> 0.00 mm
- net N$38: track 5.34 -> 0.00 mm
- net PA3: track 25.3 -> 29.5 mm
- net PA2: track 25.2 -> 29.0 mm
- net +5V: track 410.7 -> 407.0 mm
- net PA1: track 27.0 -> 30.3 mm
- net GND: track 54.3 -> 51.1 mm, vias 118 -> 123
- net PF5: track 32.4 -> 35.3 mm
- net PF7: track 30.7 -> 33.6 mm
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