File: extruderController/extruderControllerv03.sch (EAGLE design)
At the start: 73 parts, among them IC1 LM1117MPX-5.0, IC2 MAX3467CPA, IC3 ATMEGA2561-16AU, IC4 ULN2003AD, J1 RJ45, Q2 PH7030L, Q3 PH7030L, Q4 PH7030L, Q5 PH7030L, Q6 PH7030L, X1 22-23-2081, X2 22-23-2081, X3 22-23-2101, X6 22-23-2041, X8 22-23-2031, X9 22-23-2031

Commit message: f
Parts:
- removed J1: RJ45, SparkFun-Connectors:RJ45-8
- added J8: 615016137621, SamacSys_Parts:615016137621
Connections:
- removed net N$27: IC2.B, J1.7, R13.1
- removed net N$35: IC2.Y, J1.4
- removed net N$36: IC2.A, J1.8, R13.2
- removed net N$45: IC2.Z, J1.5
- new net DA: IC2.A, J8.1, J8.9, R12.2
- new net DB: IC2.B, J8.10, J8.2, R12.1
- new net DY: IC2.Y, J8.15, J8.7, R13.2
- new net DZ: IC2.Z, J8.16, J8.8, R13.1
- net GND: now also J8.11, J8.12, J8.13, J8.14, J8.3, J8.4, J8.5, J8.6; no longer J1.1, J1.2, J1.3, J1.6
Other:
- moved on the sheet: R12, R13

Commit message: e
Connections:
- net PE0: now also IC2.RO; no longer J3.7
- net PE2: now also J3.7; no longer IC2.RO

Commit message: o
Parts:
- added J1: (no value), SparkFun-Connectors:CONN_04
Connections:
- net +5V: now also J1.4
- net GND: now also J1.1
- net PE0: now also J1.2
- net PE1: now also J1.3
Changed lines of the file:
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@@
 <part name="J8" library="SamacSys_Parts" deviceset="615016137621" device=""/>
 <part name="R12" library="rcl" library_urn="urn:adsk.eagle:library:334" deviceset="R-EU_" device="R1210" package3d_urn="urn:adsk.eagle:package:23554/2" value="120"/>
+<part name="J1" library="SparkFun-Connectors" library_urn="urn:adsk.eagle:library:513" deviceset="CONN_04" device="" package3d_urn="urn:adsk.eagle:package:38085/1"/>
+<part name="GND24" library="supply1" library_urn="urn:adsk.eagle:library:371" deviceset="GND" device=""/>
+<part name="P+34" library="supply1" library_urn="urn:adsk.eagle:library:371" deviceset="+5V" device=""/>
 </parts>
 <sheets>
@@
 <attribute name="VALUE" x="123.19" y="179.578" size="1.778" layer="96"/>
 </instance>
+<instance part="J1" gate="G$1" x="76.2" y="231.14" smashed="yes">
+<attribute name="VALUE" x="71.12" y="223.774" size="1.778" layer="96" font="vector"/>
+<attribute name="NAME" x="71.12" y="239.268" size="1.778" layer="95" font="vector"/>
+</instance>
+<instance part="GND24" gate="1" x="81.28" y="226.06" smashed="yes">
+<attribute name="VALUE" x="78.74" y="223.52" size="1.778" layer="96"/>
+</instance>
+<instance part="P+34" gate="1" x="83.82" y="236.22" smashed="yes" rot="R270">
+<attribute name="VALUE" x="78.74" y="238.76" size="1.778" layer="96"/>
+</instance>
 </instances>
 <busses>
@@
 <junction x="129.54" y="220.98"/>
 <label x="121.92" y="220.98" size="1.778" layer="95"/>
+</segment>
+<segment>
+<pinref part="J1" gate="G$1" pin="1"/>
+<pinref part="GND24" gate="1" pin="GND"/>
 </segment>
 </net>
@@
 <pinref part="J5" gate="G$1" pin="11"/>
 </segment>
+<segment>
+<pinref part="J1" gate="G$1" pin="4"/>
+<pinref part="P+34" gate="1" pin="+5V"/>
+</segment>
 </net>
 <net name="N$1" class="0">
@@
 <pinref part="IC3" gate="G$1" pin="(TXD0/PDO)PE1"/>
 <wire x1="7.62" y1="20.32" x2="20.32" y2="20.32" width="0.1524" layer="91"/>
-<label x="10.16" y="20.32" size="1.778" layer="95"/>
+<label x="15.24" y="20.32" size="1.778" layer="95"/>
 </segment>
 <segment>
@@
 <label x="71.12" y="195.58" size="1.778" layer="95"/>
 </segment>
+<segment>
+<pinref part="J1" gate="G$1" pin="3"/>
+<wire x1="81.28" y1="233.68" x2="91.44" y2="233.68" width="0.1524" layer="91"/>
+<label x="86.36" y="233.68" size="1.778" layer="95"/>
+</segment>
 </net>
 <net name="PE6" class="0">
@@
 <segment>
 <pinref part="IC3" gate="G$1" pin="(RXD0/PCIN8/PDI)PE0"/>
-<wire x1="7.62" y1="17.78" x2="35.56" y2="17.78" width="0.1524" layer="91"/>
-<label x="30.48" y="17.78" size="1.778" layer="95"/>
+<wire x1="7.62" y1="17.78" x2="20.32" y2="17.78" width="0.1524" layer="91"/>
+<label x="15.24" y="17.78" size="1.778" layer="95"/>
 </segment>
 <segment>
@@
 <label x="71.12" y="185.42" size="1.778" layer="95"/>
 </segment>
-</net>
+<segment>
+<pinref part="J1" gate="G$1" pin="2"/>
+<wire x1="81.28" y1="231.14" x2="91.44" y2="231.14" width="0.1524" layer="91"/>
+<label x="86.36" y="231.14" size="1.778" layer="95"/>
+</segment>
+</net>

Commit message: d
Connections:
- net GND: no longer R18.1
- net PF6: now also R18.1
Changed lines of the file:
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@@
 <part name="LED1" library="led" library_urn="urn:adsk.eagle:library:259" deviceset="LED" device="SML1206" package3d_urn="urn:adsk.eagle:package:15829/1"/>
 <part name="R18" library="rcl" library_urn="urn:adsk.eagle:library:334" deviceset="R-EU_" device="R0805" package3d_urn="urn:adsk.eagle:package:23553/2" value="330"/>
-<part name="GND25" library="supply1" library_urn="urn:adsk.eagle:library:371" deviceset="GND" device=""/>
 <part name="P+16" library="supply1" library_urn="urn:adsk.eagle:library:371" deviceset="+5V" device=""/>
 <part name="J2" library="SparkFun-Connectors" library_urn="urn:adsk.eagle:library:513" deviceset="CONN_02" device="3.5MM" package3d_urn="urn:adsk.eagle:package:38050/1"/>
@@
 <attribute name="VALUE" x="33.782" y="186.69" size="1.778" layer="96" rot="R90"/>
 </instance>
-<instance part="GND25" gate="1" x="30.48" y="182.88" smashed="yes">
-<attribute name="VALUE" x="27.94" y="180.34" size="1.778" layer="96"/>
-</instance>
 <instance part="P+16" gate="1" x="30.48" y="208.28" smashed="yes">
 <attribute name="VALUE" x="27.94" y="208.28" size="1.778" layer="96" rot="R90"/>
@@
 <pinref part="C12" gate="G$1" pin="2"/>
 <pinref part="GND23" gate="1" pin="GND"/>
-</segment>
-<segment>
-<pinref part="R18" gate="G$1" pin="1"/>
-<pinref part="GND25" gate="1" pin="GND"/>
 </segment>
 <segment>
@@
 <pinref part="J5" gate="G$1" pin="10"/>
 </segment>
-</net>
+<segment>
+<pinref part="R18" gate="G$1" pin="1"/>
+<wire x1="30.48" y1="185.42" x2="30.48" y2="177.8" width="0.1524" layer="91"/>
+<label x="30.48" y="177.8" size="1.778" layer="95"/>
+</segment>
+</net>

Commit message: j
Parts:
- added R19: 1M, rcl:R-EU_R0805
- added R20: 27, rcl:R-EU_R0805
Connections:
- new net N$35: IC3.XTAL1, R20.1
- net N$19: now also R19.2
- net N$20: now also R19.1, R20.2; no longer IC3.XTAL1
Other:
- moved on the sheet: C3, C4, Q1
Changed lines of the file:
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@@
 <?xml version="1.0" encoding="utf-8"?>
 <!DOCTYPE eagle SYSTEM "eagle.dtd">
-<eagle version="9.3.1">
+<eagle version="9.2.2">
 <drawing>
 <settings>
@@
 <part name="GND24" library="supply1" library_urn="urn:adsk.eagle:library:371" deviceset="GND" device=""/>
 <part name="P+34" library="supply1" library_urn="urn:adsk.eagle:library:371" deviceset="+5V" device=""/>
+<part name="R19" library="rcl" library_urn="urn:adsk.eagle:library:334" deviceset="R-EU_" device="R0805" package3d_urn="urn:adsk.eagle:package:23553/2" value="1M"/>
+<part name="R20" library="rcl" library_urn="urn:adsk.eagle:library:334" deviceset="R-EU_" device="R0805" package3d_urn="urn:adsk.eagle:package:23553/2" value="27"/>
 </parts>
 <sheets>
@@
 <attribute name="VALUE" x="-195.58" y="93.98" size="1.778" layer="96" rot="R180"/>
 </instance>
-<instance part="Q1" gate="G$1" x="-76.2" y="121.92" smashed="yes" rot="R90">
-<attribute name="NAME" x="-80.01" y="116.84" size="1.778" layer="95" rot="R90"/>
-<attribute name="VALUE" x="-71.12" y="116.84" size="1.778" layer="96" rot="R90"/>
+<instance part="Q1" gate="G$1" x="-78.74" y="121.92" smashed="yes" rot="R90">
+<attribute name="NAME" x="-82.55" y="116.84" size="1.778" layer="95" rot="R90"/>
+<attribute name="VALUE" x="-73.66" y="116.84" size="1.778" layer="96" rot="R90"/>
 </instance>
 <instance part="P+8" gate="1" x="-93.98" y="96.52" smashed="yes" rot="R90">
@@
 <attribute name="NAME" x="-142.24" y="165.862" size="1.524" layer="95" rot="R180"/>
 </instance>
-<instance part="C3" gate="G$1" x="-93.98" y="124.46" smashed="yes">
-<attribute name="NAME" x="-92.456" y="124.841" size="1.778" layer="95"/>
-<attribute name="VALUE" x="-92.456" y="119.761" size="1.778" layer="96"/>
-</instance>
-<instance part="C4" gate="G$1" x="-86.36" y="114.3" smashed="yes">
-<attribute name="NAME" x="-84.836" y="114.681" size="1.778" layer="95"/>
-<attribute name="VALUE" x="-84.836" y="109.601" size="1.778" layer="96"/>
-</instance>
-<instance part="GND13" gate="1" x="-86.36" y="106.68" smashed="yes">
-<attribute name="VALUE" x="-88.9" y="104.14" size="1.778" layer="96"/>
+<instance part="C3" gate="G$1" x="-99.06" y="127" smashed="yes" rot="R270">
+<attribute name="NAME" x="-98.679" y="125.476" size="1.778" layer="95" rot="R270"/>
+<attribute name="VALUE" x="-103.759" y="125.476" size="1.778" layer="96" rot="R270"/>
+</instance>
+<instance part="C4" gate="G$1" x="-99.06" y="116.84" smashed="yes" rot="R270">
+<attribute name="NAME" x="-98.679" y="115.316" size="1.778" layer="95" rot="R270"/>
+<attribute name="VALUE" x="-103.759" y="115.316" size="1.778" layer="96" rot="R270"/>
+</instance>
+<instance part="GND13" gate="1" x="-104.14" y="111.76" smashed="yes">
+<attribute name="VALUE" x="-106.68" y="109.22" size="1.778" layer="96"/>
 </instance>
 <instance part="R1" gate="G$1" x="-76.2" y="139.7" smashed="yes">
@@
 <instance part="P+34" gate="1" x="83.82" y="236.22" smashed="yes" rot="R270">
 <attribute name="VALUE" x="78.74" y="238.76" size="1.778" layer="96"/>
+</instance>
+<instance part="R19" gate="G$1" x="-88.9" y="121.92" smashed="yes" rot="R90">
+<attribute name="NAME" x="-90.3986" y="118.11" size="1.778" layer="95" rot="R90"/>
+<attribute name="VALUE" x="-85.598" y="118.11" size="1.778" layer="96" rot="R90"/>
+</instance>
+<instance part="R20" gate="G$1" x="-71.12" y="116.84" smashed="yes" rot="R180">
+<attribute name="NAME" x="-67.31" y="115.3414" size="1.778" layer="95" rot="R180"/>
+<attribute name="VALUE" x="-67.31" y="120.142" size="1.778" layer="96" rot="R180"/>
 </instance>
 </instances>
@@
 <pinref part="GND12" gate="1" pin="GND"/>
 <wire x1="-12.7" y1="147.32" x2="-15.24" y2="147.32" width="0.1524" layer="91"/>
-</segment>
-<segment>
-<pinref part="C4" gate="G$1" pin="2"/>
-<pinref part="GND13" gate="1" pin="GND"/>
-<pinref part="C3" gate="G$1" pin="2"/>
-<wire x1="-93.98" y1="119.38" x2="-93.98" y2="109.22" width="0.1524" layer="91"/>
-<wire x1="-93.98" y1="109.22" x2="-86.36" y2="109.22" width="0.1524" layer="91"/>
-<junction x="-86.36" y="109.22"/>
 </segment>
 <segment>
@@
 <pinref part="J1" gate="G$1" pin="1"/>
 <pinref part="GND24" gate="1" pin="GND"/>
+</segment>
+<segment>
+<pinref part="GND13" gate="1" pin="GND"/>
+<pinref part="C4" gate="G$1" pin="2"/>
+<wire x1="-104.14" y1="114.3" x2="-104.14" y2="116.84" width="0.1524" layer="91"/>
+<pinref part="C3" gate="G$1" pin="2"/>
+<wire x1="-104.14" y1="127" x2="-104.14" y2="116.84" width="0.1524" layer="91"/>
+<junction x="-104.14" y="116.84"/>
 </segment>
 </net>
@@
 <wire x1="-68.58" y1="121.92" x2="-68.58" y2="127" width="0.1524" layer="91"/>
 <pinref part="Q1" gate="G$1" pin="2"/>
-<wire x1="-68.58" y1="127" x2="-76.2" y2="127" width="0.1524" layer="91"/>
+<wire x1="-68.58" y1="127" x2="-78.74" y2="127" width="0.1524" layer="91"/>
 <pinref part="C3" gate="G$1" pin="1"/>
-<wire x1="-93.98" y1="127" x2="-76.2" y2="127" width="0.1524" layer="91"/>
-<junction x="-76.2" y="127"/>
+<wire x1="-96.52" y1="127" x2="-88.9" y2="127" width="0.1524" layer="91"/>
+<junction x="-78.74" y="127"/>
+<pinref part="R19" gate="G$1" pin="2"/>
+<wire x1="-88.9" y1="127" x2="-78.74" y2="127" width="0.1524" layer="91"/>
+<junction x="-88.9" y="127"/>
 </segment>
 </net>
@@
 <pinref part="C4" gate="G$1" pin="1"/>
 <pinref part="Q1" gate="G$1" pin="1"/>
-<wire x1="-86.36" y1="116.84" x2="-76.2" y2="116.84" width="0.1524" layer="91"/>
-<pinref part="IC3" gate="G$1" pin="XTAL1"/>
-<wire x1="-63.5" y1="116.84" x2="-76.2" y2="116.84" width="0.1524" layer="91"/>
-<junction x="-76.2" y="116.84"/>
+<wire x1="-96.52" y1="116.84" x2="-88.9" y2="116.84" width="0.1524" layer="91"/>
+<pinref part="R20" gate="G$1" pin="2"/>
+<wire x1="-88.9" y1="116.84" x2="-78.74" y2="116.84" width="0.1524" layer="91"/>
+<wire x1="-76.2" y1="116.84" x2="-78.74" y2="116.84" width="0.1524" layer="91"/>
+<junction x="-78.74" y="116.84"/>
+<pinref part="R19" gate="G$1" pin="1"/>
+<junction x="-88.9" y="116.84"/>
 </segment>
 </net>
@@
 </segment>
 </net>
+<net name="N$35" class="0">
+<segment>
+<pinref part="R20" gate="G$1" pin="1"/>
+<pinref part="IC3" gate="G$1" pin="XTAL1"/>
+<wire x1="-66.04" y1="116.84" x2="-63.5" y2="116.84" width="0.1524" layer="91"/>
+</segment>
+</net>

Commit message: f
Parts:
- removed X6: 22-23-2041, con-molex:22-23-2041
- added X4: 22-23-2051, con-molex:22-23-2051
Connections:
- new net N$27: IC4.O1, X4-1.S
- net +5V: now also X4-4.S; no longer X6-3.S
- net GND: now also X4-5.S; no longer X6-4.S
- net N$15: now also X4-2.S; no longer X6-1.S
- net N$21: now also X4-3.S; no longer X6-2.S
- net PF5: now also IC4.I2; no longer J3.10
- net PF6: no longer J5.10
- net PG5: now also IC4.I1; no longer IC4.I2

Commit message: f
Parts:
- removed J1: (no value), SparkFun-Connectors:CONN_04
- added X5: TSW-102-07-G-D, con-samtec:TSW-102-07-G-D
Connections:
- net +5V: now also X5-3.1; no longer J1.4
- net GND: now also X5-4.1; no longer J1.1
- net PE0: now also X5-2.1; no longer J1.2
- net PE1: now also X5-1.1; no longer J1.3
Changed lines of the file:
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@@
 <part name="J8" library="SamacSys_Parts" deviceset="615016137621" device=""/>
 <part name="R12" library="rcl" library_urn="urn:adsk.eagle:library:334" deviceset="R-EU_" device="R1210" package3d_urn="urn:adsk.eagle:package:23554/2" value="120"/>
-<part name="J1" library="SparkFun-Connectors" library_urn="urn:adsk.eagle:library:513" deviceset="CONN_04" device="" package3d_urn="urn:adsk.eagle:package:38085/1"/>
 <part name="GND24" library="supply1" library_urn="urn:adsk.eagle:library:371" deviceset="GND" device=""/>
 <part name="P+34" library="supply1" library_urn="urn:adsk.eagle:library:371" deviceset="+5V" device=""/>
@@
 <part name="R20" library="rcl" library_urn="urn:adsk.eagle:library:334" deviceset="R-EU_" device="R0805" package3d_urn="urn:adsk.eagle:package:23553/2" value="27"/>
 <part name="X4" library="con-molex" library_urn="urn:adsk.eagle:library:165" deviceset="22-23-2051" device=""/>
+<part name="X5" library="con-samtec" library_urn="urn:adsk.eagle:library:184" deviceset="TSW-102-*-G" device="-D" technology="07"/>
 </parts>
 <sheets>
@@
 <attribute name="VALUE" x="123.19" y="179.578" size="1.778" layer="96"/>
 </instance>
-<instance part="J1" gate="G$1" x="76.2" y="231.14" smashed="yes">
-<attribute name="VALUE" x="71.12" y="223.774" size="1.778" layer="96" font="vector"/>
-<attribute name="NAME" x="71.12" y="239.268" size="1.778" layer="95" font="vector"/>
-</instance>
 <instance part="GND24" gate="1" x="81.28" y="226.06" smashed="yes">
 <attribute name="VALUE" x="78.74" y="223.52" size="1.778" layer="96"/>
@@
 <instance part="X4" gate="-5" x="-139.7" y="165.1" smashed="yes" rot="R180">
 <attribute name="NAME" x="-142.24" y="165.862" size="1.524" layer="95" rot="R180"/>
+</instance>
+<instance part="X5" gate="-1" x="78.74" y="231.14" smashed="yes" rot="R180">
+<attribute name="VALUE" x="90.17" y="245.11" size="1.778" layer="96" rot="R180"/>
+<attribute name="NAME" x="76.2" y="231.902" size="1.524" layer="95" rot="R180"/>
+</instance>
+<instance part="X5" gate="-2" x="78.74" y="233.68" smashed="yes" rot="R180">
+<attribute name="NAME" x="76.2" y="234.442" size="1.524" layer="95" rot="R180"/>
+</instance>
+<instance part="X5" gate="-3" x="78.74" y="236.22" smashed="yes" rot="R180">
+<attribute name="NAME" x="76.2" y="236.982" size="1.524" layer="95" rot="R180"/>
+</instance>
+<instance part="X5" gate="-4" x="78.74" y="228.6" smashed="yes" rot="R180">
+<attribute name="NAME" x="76.2" y="229.362" size="1.524" layer="95" rot="R180"/>
 </instance>
 </instances>
@@
 </segment>
 <segment>
-<pinref part="J1" gate="G$1" pin="1"/>
-<pinref part="GND24" gate="1" pin="GND"/>
-</segment>
-<segment>
 <pinref part="GND13" gate="1" pin="GND"/>
 <pinref part="C4" gate="G$1" pin="2"/>
@@
 <pinref part="GND20" gate="1" pin="GND"/>
 <pinref part="X4" gate="-5" pin="S"/>
+</segment>
+<segment>
+<pinref part="GND24" gate="1" pin="GND"/>
+<pinref part="X5" gate="-4" pin="1"/>
 </segment>
 </net>
@@
 </segment>
 <segment>
-<pinref part="J1" gate="G$1" pin="4"/>
 <pinref part="P+34" gate="1" pin="+5V"/>
+<pinref part="X5" gate="-3" pin="1"/>
 </segment>
 </net>
@@
 </segment>
 <segment>
-<pinref part="J1" gate="G$1" pin="3"/>
-<wire x1="81.28" y1="233.68" x2="91.44" y2="233.68" width="0.1524" layer="91"/>
-<label x="86.36" y="233.68" size="1.778" layer="95"/>
+<wire x1="81.28" y1="231.14" x2="91.44" y2="231.14" width="0.1524" layer="91"/>
+<label x="86.36" y="231.14" size="1.778" layer="95"/>
+<pinref part="X5" gate="-1" pin="1"/>
 </segment>
 </net>
@@
 </segment>
 <segment>
-<pinref part="J1" gate="G$1" pin="2"/>
-<wire x1="81.28" y1="231.14" x2="91.44" y2="231.14" width="0.1524" layer="91"/>
-<label x="86.36" y="231.14" size="1.778" layer="95"/>
-</segment>
-</net>
+<wire x1="81.28" y1="233.68" x2="91.44" y2="233.68" width="0.1524" layer="91"/>
+<label x="86.36" y="233.68" size="1.778" layer="95"/>
+<pinref part="X5" gate="-2" pin="1"/>
+</segment>
+</net>

Commit message: e
Connections:
- net PE3: now also IC4.I1
- net PG5: no longer IC4.I1
Changed lines of the file:
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@@
 <label x="12.7" y="-10.16" size="1.778" layer="95"/>
-</segment>
-<segment>
-<pinref part="IC4" gate="A" pin="I1"/>
-<wire x1="-210.82" y1="193.04" x2="-220.98" y2="193.04" width="0.1524" layer="91"/>
-<label x="-220.98" y="193.04" size="1.778" layer="95"/>
 </segment>
 </net>
@@
 <label x="30.48" y="25.4" size="1.778" layer="95"/>
 </segment>
+<segment>
+<pinref part="IC4" gate="A" pin="I1"/>
+<wire x1="-210.82" y1="193.04" x2="-220.98" y2="193.04" width="0.1524" layer="91"/>
+<label x="-220.98" y="193.04" size="1.778" layer="95"/>
+</segment>
 </net>
