File: extruderController/winderController.sch (EAGLE design)
At the start: 0 parts

Commit message: V
Parts:
- added IC1: MEGA32-A, atmel:MEGA32-A
- added X1, X2: 22-23-2051, con-molex:22-23-2051
- added X3, X4: 22-23-2031, con-molex:22-23-2031
Connections:
- new net N$1: IC1.(ADC7)PA7
- new net N$10: IC1.(MISO)PB6
- new net N$11: IC1.(MOSI)PB5
- new net N$12: IC1.(SS)PB4
- new net N$13: IC1.(AIN1/OC0)PB3
- new net N$14: IC1.(AIN0/INT2)PB2
- new net N$15: IC1.(T1)PB1
- new net N$16: IC1.(T0/XCK)PB0
- new net N$17: IC1.(TOSC2)PC7
- new net N$18: IC1.(TOSC1)PC6
- new net N$19: IC1.(TDI)PC5
- new net N$2: IC1.(ADC6)PA6
- new net N$20: IC1.(TDO)PC4
- new net N$21: IC1.(TMS)PC3
- new net N$22: IC1.(TCK)PC2
- new net N$23: IC1.PC1(SDA)
- new net N$24: IC1.PC0(SCL)
- new net N$25: IC1.(OC2)PD7
- new net N$26: IC1.(ICP)PD6
- new net N$27: IC1.(OC1A)PD5
- new net N$28: IC1.(OC1B)PD4
- new net N$29: IC1.(INT1)PD3
- new net N$3: IC1.(ADC5)PA5
- new net N$30: IC1.(INT0)PD2
- new net N$31: IC1.(TXD)PD1
- new net N$32: IC1.(RXD)PD0
- new net N$33: X1-1.S
- new net N$34: X1-2.S
- new net N$35: X1-3.S
- new net N$36: X1-4.S
- new net N$37: X1-5.S
- new net N$38: X2-1.S
- new net N$39: X2-2.S
- new net N$4: IC1.(ADC4)PA4
- new net N$40: X2-3.S
- new net N$41: X2-4.S
- new net N$42: X2-5.S
- new net N$43: X3-1.S
- new net N$44: X3-2.S
- new net N$45: X3-3.S
- new net N$46: X4-1.S
- new net N$47: X4-2.S
- new net N$48: X4-3.S
- new net N$5: IC1.(ADC3)PA3
- new net N$6: IC1.(ADC2)PA2
- new net N$7: IC1.(ADC1)PA1
- new net N$8: IC1.(ADC0)PA0
- new net N$9: IC1.(SCK)PB7
Other:
- note added: "Tension sensor"
- note added: "Winding drive motor control"
- note removed: "Manual winder control buttons"
- note removed: "Winding drive motor control 1"
- note removed: "Winding drive motor control 2"
