File: extruderController/winderController02.brd (EAGLE design)
At the start: 70.3 x 60.2 mm, 42 parts, among them IC1 LM1117MPX-5.0, IC2 MAX3467CPA, IC3 MEGA32-A, IC4 ULN2003AD, J8 615016137621, X1 22-23-2051, X2 22-23-2051, X5 TSW-102-07-G-D, X8 22-23-2031, X9 22-23-2031

Commit message: s
Parts:
- removed J6: (no value), SparkFun-Connectors:1X11
- moved C14 100.5 mm to (26.9, 31.0)
- moved C13 84.1 mm to (15.7, 30.7)
- moved C12 79.0 mm to (23.1, 59.4)
- moved J2 14.0 mm to (4.06, 64.8), turned to 90 degrees
- moved R18 13.5 mm to (50.0, 57.9), turned to 180 degrees
- moved D1 11.7 mm to (13.5, 73.4), turned to 180 degrees
- moved X8 11.2 mm to (24.6, 26.2)
- moved X9 11.0 mm to (13.7, 26.2)
- moved SV1 9.52 mm to (15.0, 55.9)
- moved J8 8.64 mm to (34.8, 77.7)
- moved J3 8.14 mm to (63.5, 42.2)
- moved J5 8.14 mm to (66.5, 42.2)
- moved LED1 8.13 mm to (50.0, 55.4), turned to 180 degrees
- moved C16 7.79 mm to (4.83, 52.6), turned to 0 degrees
- moved IC2 6.20 mm to (26.2, 55.9)
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Connections:
- removed net N$13: IC3.44
- removed net N$14: IC3.43
- removed net N$15: IC3.42
- removed net N$16: IC3.41
- removed net N$2: IC3.30
- removed net N$21: IC3.40
- removed net N$22: IC3.26
- removed net N$23: IC3.25
- removed net N$25: IC3.24
- removed net N$26: IC3.23
- removed net N$27: IC3.22
- removed net N$3: IC3.31
- removed net N$30: IC3.19
- removed net N$31: IC3.16
- removed net N$32: IC3.15
- removed net N$33: IC3.14
- removed net N$34: IC3.13
- removed net N$36: IC3.12
- removed net N$38: IC3.11
- removed net N$4: IC3.32
- removed net N$5: IC3.33
- removed net N$6: IC3.34
- removed net N$7: IC3.35
- removed net N$8: IC3.36
- removed net PE0: X5.2
- removed net PE1: X5.1
- removed net PE3: IC4.1
- removed net PE6: X9.2
- removed net PE7: X8.2
- removed net PF5: IC4.2
- removed net PF7: IC4.3
- new net N$10: IC4.12, X1.4
- new net N$11: IC4.13, X1.5
- new net N$12: IC4.14, X2.3
- new net PA4: IC3.33, J3.10
- new net PA5: IC3.32, J3.9
- new net PA6: IC3.31, J3.8
- new net PA7: IC3.30, J3.7
- new net PB0: IC3.40, J5.6
- new net PB1: IC3.41, J5.5
- new net PB2: IC3.42, J5.4
- new net PB3: IC3.43, J5.3
- new net PB4: IC3.44, J5.2
- new net PC0: IC3.19, IC4.6
- new net PC1: IC3.20, IC4.5
- new net PC2: IC3.21, IC4.3
- new net PC3: IC3.22, J3.2
- new net PC4: IC3.23, J3.3
- new net PC5: IC3.24, J3.4
- new net PC6: IC3.25, J3.5
- new net PC7: IC3.26, J3.6
- new net PD2: IC3.11, X9.2
- new net PD3: IC3.12, J5.1
- new net PD4: IC3.13, J3.1
- new net PD5: IC3.14, IC4.4
- new net PD6: IC3.15, IC4.2
- new net PD7: IC3.16, IC4.1
- net +5V: now also J3.11, X1.2, X2.2
- net GND: now also IC4.7, J5.10, J5.11, X1.1, X2.1
- net N$28: now also IC4.15, X2.4; no longer IC3.21
- net N$29: now also IC4.16, X2.5; no longer IC3.20
- net N$9: now also IC4.11, X1.3; no longer IC3.37
- net PA0: now also IC3.37, X8.2; no longer IC4.4
- net PA1: now also IC3.36, J5.7; no longer IC4.5
- net PA2: now also IC3.35, J5.8; no longer IC4.6
- net PA3: now also IC3.34, J5.9; no longer IC4.7
- net PD0: now also X5.2
- net PD1: now also X5.1
Routing:
- net +5V: track 45.5 -> 238.5 mm, vias 0 -> 6
- net PD3: track 0.00 -> 57.6 mm, vias 0 -> 1
- net PB4: track 0.00 -> 56.7 mm, vias 0 -> 1
- net PB3: track 0.00 -> 53.7 mm, vias 0 -> 1
- net PD4: track 0.00 -> 53.5 mm, vias 0 -> 1
- net PB0: track 0.00 -> 51.8 mm, vias 0 -> 1
- net PB2: track 0.00 -> 51.8 mm, vias 0 -> 1
- net PA3: track 0.00 -> 51.3 mm, vias 0 -> 1
- net PA2: track 0.00 -> 51.3 mm, vias 0 -> 1
- net PB1: track 0.00 -> 51.2 mm, vias 0 -> 1
- net PA1: track 0.00 -> 50.8 mm, vias 0 -> 1
- net PA4: track 0.00 -> 47.6 mm
- net PA5: track 0.00 -> 46.0 mm
- net PD0: track 0.00 -> 45.3 mm, vias 0 -> 3
- net PD1: track 0.00 -> 44.9 mm, vias 0 -> 3
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- added copper zone on layer 1, net +5V
- added copper zone on layer 1, net GND
- added copper zone on layer 16, net GND
Other:
- board size 70.3 x 60.2 mm -> 70.3 x 57.4 mm
- board text added: "2019"
- board text added: "Endstop"
- board text added: "Krists"
- board text added: "Pudzens"
- board text added: "Tension"

Commit message: c
Routing:
- net GND: track 31.2 -> 25.5 mm, vias 32 -> 35
- net +5V: track 238.5 -> 243.7 mm, vias 6 -> 10
- net N$19: track 16.1 -> 14.8 mm
- net PA0: track 31.1 -> 31.8 mm
Other:
- board text added: "+5V"
- board text added: "DIR"
- board text added: "ENA"
- board text added: "GND"
- board text added: "STEP"

Commit message: h
Parts:
- moved LED1 6.93 mm to (56.1, 52.1)
- moved R18 5.93 mm to (51.1, 52.1), turned to 0 degrees
- moved X5 4.07 mm to (47.0, 56.4)
- moved C13 2.81 mm to (18.5, 31.0), turned to 90 degrees
- moved C14 2.54 mm to (29.5, 31.0), turned to 90 degrees
- moved C1 0.92 mm to (14.0, 66.3), turned to 180 degrees
- moved Q1 0.51 mm to (7.11, 38.1)
Connections:
- removed net PF6: R18.1
- net PA4: now also R18.1
Routing:
- net +5V: track 243.7 -> 248.8 mm
- net PD1: track 44.9 -> 49.1 mm
- net PD0: track 45.3 -> 49.5 mm
- net PA4: track 47.6 -> 50.9 mm
- net N$20: track 11.2 -> 10.7 mm
- net N$19: track 14.8 -> 14.3 mm
- net GND: vias 35 -> 43
Other:
- board text added: "5V"
- board text added: "ATMEGA32"
- board text added: "ENDSTOP"
- board text added: "MISO"
- board text added: "Mot1"
- board text added: "Mot2"
- board text added: "RESET"
- board text added: "RS485"
- board text added: "RX"
- board text added: "SCK"
- board text added: "TENS."
- board text added: "TX"
- board text added: "UART"
- board text removed: "Endstop"
- board text removed: "Tension"
