File: extruderController/winderController02.sch (EAGLE design)
At the start: 42 parts, among them IC1 LM1117MPX-5.0, IC2 MAX3467CPA, IC3 MEGA32-A, IC4 ULN2003AD, J8 615016137621, X1 22-23-2051, X2 22-23-2051, X5 TSW-102-07-G-D, X8 22-23-2031, X9 22-23-2031

Commit message: s
Parts:
- removed J6: (no value), SparkFun-Connectors:CONN_11
Connections:
- removed net N$13: IC3.(SS)PB4
- removed net N$14: IC3.(AIN1/OC0)PB3
- removed net N$15: IC3.(AIN0/INT2)PB2
- removed net N$16: IC3.(T1)PB1
- removed net N$2: IC3.(ADC7)PA7
- removed net N$21: IC3.(T0/XCK)PB0
- removed net N$22: IC3.(TOSC2)PC7
- removed net N$23: IC3.(TOSC1)PC6
- removed net N$25: IC3.(TDI)PC5
- removed net N$26: IC3.(TDO)PC4
- removed net N$27: IC3.(TMS)PC3
- removed net N$3: IC3.(ADC6)PA6
- removed net N$30: IC3.PC0(SCL)
- removed net N$31: IC3.(OC2)PD7
- removed net N$32: IC3.(ICP)PD6
- removed net N$33: IC3.(OC1A)PD5
- removed net N$34: IC3.(OC1B)PD4
- removed net N$36: IC3.(INT1)PD3
- removed net N$38: IC3.(INT0)PD2
- removed net N$4: IC3.(ADC5)PA5
- removed net N$5: IC3.(ADC4)PA4
- removed net N$6: IC3.(ADC3)PA3
- removed net N$7: IC3.(ADC2)PA2
- removed net N$8: IC3.(ADC1)PA1
- removed net PE0: X5-2.1
- removed net PE1: X5-1.1
- removed net PE3: IC4.I1
- removed net PE6: X9-2.S
- removed net PE7: X8-2.S
- removed net PF5: IC4.I2
- removed net PF7: IC4.I3
- new net N$10: IC4.O5, X1-4.S
- new net N$11: IC4.O4, X1-5.S
- new net N$12: IC4.O3, X2-3.S
- new net PA4: IC3.(ADC4)PA4, J3.10
- new net PA5: IC3.(ADC5)PA5, J3.9
- new net PA6: IC3.(ADC6)PA6, J3.8
- new net PA7: IC3.(ADC7)PA7, J3.7
- new net PB0: IC3.(T0/XCK)PB0, J5.6
- new net PB1: IC3.(T1)PB1, J5.5
- new net PB2: IC3.(AIN0/INT2)PB2, J5.4
- new net PB3: IC3.(AIN1/OC0)PB3, J5.3
- new net PB4: IC3.(SS)PB4, J5.2
- new net PC0: IC3.PC0(SCL), IC4.I6
- new net PC1: IC3.PC1(SDA), IC4.I5
- new net PC2: IC3.(TCK)PC2, IC4.I3
- new net PC3: IC3.(TMS)PC3, J3.2
- new net PC4: IC3.(TDO)PC4, J3.3
- new net PC5: IC3.(TDI)PC5, J3.4
- new net PC6: IC3.(TOSC1)PC6, J3.5
- new net PC7: IC3.(TOSC2)PC7, J3.6
- new net PD2: IC3.(INT0)PD2, X9-2.S
- new net PD3: IC3.(INT1)PD3, J5.1
- new net PD4: IC3.(OC1B)PD4, J3.1
- new net PD5: IC3.(OC1A)PD5, IC4.I4
- new net PD6: IC3.(ICP)PD6, IC4.I2
- new net PD7: IC3.(OC2)PD7, IC4.I1
- net +5V: now also J3.11, X1-2.S, X2-2.S
- net GND: now also IC4.I7, J5.10, J5.11, X1-1.S, X2-1.S
- net N$28: now also IC4.O2, X2-4.S; no longer IC3.(TCK)PC2
- net N$29: now also IC4.O1, X2-5.S; no longer IC3.PC1(SDA)
- net N$9: now also IC4.O6, X1-3.S; no longer IC3.(ADC0)PA0
- net PA0: now also IC3.(ADC0)PA0, X8-2.S; no longer IC4.I4
- net PA1: now also IC3.(ADC1)PA1, J5.7; no longer IC4.I5
- net PA2: now also IC3.(ADC2)PA2, J5.8; no longer IC4.I6
- net PA3: now also IC3.(ADC3)PA3, J5.9; no longer IC4.I7
- net PD0: now also X5-2.1
- net PD1: now also X5-1.1
Other:
- moved on the sheet: H1, H2, H3, H4, X1-1, X1-2, X1-3, X1-4, X1-5, X2-1, X2-2, X2-3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

Commit message: h
Connections:
- removed net PF6: R18.1
- net PA4: now also R18.1
Other:
- note added: "Stepper1, Stepper2"
- note removed: "Heater SSR output x4"
- note removed: "Main stepper control output"
Changed lines of the file:
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@@
 <text x="-106.68" y="218.44" size="5.08" layer="91">Power supply, 12V in, 5vout</text>
 <text x="-106.68" y="160.02" size="5.08" layer="95">ATMEGA</text>
-<text x="-243.84" y="218.44" size="5.08" layer="91">Heater SSR output x4</text>
-<text x="-243.84" y="210.82" size="5.08" layer="91">Main stepper control output</text>
+<text x="-243.84" y="215.9" size="5.08" layer="91">Stepper1, Stepper2</text>
 <text x="66.04" y="76.2" size="5.08" layer="91">End stop</text>
 <text x="66.04" y="256.54" size="5.08" layer="91">RS485 communication</text>
@@
 </segment>
 </net>
-<net name="PF6" class="0">
-<segment>
-<pinref part="R18" gate="G$1" pin="1"/>
-<wire x1="30.48" y1="185.42" x2="30.48" y2="177.8" width="0.1524" layer="91"/>
-<label x="30.48" y="177.8" size="1.778" layer="95"/>
-</segment>
-</net>
 <net name="N$24" class="0">
 <segment>
@@
 <label x="121.92" y="121.92" size="1.778" layer="95"/>
 </segment>
-</net>
+<segment>
+<pinref part="R18" gate="G$1" pin="1"/>
+<wire x1="30.48" y1="185.42" x2="30.48" y2="177.8" width="0.1524" layer="91"/>
+<label x="30.48" y="177.8" size="1.778" layer="95"/>
+</segment>
+</net>
