File: wsleddriver/leddriver.sch (EAGLE design)
At the start: 4 parts, among them IC1 WS2811-SOP8

Commit message: h
Parts:
- removed INPUT, OUTPUT: (no value), SparkFun-Connectors:CONN_03LONGPADS
- added C1: (no value), rcl:C-EUC1206
- added IN/OUT: (no value), SparkFun-Connectors:CONN_04LONGPADS
- added R1: 33, rcl:R-EU_R0805
- added R2: 2.7K, rcl:R-EU_R0805
- added R3, R5, R7: 100, rcl:R-EU_R0805
- added R4, R6, R8: 10K, rcl:R-EU_R0805
- added TB, TG, TR: 5.8A/30V/35mΩ, SparkFun-DiscreteSemi:MOSFET-NCH-AO3404A
Connections:
- new net B: IC1.B, R7.1
- new net DIN_IN: IN/OUT.3, R1.2
- new net DOUT_OUT: IC1.DO, IN/OUT.2
- new net G: IC1.G, R5.1
- new net N$1: IC1.DIN, R1.1
- new net N$2: R5.2, R6.2, TG.G
- new net N$3: R7.2, R8.2, TB.G
- new net N$5: R3.2, R4.2, TR.G
- new net NEG_B: LEDSTRIP.1, TB.D
- new net NEG_G: LEDSTRIP.2, TG.D
- new net NEG_R: LEDSTRIP.3, TR.D
- new net R: IC1.R, R3.1
- new net VDD: C1.2, IC1.VDD, R2.1
- net +12V: now also IN/OUT.4, LEDSTRIP.4, R2.2, R4.1, R6.1, R8.1; no longer INPUT.3, OUTPUT.3
- net GND: now also C1.1, IC1.GND, IN/OUT.1, TB.S, TG.S, TR.S; no longer INPUT.1, OUTPUT.1
Other:
- moved on the sheet: IC1

Commit message: a
Parts:
- removed LEDSTRIP: (no value), SparkFun-Connectors:CONN_04LONGPADS
- removed R1: 33, rcl:R-EU_R0805
- removed R2: 2.7K, rcl:R-EU_R0805
- added JP1: (no value), pinhead:PINHD-1X3
- added R10: 100, rcl:R-EU_R0805
- added R9: 10k, rcl:R-EU_R0805
- R3: value 100 -> 10k
- R4: value 10K -> 10k
- R6: value 10K -> 100
- R7: value 100 -> 2.7k
- R8: value 10K -> 33
Connections:
- removed net N$5: R3.2, R4.2, TR.G
- new net N$4: R10.2, R9.2, TR.G
- net +12V: now also R3.1, R7.2, R9.1; no longer LEDSTRIP.4, R2.2, R6.1, R8.1
- net B: now also R6.1; no longer R7.1
- net DIN_IN: now also R8.2; no longer R1.2
- net N$1: now also R8.1; no longer R1.1
- net N$2: now also R3.2; no longer R6.2
- net N$3: now also R4.2, R6.2; no longer R7.2, R8.2
- net NEG_B: now also JP1.1; no longer LEDSTRIP.1
- net NEG_G: now also JP1.2; no longer LEDSTRIP.2
- net NEG_R: now also JP1.3; no longer LEDSTRIP.3
- net R: now also R10.1; no longer R3.1
- net VDD: now also R7.1; no longer R2.1
Other:
- moved on the sheet: R3, R4, R6, R7, R8

Commit message: f
Parts:
- removed JP1: (no value), pinhead:PINHD-1X3
- added PAD1, PAD2, PAD3: (no value), wirepad:3,81/1,4
- C1: value (none) -> 0.1uF
Connections:
- net NEG_B: now also PAD3.P; no longer JP1.1
- net NEG_G: now also PAD2.P; no longer JP1.2
- net NEG_R: now also PAD1.P; no longer JP1.3
Changed lines of the file:
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@@
 <?xml version="1.0" encoding="utf-8"?>
 <!DOCTYPE eagle SYSTEM "eagle.dtd">
-<eagle version="9.2.2">
+<eagle version="9.3.1">
 <drawing>
 <settings>
@@
 <part name="P+3" library="supply1" library_urn="urn:adsk.eagle:library:371" deviceset="+12V" device=""/>
 <part name="GND3" library="supply1" library_urn="urn:adsk.eagle:library:371" deviceset="GND" device=""/>
-<part name="C1" library="rcl" library_urn="urn:adsk.eagle:library:334" deviceset="C-EU" device="C1206" package3d_urn="urn:adsk.eagle:package:23618/2"/>
+<part name="C1" library="rcl" library_urn="urn:adsk.eagle:library:334" deviceset="C-EU" device="C1206" package3d_urn="urn:adsk.eagle:package:23618/2" value="0.1uF"/>
 <part name="GND4" library="supply1" library_urn="urn:adsk.eagle:library:371" deviceset="GND" device=""/>
 <part name="TR" library="SparkFun-DiscreteSemi" library_urn="urn:adsk.eagle:library:514" deviceset="MOSFET-NCH" device="-AO3404A" package3d_urn="urn:adsk.eagle:package:38446/1" value="5.8A/30V/35mΩ"/>
@@
 <part name="R7" library="rcl" library_urn="urn:adsk.eagle:library:334" deviceset="R-EU_" device="R0805" package3d_urn="urn:adsk.eagle:package:23553/2" value="2.7k"/>
 <part name="R8" library="rcl" library_urn="urn:adsk.eagle:library:334" deviceset="R-EU_" device="R0805" package3d_urn="urn:adsk.eagle:package:23553/2" value="33"/>
-<part name="JP1" library="pinhead" library_urn="urn:adsk.eagle:library:325" deviceset="PINHD-1X3" device="" package3d_urn="urn:adsk.eagle:package:22458/2"/>
+<part name="PAD1" library="wirepad" library_urn="urn:adsk.eagle:library:412" deviceset="3,81/1,4" device="" package3d_urn="urn:adsk.eagle:package:30835/1"/>
+<part name="PAD2" library="wirepad" library_urn="urn:adsk.eagle:library:412" deviceset="3,81/1,4" device="" package3d_urn="urn:adsk.eagle:package:30835/1"/>
+<part name="PAD3" library="wirepad" library_urn="urn:adsk.eagle:library:412" deviceset="3,81/1,4" device="" package3d_urn="urn:adsk.eagle:package:30835/1"/>
 </parts>
 <sheets>
@@
 <attribute name="VALUE" x="100.33" y="52.578" size="1.778" layer="96"/>
 </instance>
-<instance part="JP1" gate="A" x="35.56" y="30.48" smashed="yes" rot="R180">
-<attribute name="NAME" x="41.91" y="24.765" size="1.778" layer="95" rot="R180"/>
-<attribute name="VALUE" x="41.91" y="38.1" size="1.778" layer="96" rot="R180"/>
+<instance part="PAD1" gate="1" x="17.78" y="33.02" smashed="yes">
+<attribute name="NAME" x="16.637" y="34.8742" size="1.778" layer="95"/>
+<attribute name="VALUE" x="16.637" y="29.718" size="1.778" layer="96"/>
+</instance>
+<instance part="PAD2" gate="1" x="17.78" y="27.94" smashed="yes">
+<attribute name="NAME" x="16.637" y="29.7942" size="1.778" layer="95"/>
+<attribute name="VALUE" x="16.637" y="24.638" size="1.778" layer="96"/>
+</instance>
+<instance part="PAD3" gate="1" x="17.78" y="22.86" smashed="yes">
+<attribute name="NAME" x="16.637" y="24.7142" size="1.778" layer="95"/>
+<attribute name="VALUE" x="16.637" y="19.558" size="1.778" layer="96"/>
 </instance>
 </instances>
@@
 </segment>
 <segment>
-<pinref part="JP1" gate="A" pin="3"/>
-<wire x1="38.1" y1="33.02" x2="55.88" y2="33.02" width="0.1524" layer="91"/>
-<label x="48.26" y="33.02" size="1.778" layer="95"/>
+<pinref part="PAD1" gate="1" pin="P"/>
+<wire x1="20.32" y1="33.02" x2="30.48" y2="33.02" width="0.1524" layer="91"/>
+<label x="22.86" y="33.02" size="1.778" layer="95"/>
 </segment>
 </net>
@@
 </segment>
 <segment>
-<pinref part="JP1" gate="A" pin="2"/>
-<wire x1="38.1" y1="30.48" x2="55.88" y2="30.48" width="0.1524" layer="91"/>
-<label x="48.26" y="30.48" size="1.778" layer="95"/>
+<pinref part="PAD2" gate="1" pin="P"/>
+<wire x1="20.32" y1="27.94" x2="30.48" y2="27.94" width="0.1524" layer="91"/>
+<label x="22.86" y="27.94" size="1.778" layer="95"/>
 </segment>
 </net>
@@
 </segment>
 <segment>
-<pinref part="JP1" gate="A" pin="1"/>
-<wire x1="38.1" y1="27.94" x2="55.88" y2="27.94" width="0.1524" layer="91"/>
-<label x="48.26" y="27.94" size="1.778" layer="95"/>
+<pinref part="PAD3" gate="1" pin="P"/>
+<wire x1="20.32" y1="22.86" x2="30.48" y2="22.86" width="0.1524" layer="91"/>
+<label x="22.86" y="22.86" size="1.778" layer="95"/>
 </segment>
 </net>
@@
 <pinref part="R9" gate="G$1" pin="2"/>
 <junction x="0" y="111.76"/>
-<pinref part="R9" gate="G$1" pin="2"/>
 </segment>
 </net>
@@
 <pinref part="R5" gate="G$1" pin="2"/>
 <junction x="55.88" y="111.76"/>
-<pinref part="R5" gate="G$1" pin="2"/>
 </segment>
 </net>
@@
 <pinref part="R6" gate="G$1" pin="2"/>
 <junction x="114.3" y="111.76"/>
-<pinref part="R6" gate="G$1" pin="2"/>
-</segment>
-</net>
+</segment>
+</net>
