File: wsleddriver/leddriver.sch (EAGLE design)
At the start: 19 parts, among them IC1 WS2811-SOP8, X1 TSW-104-07-G-S, X2 TSW-104-07-G-S

Commit message: w
Parts:
- removed X1, X2: TSW-104-07-G-S, con-samtec:TSW-104-07-G-S
Changed lines of the file:
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@@
 <?xml version="1.0" encoding="utf-8"?>
 <!DOCTYPE eagle SYSTEM "eagle.dtd">
-<eagle version="9.2.2">
+<eagle version="9.4.2">
 <drawing>
 <settings>
@@
 <part name="PAD2" library="wirepad" library_urn="urn:adsk.eagle:library:412" deviceset="3,81/1,4" device="" package3d_urn="urn:adsk.eagle:package:30835/1"/>
 <part name="PAD3" library="wirepad" library_urn="urn:adsk.eagle:library:412" deviceset="3,81/1,4" device="" package3d_urn="urn:adsk.eagle:package:30835/1"/>
-<part name="X1" library="con-samtec" library_urn="urn:adsk.eagle:library:184" deviceset="TSW-104-*-G-S" device="" technology="07"/>
-<part name="X2" library="con-samtec" library_urn="urn:adsk.eagle:library:184" deviceset="TSW-104-*-G-S" device="" technology="07"/>
 </parts>
 <sheets>
@@
 <attribute name="VALUE" x="16.637" y="19.558" size="1.778" layer="96"/>
 </instance>
-<instance part="X1" gate="-1" x="-54.61" y="60.96" smashed="yes">
-<attribute name="VALUE" x="-55.88" y="62.23" size="1.778" layer="96"/>
-<attribute name="NAME" x="-52.07" y="60.198" size="1.524" layer="95"/>
-</instance>
-<instance part="X1" gate="-2" x="-54.61" y="58.42" smashed="yes">
-<attribute name="NAME" x="-52.07" y="57.658" size="1.524" layer="95"/>
-</instance>
-<instance part="X1" gate="-3" x="-54.61" y="55.88" smashed="yes">
-<attribute name="NAME" x="-52.07" y="55.118" size="1.524" layer="95"/>
-</instance>
-<instance part="X1" gate="-4" x="-54.61" y="53.34" smashed="yes">
-<attribute name="NAME" x="-52.07" y="52.578" size="1.524" layer="95"/>
-</instance>
-<instance part="X2" gate="-1" x="-54.61" y="43.18" smashed="yes">
-<attribute name="VALUE" x="-55.88" y="44.45" size="1.778" layer="96"/>
-<attribute name="NAME" x="-52.07" y="42.418" size="1.524" layer="95"/>
-</instance>
-<instance part="X2" gate="-2" x="-54.61" y="40.64" smashed="yes">
-<attribute name="NAME" x="-52.07" y="39.878" size="1.524" layer="95"/>
-</instance>
-<instance part="X2" gate="-3" x="-54.61" y="38.1" smashed="yes">
-<attribute name="NAME" x="-52.07" y="37.338" size="1.524" layer="95"/>
-</instance>
-<instance part="X2" gate="-4" x="-54.61" y="35.56" smashed="yes">
-<attribute name="NAME" x="-52.07" y="34.798" size="1.524" layer="95"/>
-</instance>
 </instances>
