File: wsleddriver/leddriver.brd (EAGLE design)
At the start: 35.2 x 13.7 mm, 15 parts, among them IC1 WS2811-SOP8

Commit message: a
Parts:
- removed LEDSTRIP: (no value), SparkFun-Connectors:1X04_LONGPADS
- removed R1: 33, rcl:R0805
- removed R2: 2.7K, rcl:R0805
- added JP1: (no value), pinhead:1X03
- added R10: 100, rcl:R0805
- added R9: 10k, rcl:R0805
- R3: value 100 -> 10k
- R4: value 10K -> 10k
- R6: value 10K -> 100
- R7: value 100 -> 2.7k
- R8: value 10K -> 33
- moved IN/OUT 14.8 mm to (15.6, 2.67), turned to 180 degrees
- moved R8 12.0 mm to (7.37, 10.9), turned to 270 degrees
- moved R7 10.9 mm to (8.13, 6.10), turned to 180 degrees
- moved IC1 6.70 mm to (12.8, 10.2)
- moved R4 6.12 mm to (19.8, 9.91)
- moved R3 4.34 mm to (19.8, 5.84)
- moved R6 4.10 mm to (19.8, 11.9)
- moved C1 3.14 mm to (12.7, 6.10), turned to 180 degrees
- moved R5 2.54 mm to (19.8, 7.87)
- moved TB 2.34 mm to (26.9, 11.4)
- moved TR 2.34 mm to (26.9, 2.29)
- moved TG 2.29 mm to (26.9, 6.86)
Connections:
- removed net N$5: R3.2, R4.2, TR.1
- new net N$4: R10.2, R9.2, TR.1
- net +12V: now also R3.1, R7.2, R9.1; no longer LEDSTRIP.4, R2.2, R6.1, R8.1
- net B: now also R6.1; no longer R7.1
- net DIN_IN: now also R8.2; no longer R1.2
- net N$1: now also R8.1; no longer R1.1
- net N$2: now also R3.2; no longer R6.2
- net N$3: now also R4.2, R6.2; no longer R7.2, R8.2
- net NEG_B: now also JP1.1; no longer LEDSTRIP.1
- net NEG_G: now also JP1.2; no longer LEDSTRIP.2
- net NEG_R: now also JP1.3; no longer LEDSTRIP.3
- net R: now also R10.1; no longer R3.1
- net VDD: now also R7.1; no longer R2.1
Routing:
- net +12V: track 53.5 -> 12.3 mm, vias 4 -> 3
- net VDD: track 10.5 -> 0.00 mm
- net N$4: track 0.00 -> 8.25 mm
- net DOUT_OUT: track 6.66 -> 0.51 mm
- net N$5: track 5.86 -> 0.00 mm
- net DIN_IN: track 4.33 -> 0.00 mm
- net B: track 7.28 -> 3.54 mm
- net R: track 2.84 -> 6.01 mm
- net N$1: track 2.65 -> 0.52 mm
- net N$2: track 5.86 -> 7.92 mm
- net N$3: track 6.57 -> 7.38 mm
- net GND: track 0.32 -> 0.00 mm, vias 2 -> 38
- added copper zone on layer 1, net NEG_B
- added copper zone on layer 1, net NEG_G
- added copper zone on layer 1, net NEG_R
- removed copper zone on layer 16, net +12V
Other:
- board size 35.2 x 13.7 mm -> 29.9 x 14.2 mm

Commit message: f
Parts:
- removed JP1: (no value), pinhead:1X03
- added PAD1, PAD2, PAD3: (no value), wirepad:3,81/1,4
- C1: value (none) -> 0.1uF
- moved R8 1.20 mm to (7.75, 9.78)
- moved C1 0.13 mm to (12.7, 5.97)
- moved R7 0.13 mm to (8.13, 5.97)
Connections:
- net NEG_B: now also PAD3.1; no longer JP1.1
- net NEG_G: now also PAD2.1; no longer JP1.2
- net NEG_R: now also PAD1.1; no longer JP1.3
Routing:
- net +12V: track 12.3 -> 34.1 mm
- net DOUT_OUT: track 0.51 -> 13.1 mm, vias 0 -> 2
- net DIN_IN: track 0.00 -> 9.00 mm, vias 0 -> 2
- net VDD: track 0.00 -> 4.58 mm
- net N$1: track 0.52 -> 2.13 mm
- added copper zone on layer 16, net NEG_B
- added copper zone on layer 16, net NEG_G
- added copper zone on layer 16, net NEG_R
Other:
- board size 29.9 x 14.2 mm -> 29.9 x 14.3 mm
- board text added: "B"
- board text added: "G"
- board text added: "R"
- board text added: "WS2811"

Commit message: c
Parts:
- removed R10: 100, rcl:R0805
- removed R9: 10k, rcl:R0805
- added R1: 10k, rcl:R0805
- added R2: 100, rcl:R0805
- added X1, X2: TSW-104-07-G-S, con-samtec:TSW-104-XX-G-S
- R4: value 10k -> 100
- R5: value 100 -> 10k
- moved R4 2.07 mm to (19.4, 7.87)
- moved R5 2.07 mm to (19.4, 9.91)
- moved R3 0.38 mm to (19.4, 5.84)
- moved R6 0.38 mm to (19.4, 11.9)
Connections:
- net +12V: now also R1.1, R5.1; no longer R4.1, R9.1
- net G: now also R4.1; no longer R5.1
- net N$2: now also R4.2; no longer R5.2
- net N$3: now also R5.2; no longer R4.2
- net N$4: now also R1.2, R2.2; no longer R10.2, R9.2
- net R: now also R2.1; no longer R10.1
Routing:
- net +12V: track 34.1 -> 35.1 mm
Other:
- board text added: "C1"
- board text added: "R1"
- board text added: "R2"
- board text added: "R3"
- board text added: "R4"
- board text added: "R5"
- board text added: "R6"
- board text added: "R7"
- board text added: "R8"

Commit message: w
Parts:
- removed X1, X2: TSW-104-07-G-S, con-samtec:TSW-104-XX-G-S
Other:
- board text added: "100"
- board text added: "10K"
Changed lines of the file:
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@@
 <?xml version="1.0" encoding="utf-8"?>
 <!DOCTYPE eagle SYSTEM "eagle.dtd">
-<eagle version="9.2.2">
+<eagle version="9.4.2">
 <drawing>
 <settings>
@@
 <text x="28.829" y="10.795" size="1.27" layer="25" font="vector" ratio="15">B</text>
 <text x="12.192" y="8.001" size="0.8128" layer="25" font="vector" ratio="15" rot="R90">WS2811</text>
-<text x="17.653" y="1.143" size="0.8128" layer="25" font="vector" ratio="15" rot="R90">R1</text>
-<text x="17.653" y="3.175" size="0.8128" layer="25" font="vector" ratio="15" rot="R90">R2</text>
-<text x="17.653" y="7.239" size="0.8128" layer="25" font="vector" ratio="15" rot="R90">R4</text>
-<text x="17.653" y="9.398" size="0.8128" layer="25" font="vector" ratio="15" rot="R90">R5</text>
-<text x="17.653" y="11.303" size="0.8128" layer="25" font="vector" ratio="15" rot="R90">R6</text>
-<text x="17.653" y="5.334" size="0.8128" layer="25" font="vector" ratio="15" rot="R90">R3</text>
-<text x="15.113" y="5.461" size="0.8128" layer="25" font="vector" ratio="15">C1</text>
+<text x="21.59" y="1.778" size="0.8128" layer="25" font="vector" ratio="15">R1</text>
+<text x="21.59" y="3.81" size="0.8128" layer="25" font="vector" ratio="15">R2</text>
+<text x="21.59" y="7.874" size="0.8128" layer="25" font="vector" ratio="15">R4</text>
+<text x="21.59" y="9.906" size="0.8128" layer="25" font="vector" ratio="15">R5</text>
+<text x="21.59" y="11.938" size="0.8128" layer="25" font="vector" ratio="15">R6</text>
+<text x="21.59" y="5.842" size="0.8128" layer="25" font="vector" ratio="15">R3</text>
+<text x="15.24" y="5.461" size="0.8128" layer="25" font="vector" ratio="15">C1</text>
 <text x="7.239" y="11.557" size="0.8128" layer="25" font="vector" ratio="15">R8</text>
 <text x="6.35" y="6.858" size="0.8128" layer="25" font="vector" ratio="15">R7</text>
+<text x="21.59" y="11.049" size="0.6096" layer="25" font="vector" ratio="15">100</text>
+<text x="21.59" y="9.144" size="0.6096" layer="25" font="vector" ratio="15">10K</text>
+<text x="21.59" y="5.08" size="0.6096" layer="25" font="vector" ratio="15">10K</text>
+<text x="21.59" y="1.016" size="0.6096" layer="25" font="vector" ratio="15">10K</text>
+<text x="21.59" y="7.112" size="0.6096" layer="25" font="vector" ratio="15">100</text>
+<text x="21.59" y="3.048" size="0.6096" layer="25" font="vector" ratio="15">100</text>
 </plain>
 <attributes>
@@
 <attribute name="VALUE" x="32.258" y="12.249" size="0.0254" layer="27"/>
 </element>
-<element name="X1" library="con-samtec" library_urn="urn:adsk.eagle:library:184" package="TSW-104-XX-G-S" value="TSW-104-07-G-S" x="11.811" y="1.524" smashed="yes">
-<attribute name="MF" value="Samtec Inc." x="11.811" y="1.524" size="1.778" layer="27" display="off"/>
-<attribute name="MPN" value="TSW-104-07-G-S" x="11.811" y="1.524" size="1.778" layer="27" display="off"/>
-<attribute name="NAME" x="6.096" y="0.254" size="1.27" layer="25" rot="R90"/>
-<attribute name="OC_FARNELL" value="" x="11.811" y="1.524" size="1.778" layer="27" display="off"/>
-<attribute name="OC_NEWARK" value="" x="11.811" y="1.524" size="1.778" layer="27" display="off"/>
-<attribute name="VALUE" x="18.796" y="0.254" size="1.27" layer="27" rot="R90"/>
-</element>
-<element name="X2" library="con-samtec" library_urn="urn:adsk.eagle:library:184" package="TSW-104-XX-G-S" value="TSW-104-07-G-S" x="11.557" y="12.065" smashed="yes">
-<attribute name="MF" value="Samtec Inc." x="11.557" y="12.065" size="1.778" layer="27" display="off"/>
-<attribute name="MPN" value="TSW-104-07-G-S" x="11.557" y="12.065" size="1.778" layer="27" display="off"/>
-<attribute name="NAME" x="5.842" y="10.795" size="1.27" layer="25" rot="R90"/>
-<attribute name="OC_FARNELL" value="" x="11.557" y="12.065" size="1.778" layer="27" display="off"/>
-<attribute name="OC_NEWARK" value="" x="11.557" y="12.065" size="1.778" layer="27" display="off"/>
-<attribute name="VALUE" x="18.542" y="10.795" size="1.27" layer="27" rot="R90"/>
-</element>
 </elements>
 <signals>
@@
 <contactref element="R3" pad="1"/>
 <contactref element="R5" pad="1"/>
-<wire x1="16.9898" y1="6.858" x2="17.465" y2="6.858" width="0.4064" layer="1"/>
-<wire x1="18.481" y1="5.842" x2="17.465" y2="6.858" width="0.4064" layer="1"/>
+<wire x1="18.227" y1="5.842" x2="17.211" y2="6.858" width="0.4064" layer="1"/>
+<wire x1="16.9898" y1="6.858" x2="17.211" y2="6.858" width="0.4064" layer="1"/>
+<wire x1="18.481" y1="5.842" x2="18.227" y2="5.842" width="0.4064" layer="1"/>
 <via x="16.9898" y="6.858" extent="1-16" drill="0.35"/>
 <wire x1="18.481" y1="9.906" x2="18.354" y2="10.033" width="0.4064" layer="1"/>
