File: wsleddriver/leddriverX3.sch (EAGLE design)
At the start: 40 parts, among them IC1 WS2811-SOP8, IC2 WS2811-SOP8, IC3 WS2811-SOP8

Commit message: c
Parts:
- added PAD1, PAD2, PAD3, PAD4, PAD5, PAD6, PAD7, PAD8, PAD9: (no value), wirepad:SMD5
Connections:
- new net NEG_B2: TB1.D
- new net NEG_B3: TB.D
- new net NEG_G2: TG1.D
- new net NEG_G3: TG.D
- new net NEG_R2: TR1.D
- new net NEG_R3: TR.D
- net B: no longer R18.1, R6.1
- net B2: now also R18.1
- net B3: now also R6.1
- net G: no longer R17.1, R5.1
- net G2: now also R17.1
- net G3: now also R5.1
- net NEG_B: now also PAD3.P; no longer TB.D, TB1.D
- net NEG_G: now also PAD2.P; no longer TG.D, TG1.D
- net NEG_R: now also PAD1.P; no longer TR.D, TR1.D
- net R: no longer R10.1, R14.1
- net R2: now also R14.1
- net R3: now also R10.1

Commit message: w
Parts:
- added RN1, RN2, RN3: YC358TJK-0710KL, SamacSys_Parts:YC358TJK-0710KL
- added RN4, RN5, RN6: YC324-JK-07100RL, SamacSys_Parts:YC324-JK-07100RL
Connections:
- new net N$15: RN1.2, RN1.7, RN4.3
- new net N$16: RN1.3, RN1.8, RN4.2
- new net N$17: RN1.4, RN1.9, RN4.1
Changed lines of the file:
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@@
 <?xml version="1.0" encoding="utf-8"?>
 <!DOCTYPE eagle SYSTEM "eagle.dtd">
-<eagle version="9.2.2">
+<eagle version="9.4.2">
 <drawing>
 <settings>
@@
 <part name="PAD8" library="wirepad" library_urn="urn:adsk.eagle:library:412" deviceset="SMD5" device="" package3d_urn="urn:adsk.eagle:package:30841/1"/>
 <part name="PAD9" library="wirepad" library_urn="urn:adsk.eagle:library:412" deviceset="SMD5" device="" package3d_urn="urn:adsk.eagle:package:30841/1"/>
+<part name="RN1" library="SamacSys_Parts" deviceset="YC358TJK-0710KL" device=""/>
+<part name="RN2" library="SamacSys_Parts" deviceset="YC358TJK-0710KL" device=""/>
+<part name="RN3" library="SamacSys_Parts" deviceset="YC358TJK-0710KL" device=""/>
+<part name="RN4" library="SamacSys_Parts" deviceset="YC324-JK-07100RL" device=""/>
+<part name="RN5" library="SamacSys_Parts" deviceset="YC324-JK-07100RL" device=""/>
+<part name="RN6" library="SamacSys_Parts" deviceset="YC324-JK-07100RL" device=""/>
 </parts>
 <sheets>
@@
 <attribute name="VALUE" x="9.017" y="-18.542" size="1.778" layer="96"/>
 </instance>
+<instance part="RN1" gate="G$1" x="-104.14" y="139.7" smashed="yes" rot="R270">
+<attribute name="NAME" x="-96.52" y="120.65" size="1.778" layer="95" rot="R270" align="center-left"/>
+<attribute name="VALUE" x="-99.06" y="120.65" size="1.778" layer="96" rot="R270" align="center-left"/>
+</instance>
+<instance part="RN2" gate="G$1" x="-124.46" y="96.52" smashed="yes">
+<attribute name="NAME" x="-105.41" y="104.14" size="1.778" layer="95" align="center-left"/>
+<attribute name="VALUE" x="-105.41" y="101.6" size="1.778" layer="96" align="center-left"/>
+</instance>
+<instance part="RN3" gate="G$1" x="-124.46" y="71.12" smashed="yes">
+<attribute name="NAME" x="-105.41" y="78.74" size="1.778" layer="95" align="center-left"/>
+<attribute name="VALUE" x="-105.41" y="76.2" size="1.778" layer="96" align="center-left"/>
+</instance>
+<instance part="RN4" gate="G$1" x="-111.76" y="142.24" smashed="yes" rot="R90">
+<attribute name="NAME" x="-119.38" y="158.75" size="1.778" layer="95" rot="R90" align="center-left"/>
+<attribute name="VALUE" x="-116.84" y="158.75" size="1.778" layer="96" rot="R90" align="center-left"/>
+</instance>
+<instance part="RN5" gate="G$1" x="-76.2" y="99.06" smashed="yes">
+<attribute name="NAME" x="-59.69" y="106.68" size="1.778" layer="95" align="center-left"/>
+<attribute name="VALUE" x="-59.69" y="104.14" size="1.778" layer="96" align="center-left"/>
+</instance>
+<instance part="RN6" gate="G$1" x="-76.2" y="68.58" smashed="yes">
+<attribute name="NAME" x="-59.69" y="76.2" size="1.778" layer="95" align="center-left"/>
+<attribute name="VALUE" x="-59.69" y="73.66" size="1.778" layer="96" align="center-left"/>
+</instance>
 </instances>
 <busses>
@@
 </segment>
 </net>
+<net name="N$15" class="0">
+<segment>
+<pinref part="RN1" gate="G$1" pin="7"/>
+<pinref part="RN1" gate="G$1" pin="2"/>
+<wire x1="-106.68" y1="116.84" x2="-106.68" y2="139.7" width="0.1524" layer="91"/>
+<pinref part="RN4" gate="G$1" pin="3"/>
+<wire x1="-106.68" y1="139.7" x2="-106.68" y2="142.24" width="0.1524" layer="91"/>
+<junction x="-106.68" y="139.7"/>
+</segment>
+</net>
+<net name="N$16" class="0">
+<segment>
+<pinref part="RN4" gate="G$1" pin="2"/>
+<pinref part="RN1" gate="G$1" pin="8"/>
+<wire x1="-109.22" y1="142.24" x2="-109.22" y2="116.84" width="0.1524" layer="91"/>
+<pinref part="RN1" gate="G$1" pin="3"/>
+<wire x1="-109.22" y1="116.84" x2="-109.22" y2="139.7" width="0.1524" layer="91"/>
+<junction x="-109.22" y="116.84"/>
+</segment>
+</net>
+<net name="N$17" class="0">
+<segment>
+<pinref part="RN1" gate="G$1" pin="9"/>
+<pinref part="RN1" gate="G$1" pin="4"/>
+<wire x1="-111.76" y1="116.84" x2="-111.76" y2="139.7" width="0.1524" layer="91"/>
+<pinref part="RN4" gate="G$1" pin="1"/>
+<wire x1="-111.76" y1="139.7" x2="-111.76" y2="142.24" width="0.1524" layer="91"/>
+<junction x="-111.76" y="139.7"/>
+</segment>
+</net>

Commit message: h
Parts:
- removed PAD1, PAD2, PAD3, PAD4, PAD5, PAD6, PAD7, PAD8, PAD9: (no value), wirepad:SMD5
- removed R10, R14, R17, R18, R20, R23, R24, R5, R6: 100, rcl:R-EU_R0805
- removed R13, R15, R16, R19, R21, R22, R3, R4, R9: 10k, rcl:R-EU_R0805
- removed RN3: YC358TJK-0710KL, SamacSys_Parts:YC358TJK-0710KL
- added PB1, PB2, PB3, PG1, PG2, PG3, PR1, PR2, PR3: (no value), wirepad:3,81/1,4
Connections:
- removed net N$10: R21.2, R23.2, TG2.G
- removed net N$12: R22.2, R24.2, TB2.G
- removed net N$15: RN1.2, RN1.7, RN4.3
- removed net N$16: RN1.3, RN1.8, RN4.2
- removed net N$17: RN1.4, RN1.9, RN4.1
- removed net N$2: R3.2, R5.2, TG.G
- removed net N$3: R4.2, R6.2, TB.G
- removed net N$4: R10.2, R9.2, TR.G
- removed net N$6: R13.2, R14.2, TR1.G
- removed net N$7: R15.2, R17.2, TG1.G
- removed net N$8: R16.2, R18.2, TB1.G
- removed net N$9: R19.2, R20.2, TR2.G
- new net TB: RN1.9, RN4.4, TB2.G
- new net TB2: RN1.4, RN5.3, TB1.G
- new net TB3: RN2.4, RN6.3, TB.G
- new net TG: RN1.8, RN4.3, TG2.G
- new net TG2: RN1.3, RN5.2, TG1.G
- new net TG3: RN2.3, RN6.2, TG.G
- new net TR: RN1.7, RN4.2, TR2.G
- new net TR2: RN1.2, RN5.1, TR1.G
- new net TR3: RN2.2, RN6.1, TR.G
- new net VDD1: IC2.VDD, R11.1
- new net VDD2: IC3.VDD, R12.1
- net +12V: now also C1.2, C2.2, C3.2, IN/OUT.2, RN1.1, RN1.6, RN2.1, RN2.6; no longer IN/OUT.4, R13.1, R15.1, R16.1, R19.1, R21.1, R22.1, R3.1, R4.1, R9.1
- net B: now also RN4.8; no longer R24.1
- net B2: now also RN5.7; no longer R18.1
- net B3: now also RN6.7; no longer R6.1
- net DOUT_OUT: now also IN/OUT.4; no longer IN/OUT.2
- net G: now also RN4.7; no longer R23.1
- net G2: now also RN5.6; no longer R17.1
- net G3: now also RN6.6; no longer R5.1
- net NEG_B: now also PB1.P; no longer PAD3.P
- net NEG_B2: now also PB2.P
- net NEG_B3: now also PB3.P
- net NEG_G: now also PG1.P; no longer PAD2.P
- net NEG_G2: now also PG2.P
- net NEG_G3: now also PG3.P
- net NEG_R: now also PR1.P; no longer PAD1.P
- net NEG_R2: now also PR2.P
- net NEG_R3: now also PR3.P
- net R: now also RN4.6; no longer R20.1
- net R2: now also RN5.5; no longer R14.1
- net R3: now also RN6.5; no longer R10.1
- net VDD: no longer C1.2, C2.2, C3.2, IC2.VDD, IC3.VDD, R11.1, R12.1
Other:
- moved on the sheet: RN1, RN2, RN4, RN6
