File: wsleddriver/leddriverv3.brd (EAGLE design)
At the start: 32.3 x 15.4 mm, 13 parts, among them IC1 WS2811-SOP8

Commit message: c
Parts:
- moved R7 3.24 mm to (12.8, 2.29), turned to 270 degrees
- moved SV1 1.40 mm to (5.46, 4.95)
- moved R8 1.31 mm to (8.51, 5.08), turned to 270 degrees
- moved C1 1.02 mm to (10.7, 2.79), turned to 270 degrees
Connections:
- net +12V: now also C1.2
- net VDD: no longer C1.2
Routing:
- net VDD: track 9.50 -> 7.23 mm
- net +12V: track 18.4 -> 16.5 mm
- net N$1: track 7.08 -> 5.53 mm, vias 2 -> 0
- net DOUT: track 3.98 -> 4.63 mm
Other:
- board size 32.3 x 15.4 mm -> 32.3 x 15.5 mm

Commit message: h
Parts:
- moved RN2 0.63 mm to (17.4, 2.29)
Connections:
- net B: no longer RN2.7
- net BT: now also RN2.9
- net G: no longer RN2.8
- net GT: now also RN2.8
- net R: no longer RN2.9
- net RT: now also RN2.7
Routing:
- net BT: track 8.57 -> 17.1 mm
- net B: track 9.18 -> 1.98 mm
- net GT: track 6.47 -> 12.8 mm
- net G: track 7.44 -> 1.98 mm
- net R: track 5.61 -> 1.98 mm
- net RT: track 9.56 -> 12.7 mm
Other:
- board text added: "SR2019"
