File: wsleddriver/leddriverv3.sch (EAGLE design)
At the start: 13 parts, among them IC1 WS2811-SOP8

Commit message: c
Connections:
- net +12V: now also C1.2
- net VDD: no longer C1.2
Changed lines of the file:
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@@
 <?xml version="1.0" encoding="utf-8"?>
 <!DOCTYPE eagle SYSTEM "eagle.dtd">
-<eagle version="9.4.2">
+<eagle version="9.2.2">
 <drawing>
 <settings>
@@
 <part name="P+1" library="supply1" library_urn="urn:adsk.eagle:library:371" deviceset="+12V" device=""/>
 <part name="GND1" library="supply1" library_urn="urn:adsk.eagle:library:371" deviceset="GND" device=""/>
+<part name="P+2" library="supply1" library_urn="urn:adsk.eagle:library:371" deviceset="+12V" device=""/>
 </parts>
 <sheets>
@@
 <attribute name="VALUE" x="-2.54" y="40.64" size="1.778" layer="96"/>
 </instance>
+<instance part="P+2" gate="1" x="96.52" y="73.66" smashed="yes" rot="R270">
+<attribute name="VALUE" x="99.06" y="73.66" size="1.778" layer="96"/>
+</instance>
 </instances>
 <busses>
@@
 <pinref part="P+1" gate="1" pin="+12V"/>
 </segment>
+<segment>
+<pinref part="C1" gate="G$1" pin="2"/>
+<wire x1="83.82" y1="73.66" x2="93.98" y2="73.66" width="0.1524" layer="91"/>
+<pinref part="P+2" gate="1" pin="+12V"/>
+</segment>
 </net>
 <net name="GND" class="0">
@@
 <net name="VDD" class="0">
 <segment>
-<pinref part="C1" gate="G$1" pin="2"/>
-<wire x1="83.82" y1="73.66" x2="93.98" y2="73.66" width="0.1524" layer="91"/>
-<label x="88.9" y="73.66" size="1.778" layer="95"/>
-</segment>
-<segment>
 <pinref part="IC1" gate="G$1" pin="VDD"/>

Commit message: h
Connections:
- net B: no longer RN2.7
- net BT: now also RN2.9
- net G: no longer RN2.8
- net GT: now also RN2.8
- net R: no longer RN2.9
- net RT: now also RN2.7
Other:
- moved on the sheet: RN1, RN2, SV1
